File: hardware/ledaw/ledaw.kicad_sch (KiCad schematic)
At the start: 1 part

Commit message: hw: done codec?
Other:
- sheet codec ports: added CODEC_BCLKS1, CODEC_BCLKS2, CODEC_CLKEN, CODEC_LRCLKS1, CODEC_LRCLKS2, CODEC_SCL, CODEC_SDA, CODEC_SDINS1, CODEC_SDINS2, CODEC_SDOUTS1, CODEC_SDOUTS2, CODEC_~{IRQ}; removed none
Changed lines of the file:
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@@
 	)
 	(sheet
-		(at 129.54 41.91)
-		(size 12.7 24.13)
+		(at 135.89 41.91)
+		(size 30.48 44.45)
 		(exclude_from_sim no)
 		(in_bom yes)
@@
 		)
 		(property "Sheetname" "codec"
-			(at 129.54 41.1984 0)
+			(at 135.89 41.1984 0)
 			(show_name no)
 			(do_not_autoplace no)
@@
 		)
 		(property "Sheetfile" "codec.kicad_sch"
-			(at 129.54 66.6246 0)
+			(at 135.89 86.9446 0)
 			(show_name no)
 			(do_not_autoplace no)
@@
 			)
 		)
+		(pin "CODEC_SDOUTS2" input
+			(at 135.89 80.01 180)
+			(effects
+				(font
+					(size 1.27 1.27)
+				)
+				(justify left)
+			)
+		)
+		(pin "CODEC_SDINS2" input
+			(at 135.89 77.47 180)
+			(effects
+				(font
+					(size 1.27 1.27)
+				)
+				(justify left)
+			)
+		)
+		(pin "CODEC_BCLKS2" input
+			(at 135.89 72.39 180)
+			(effects
+				(font
+					(size 1.27 1.27)
+				)
+				(justify left)
+			)
+		)
+		(pin "CODEC_LRCLKS2" input
+			(at 135.89 74.93 180)
+			(effects
+				(font
+					(size 1.27 1.27)
+				)
+				(justify left)
+			)
+		)
+		(pin "CODEC_SDOUTS1" input
+			(at 135.89 59.69 180)
+			(effects
+				(font
+					(size 1.27 1.27)
+				)
+				(justify left)
+			)
+		)
+		(pin "CODEC_LRCLKS1" input
+			(at 135.89 54.61 180)
+			(effects
+				(font
+					(size 1.27 1.27)
+				)
+				(justify left)
+			)
+		)
+		(pin "CODEC_SDINS1" input
+			(at 135.89 57.15 180)
+			(effects
+				(font
+					(size 1.27 1.27)
+				)
+				(justify left)
+			)
+		)
+		(pin "CODEC_BCLKS1" input
+			(at 135.89 52.07 180)
+			(effects
+				(font
+					(size 1.27 1.27)
+				)
+				(justify left)
+			)
+		)
+		(pin "CODEC_SCL" input
+			(at 135.89 66.04 180)
+			(effects
+				(font
+					(size 1.27 1.27)
+				)
+				(justify left)
+			)
+		)
+		(pin "CODEC_~{IRQ}" input
+			(at 135.89 68.58 180)
+			(effects
+				(font
+					(size 1.27 1.27)
+				)
+				(justify left)
+			)
+		)
+		(pin "CODEC_SDA" input
+			(at 135.89 63.5 180)
+			(effects
+				(font
+					(size 1.27 1.27)
+				)
+				(justify left)
+			)
+		)
+		(pin "CODEC_CLKEN" input
+			(at 135.89 48.26 180)
+			(effects
+				(font
+					(size 1.27 1.27)
+				)
+				(justify left)
+			)
+		)

Commit message: hw:hat
Other:
- sheet codec ports: added none; removed CODEC_BCLKS2, CODEC_LRCLKS2, CODEC_SDINS2, CODEC_SDOUTS2
Changed lines of the file:
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@@
-			)
-		)
-		(pin "CODEC_SDOUTS2" input
-			(at 135.89 80.01 180)
-			(effects
-				(font
-					(size 1.27 1.27)
-				)
-				(justify left)
-			)
-		)
-		(pin "CODEC_SDINS2" input
-			(at 135.89 77.47 180)
-			(effects
-				(font
-					(size 1.27 1.27)
-				)
-				(justify left)
-			)
-		)
-		(pin "CODEC_BCLKS2" input
-			(at 135.89 72.39 180)
-			(effects
-				(font
-					(size 1.27 1.27)
-				)
-				(justify left)
-			)
-		)
-		(pin "CODEC_LRCLKS2" input
-			(at 135.89 74.93 180)
-			(effects
-				(font
-					(size 1.27 1.27)
-				)
-				(justify left)
 			)
 		)
