File: hardware/hat/hat.kicad_pcb (KiCad board)
At the start: 2 copper layers, 65 x 56 mm, 5 parts, among them J1 GPIO

Commit message: hw: assign
Parts:
- added D1: ESDA6V1BC6, Package_TO_SOT_SMD:SOT-23-6, F.Cu at (122.6, 69.6)
- added MK1: MicL, Sensor_Audio:Knowles_LGA-5_3.5x2.65mm, F.Cu at (122.3, 64.7)
- added MK2: MicR, Sensor_Audio:Knowles_LGA-5_3.5x2.65mm, F.Cu at (126.7, 64.7)
- added U3: TPS7A20xxxDBV, Package_TO_SOT_SMD:SOT-23-5, F.Cu at (122.6, 76.2)
- added Y1: 12.288MHz, Oscillator:Oscillator_SMD_SeikoEpson_SG210-4Pin_2.5x2.0mm, F.Cu at (127.4, 69.2)
Connections:
- J1 pad 16: /GPIO23 -> /1V8_EN
