File: hardware/hat/hat.kicad_pcb (KiCad board)
At the start: 2 copper layers, 65 x 56 mm, 10 parts, among them J1 GPIO, U3 TPS7A20xxxDBV, Y1 12.288MHz

Commit message: hw: sync
Parts:
- added C1: 100n, Capacitor_SMD:C_0805_2012Metric, F.Cu at (127.5, 100.4)
- added C10: 1uF, Capacitor_SMD:C_0805_2012Metric, F.Cu at (114.7, 72.6)
- added C11: 1uF, Capacitor_SMD:C_0805_2012Metric, F.Cu at (114.7, 75.6)
- added C12: 0.1uF, Capacitor_SMD:C_0805_2012Metric, F.Cu at (119.2, 54.5)
- added C13: 1uF, Capacitor_SMD:C_0805_2012Metric, F.Cu at (119.2, 57.5)
- added C14: 10uF, Capacitor_SMD:C_0805_2012Metric, F.Cu at (119.2, 60.5)
- added C15: 1uF, Capacitor_SMD:C_0805_2012Metric, F.Cu at (119.2, 63.5)
- added C16: 1uF, Capacitor_SMD:C_0805_2012Metric, F.Cu at (119.2, 66.5)
- added C17: 10uF, Capacitor_SMD:C_0805_2012Metric, F.Cu at (119.2, 69.6)
- added C18: 1uF, Capacitor_SMD:C_0805_2012Metric, F.Cu at (119.2, 72.6)
- added C19: 1uF, Capacitor_SMD:C_0805_2012Metric, F.Cu at (119.2, 75.6)
- added C2: 1uF, Capacitor_SMD:C_0805_2012Metric, F.Cu at (127.5, 103.4)
- added C20: 1uF, Capacitor_SMD:C_0805_2012Metric, F.Cu at (123.6, 54.5)
- added C21: 1uF, Capacitor_SMD:C_0805_2012Metric, F.Cu at (123.6, 57.5)
- added C22: 1uF, Capacitor_SMD:C_0805_2012Metric, F.Cu at (123.6, 60.5)
- added C23: 0.1uF, Capacitor_SMD:C_0805_2012Metric, F.Cu at (123.6, 63.5)
- added C24: 1uF, Capacitor_SMD:C_0805_2012Metric, F.Cu at (123.6, 66.5)
- added C25: 2.2uF, Capacitor_SMD:C_0805_2012Metric, F.Cu at (123.6, 69.6)
- added C26: 10uF, Capacitor_SMD:C_0805_2012Metric, F.Cu at (123.6, 72.6)
- added C27: 10uF, Capacitor_SMD:C_0805_2012Metric, F.Cu at (123.6, 75.6)
- added C28: 470pF, Capacitor_SMD:C_0805_2012Metric, F.Cu at (128.1, 54.5)
- added C29: 470pF, Capacitor_SMD:C_0805_2012Metric, F.Cu at (128.1, 57.5)
- added C3: 1uF, Capacitor_SMD:C_0805_2012Metric, F.Cu at (127.5, 106.4)
- added C30: 470pF, Capacitor_SMD:C_0805_2012Metric, F.Cu at (128.1, 60.5)
- added C31: 470pF, Capacitor_SMD:C_0805_2012Metric, F.Cu at (128.1, 63.5)
- added C4: 0.1uF X7R, Capacitor_SMD:C_0805_2012Metric, F.Cu at (114.7, 54.5)
- added C5: 0.1uF X7R, Capacitor_SMD:C_0805_2012Metric, F.Cu at (114.7, 57.5)
- added C6: 0.1uF X7R, Capacitor_SMD:C_0805_2012Metric, F.Cu at (114.7, 60.5)
- added C7: 47pF, Capacitor_SMD:C_0805_2012Metric, F.Cu at (114.7, 63.5)
- added C8: 1uF, Capacitor_SMD:C_0805_2012Metric, F.Cu at (114.7, 66.5)
- added C9: 1uF, Capacitor_SMD:C_0805_2012Metric, F.Cu at (114.7, 69.6)
- added FB1: 600Ohm@100MHz, Inductor_SMD:L_0805_2012Metric, F.Cu at (144.8, 81.7)
- added FB2: 600Ohm@100MHz, Inductor_SMD:L_0805_2012Metric, F.Cu at (144.8, 84.5)
- added FB3: 600Ohm@100MHz, Inductor_SMD:L_0805_2012Metric, F.Cu at (144.8, 87.2)
- added FB4: 600Ohm@100MHz, Inductor_SMD:L_0805_2012Metric, F.Cu at (144.8, 90.0)
- added FB5: 600Ohm@100MHz, Inductor_SMD:L_0805_2012Metric, F.Cu at (144.8, 92.7)
- added FB6: 600Ohm@100MHz, Inductor_SMD:L_0805_2012Metric, F.Cu at (144.8, 95.5)
- added J2: Uart, Connector_PinHeader_2.54mm:PinHeader_1x03_P2.54mm_Vertical, F.Cu at (122.9, 101.1)
- added J3: LineIn, Connector_Audio:Jack_3.5mm_PJ311_Horizontal, F.Cu at (135.8, 62.8)
- added J4: LineOut, Connector_Audio:Jack_3.5mm_PJ311_Horizontal, F.Cu at (146.9, 62.8)
- added J5: Headphone, Connector_Audio:Jack_3.5mm_PJ320D_Horizontal, F.Cu at (151.8, 74.8)
- added JP1: ID_WP, Jumper:SolderJumper-3_P1.3mm_Open_RoundedPad1.0x1.5mm_NumberLabels, F.Cu at (132.7, 116.9)
- added LS1: SpeakerL, TerminalBlock_Phoenix:TerminalBlock_Phoenix_MKDS-1,5-2-5.08_1x02_P5.08mm_Horizontal, F.Cu at (133.9, 75.5)
- added LS2: SpeakerR, TerminalBlock_Phoenix:TerminalBlock_Phoenix_MKDS-1,5-2-5.08_1x02_P5.08mm_Horizontal, F.Cu at (133.9, 87.7)
- added R1: 10k, Resistor_SMD:R_0805_2012Metric, F.Cu at (131.9, 100.3)
- added R2: 3.9k, Resistor_SMD:R_0805_2012Metric, F.Cu at (131.9, 103.3)
- added R3: 3.9k, Resistor_SMD:R_0805_2012Metric, F.Cu at (131.9, 106.2)
- added R4: 10k, Resistor_SMD:R_0805_2012Metric, F.Cu at (154.6, 54.5)
- added R5: 2.2k, Resistor_SMD:R_0805_2012Metric, F.Cu at (154.6, 57.4)
- added TP1: MICBIAS, TestPoint:TestPoint_Pad_D2.0mm, F.Cu at (114.5, 79.1)
- added TP10: JACKSENSE, TestPoint:TestPoint_Pad_D2.0mm, F.Cu at (122.6, 83.2)
- added TP11: RECP, TestPoint:TestPoint_Pad_D2.0mm, F.Cu at (122.6, 87.2)
- added TP12: RECN, TestPoint:TestPoint_Pad_D2.0mm, F.Cu at (122.6, 91.3)
- added TP13: SPKLP, TestPoint:TestPoint_Pad_D2.0mm, F.Cu at (126.7, 79.1)
- added TP14: SPKLN, TestPoint:TestPoint_Pad_D2.0mm, F.Cu at (126.7, 83.2)
- added TP15: SPKRP, TestPoint:TestPoint_Pad_D2.0mm, F.Cu at (126.7, 87.2)
- added TP16: SPKRN, TestPoint:TestPoint_Pad_D2.0mm, F.Cu at (126.7, 91.3)
- added TP17: LDO_IN, TestPoint:TestPoint_Pad_D2.0mm, F.Cu at (122.7, 110.5)
- added TP18: LDO_OUT, TestPoint:TestPoint_Pad_D2.0mm, F.Cu at (122.7, 114.6)
- added TP19: 5V, TestPoint:TestPoint_THTPad_1.5x1.5mm_Drill0.7mm, F.Cu at (118.9, 100.6)
- added TP2: INA1, TestPoint:TestPoint_Pad_D2.0mm, F.Cu at (114.5, 83.2)
- added TP20: GND, TestPoint:TestPoint_THTPad_1.5x1.5mm_Drill0.7mm, F.Cu at (118.9, 104.2)
- added TP21: 3V3, TestPoint:TestPoint_THTPad_1.5x1.5mm_Drill0.7mm, F.Cu at (118.9, 107.7)
- added TP3: INA2, TestPoint:TestPoint_Pad_D2.0mm, F.Cu at (114.5, 87.2)
- added TP4: CODEC_MCLK, TestPoint:TestPoint_Pad_D2.0mm, F.Cu at (114.5, 91.3)
- added TP5: MIC2P, TestPoint:TestPoint_Pad_D2.0mm, F.Cu at (118.6, 79.1)
- added TP6: MIC2N, TestPoint:TestPoint_Pad_D2.0mm, F.Cu at (118.6, 83.2)
- added TP7: HPSNS, TestPoint:TestPoint_Pad_D2.0mm, F.Cu at (118.6, 87.2)
- added TP8: HPR, TestPoint:TestPoint_Pad_D2.0mm, F.Cu at (118.6, 91.3)
- added TP9: HPL, TestPoint:TestPoint_Pad_D2.0mm, F.Cu at (122.6, 79.1)
- added U1: CAT24C256, Package_SO:SOIC-8_3.9x4.9mm_P1.27mm, F.Cu at (128.9, 111.9)
- added U2: TPS7A20xxxDBV, Package_TO_SOT_SMD:SOT-23-5, F.Cu at (127.3, 117.5)
- added U4: MAX98089ETN_T, footprints:MAX98089ETN_T, F.Cu at (152.3, 85.0)
- U3: value TPS7A20xxxDBV -> Oled; footprint Package_TO_SOT_SMD:SOT-23-5 -> Connector_PinHeader_2.54mm:PinHeader_1x07_P2.54mm_Vertical
- moved MK2 38.7 mm to (153.7, 92.3)
- moved MK1 38.7 mm to (149.3, 92.3)
- moved D1 33.5 mm to (155.0, 61.3)
- moved Y1 27.5 mm to (154.7, 65.5)
- moved U3 26.1 mm to (114.8, 101.2)
Connections:
- U3 pad 3: /1V8_EN -> /GPIO10/SPI0.MOSI
- U3 pad 4: unconnected-(U3-NC-Pad4) -> /GPIO11/SPI0.SCLK
- U3 pad 5: +1V8 -> /GPIO8/SPI0.CE0

Commit message: hw: placement
Parts:
- J3, J4: footprint Connector_Audio:Jack_3.5mm_PJ311_Horizontal -> Connector_Audio:Jack_3.5mm_CUI_SJ-3523-SMT_Horizontal
- J5: footprint Connector_Audio:Jack_3.5mm_PJ320D_Horizontal -> footprints:CUI_SJ-43514-SMT-TR
- moved C23 83.4 mm to (180.0, 125.0)
- moved C28 83.4 mm to (184.4, 116.0)
- moved C29 83.4 mm to (184.4, 119.0)
- moved C30 83.4 mm to (184.4, 122.0)
- moved C31 83.4 mm to (184.4, 125.0)
- moved JP1 66.5 mm to (112.5, 53.5)
- moved U2 65.7 mm to (139.9, 53.0)
- moved U3 62.1 mm to (162.0, 60.8)
- moved U1 61.0 mm to (105.5, 55.5)
- moved C3 55.2 mm to (144.9, 54.0)
- moved C2 55.2 mm to (144.9, 51.0)
- moved R3 54.1 mm to (117.8, 54.0)
- moved C5 48.7 mm to (156.5, 82.5)
- moved J2 47.7 mm to (121.9, 53.5), turned to 90 degrees
- moved R2 46.3 mm to (116.8, 59.5)
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Connections:
- C10 pad 2: Net-(U4-MIC2P) -> Net-(U4-INA1/EXTMICP)
- C11 pad 2: Net-(U4-MIC2N) -> Net-(U4-INA2/EXTMICN)
- C8 pad 2: Net-(U4-INA1/EXTMICP) -> Net-(U4-MIC2P)
- C9 pad 2: Net-(U4-INA2/EXTMICN) -> Net-(U4-MIC2N)
- TP2 pad 1: Net-(U4-INA1/EXTMICP) -> Net-(U4-MIC2P)
- TP3 pad 1: Net-(U4-INA2/EXTMICN) -> Net-(U4-MIC2N)
- TP5 pad 1: Net-(U4-MIC2P) -> Net-(U4-INA1/EXTMICP)
- TP6 pad 1: Net-(U4-MIC2N) -> Net-(U4-INA2/EXTMICN)
Other:
- outline, holes or cut-outs redrawn
- board text removed: "CAMERA (OPTIONAL)"
- board text removed: "DISPLAY (OPTIONAL)"
- board text removed: "Extend PCB edge 0.5mm if using SMT header"
- board text removed: "USB"

Commit message: place all components
Parts:
- TP1, TP10, TP11, TP12, TP13, TP14, TP15, TP16, TP17, TP18, TP19, TP2, TP20, TP21, TP3, TP4, TP5, TP6, TP7, TP8, TP9: moved to B.Cu
- moved C28 86.6 mm to (114.5, 65.0)
- moved C29 86.0 mm to (114.5, 69.0)
- moved C30 84.3 mm to (114.5, 75.0)
- moved C31 83.8 mm to (114.4, 79.0)
- moved C23 74.4 mm to (143.0, 60.5)
- moved TP17 47.3 mm to (112.0, 113.0), turned to 180 degrees
- moved TP18 47.3 mm to (112.0, 117.0), turned to 180 degrees
- moved TP1 40.7 mm to (156.1, 110.5), turned to 180 degrees
- moved TP2 40.7 mm to (156.1, 114.5), turned to 180 degrees
- moved TP3 40.7 mm to (156.1, 118.5), turned to 180 degrees
- moved TP4 40.7 mm to (156.1, 122.6), turned to 180 degrees
- moved TP20 38.3 mm to (106.0, 111.5), turned to 180 degrees
- moved TP19 38.3 mm to (106.0, 108.0), turned to 180 degrees
- moved TP21 38.3 mm to (106.0, 115.1), turned to 180 degrees
- moved TP7 33.2 mm to (152.1, 118.5), turned to 180 degrees
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Other:
- copper layers 2 -> 4
