File: hardware/hat/codec.kicad_sch (KiCad schematic)
At the start: 68 parts, among them J201 LineOut, J202 LineIn, J203 Headphone, U201 MAX98089ETN_T, U202 TPS7A20xxxDBV, Y201 12.288MHz

Commit message: use H label for 1v8en
Connections:
- net 1V8_EN renamed CODEC_1V8EN
Changed lines of the file:
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@@
-	(wire
-		(pts
-			(xy 41.91 171.45) (xy 49.53 171.45)
-		)
-		(stroke
-			(width 0)
-			(type default)
-		)
-	)
 	(wire
 		(pts
@@
 		(pts
 			(xy 82.55 172.72) (xy 82.55 176.53)
-		)
-		(stroke
-			(width 0)
-			(type default)
-		)
-	)
-	(wire
-		(pts
-			(xy 49.53 175.26) (xy 49.53 171.45)
 		)
 		(stroke
@@
 		)
 	)
-	(label "1V8_EN"
-		(at 41.91 175.26 0)
-		(effects
-			(font
-				(size 1.27 1.27)
-			)
-			(justify left bottom)
-		)
-	)
 	(label "DIGMICDATA"
 		(at 62.23 87.63 180)
@@
 	(label "DIGMICCLK"
 		(at 86.36 101.6 0)
-		(effects
-			(font
-				(size 1.27 1.27)
-			)
-			(justify left bottom)
-		)
-	)
-	(label "GPIO23"
-		(at 41.91 171.45 0)
 		(effects
 			(font
@@
 		(effects
 			(font
+				(size 1.27 1.27)
+			)
+			(justify right)
+		)
+	)
+	(hierarchical_label "CODEC_1V8EN"
+		(shape input)
+		(at 41.91 175.26 180)
+		(effects
+			(font

Commit message: delete FB and cap from hat
Parts:
- removed C221: 47pF, Capacitor_SMD:C_0805_2012Metric, symbol Device:C_Small
- removed FB205: 600Ohm@100MHz, Inductor_SMD:L_0805_2012Metric, symbol Device:FerriteBead_Small
- renumbered C222 to C221, C223 to C222, C224 to C223, C225 to C224, C226 to C225, C227 to C226, C228 to C227, C229 to C228, C230 to C229, FB206 to FB205
Connections:
- net JackS: now also C220.1
