File: hardware/board/mcu.kicad_sch (KiCad schematic)
At the start: 7 parts, among them J1 MidiIn, J2 MidiOut, SW1 RotaryEncoder, SW2 RotaryEncoder, SW3 RotaryEncoder, SW4 RotaryEncoder, U1 RP2350B

Commit message: add hella parts
Parts:
- removed SW1, SW2, SW3, SW4: RotaryEncoder, symbol Device:RotaryEncoder
- added C1, C2: 15p, Capacitor_SMD:C_0402_1005Metric, symbol Device:C
- added C10, C11, C12, C13, C14, C15, C16, C17, C18, C19, C6: 100n, Capacitor_SMD:C_0402_1005Metric, symbol Device:C
- added C3, C5: 4.7u, RP2350_80QFN_minimal:C_0402_1005Metric_small_pads, symbol Device:C
- added C4, C7: 10u, Capacitor_SMD:C_0805_2012Metric, symbol Device:C
- added C8, C9: 4.7u, Capacitor_SMD:C_0402_1005Metric, symbol Device:C
- added ENC1, ENC2, ENC3, ENC4: RotaryEncoder_Switch, ledaw:XDCR_PEC11R-4015F-S0024, symbol Device:RotaryEncoder_Switch
- added J1: USB_B_Micro, Connector_USB:USB_Micro-B_Amphenol_10103594-0001LF_Horizontal, symbol Connector:USB_B_Micro
- added J2: SM03B-SRSS-TB, Connector_JST:JST_SH_SM03B-SRSS-TB_1x03-1MP_P1.00mm_Horizontal, symbol Connector_Generic_MountingPin:Conn_01x03_MountingPin
- added L1: 3.3u, RP2350_80QFN_minimal:L_pol_2016, symbol Device:L
- added R1, R2, R4: 1k, Resistor_SMD:R_0402_1005Metric, symbol Device:R
- added R3: 33, Resistor_SMD:R_0402_1005Metric, symbol Device:R
- added R5, R6: 27, Resistor_SMD:R_0402_1005Metric, symbol Device:R
- added SW1, SW2: SW_Push, Button_Switch_SMD:SW_Push_1P1T_NO_Vertical_Wuerth_434133025816, symbol Switch:SW_Push
- added U1: NCP1117-3.3_SOT223, Package_TO_SOT_SMD:SOT-223-3_TabPin2, symbol Regulator_Linear:NCP1117-3.3_SOT223
- added U2: RP2350_80QFN, RP2350_80QFN_minimal:RP2350-QFN-80-1EP_10x10_P0.4mm_EP3.4x3.4mm_ThermalVias, symbol MCU_RaspberryPi_RP2350:RP2350_80QFN
- added U4: THB001P, ledaw:THB001P, symbol THB001P:THB001P
- added Y1: ABM8-272-T3, Crystal:Crystal_SMD_3225-4Pin_3.2x2.5mm, symbol Device:Crystal_GND24
- J3: renamed from J1; footprint (none) -> ledaw:CUI_SJ-3523-SMT-TR
- J4: renamed from J2; footprint (none) -> ledaw:CUI_SJ-3523-SMT-TR
- renumbered U1 to U3
Connections:
- new net: R1.1, SW2.1
- new net: R5.2, U2.67 (USB_DP)
- new net: C2.1, R2.2, Y1.3
- new net: U4.A, U4.B
- new net: U4.C, U4.D
- new net: R6.2, U2.66 (USB_DM)
- new net +1V1: C10.1, C5.1, C6.1, C9.1, L1.1, U2.10 (DVDD), U2.32 (DVDD), U2.51 (DVDD), U2.65 (VREG_FB)
- new net +3V3: C11.1, C12.1, C13.1, C14.1, C15.1, C16.1, C17.1, C18.1, C19.1, C3.1, C7.1, R3.1, U1.2 (VO), U2.15 (IOVDD), U2.24 (IOVDD), U2.29 (IOVDD), U2.41 (IOVDD), U2.5 (IOVDD), U2.50 (IOVDD), U2.59 (ADC_AVDD), U2.60 (IOVDD), U2.64 (VREG_VIN), U2.68 (USB_OTP_VDD), U2.69 (QSPI_IOVDD), U2.76 (IOVDD)
- new net GND: C1.2, C10.2, C11.2, C12.2, C13.2, C14.2, C15.2, C16.2, C17.2, C18.2, C19.2, C2.2, C3.2, C4.2, C5.2, C6.2, C7.2, C8.2, C9.2, J1.5 (GND), J1.6 (Shield), J2.2 (Pin_2), J2.MP (MountPin), R1.2, SW1.1, U1.1 (GND), U2.62 (VREG_PGND), U2.81 (GND), Y1.2, Y1.4
- new net GPIO0: U2.77 (GPIO0)
- new net GPIO1: U2.78 (GPIO1)
- new net GPIO10: U2.8 (GPIO10)
- new net GPIO11: U2.9 (GPIO11)
- new net GPIO12: U2.11 (GPIO12)
- new net GPIO13: U2.12 (GPIO13)
- new net GPIO14: U2.13 (GPIO14)
- new net GPIO15: U2.14 (GPIO15)
- new net GPIO16: U2.16 (GPIO16)
- new net GPIO17: U2.17 (GPIO17)
- new net GPIO18: U2.18 (GPIO18)
- new net GPIO19: U2.19 (GPIO19)
- new net GPIO2: U2.79 (GPIO2)
- new net GPIO20: U2.20 (GPIO20)
- new net GPIO21: U2.21 (GPIO21)
- new net GPIO22: U2.22 (GPIO22)
- new net GPIO23: U2.23 (GPIO23)
- new net GPIO24: U2.25 (GPIO24)
- new net GPIO25: U2.26 (GPIO25)
- new net GPIO26: U2.27 (GPIO26)
- new net GPIO27: U2.28 (GPIO27)
- new net GPIO28: U2.36 (GPIO28)
- new net GPIO29: U2.37 (GPIO29)
- new net GPIO3: U2.80 (GPIO3)
- new net GPIO30: U2.38 (GPIO30)
- new net GPIO31: U2.39 (GPIO31)
- new net GPIO32: U2.40 (GPIO32)
- new net GPIO33: U2.42 (GPIO33)
- new net GPIO34: U2.43 (GPIO34)
- new net GPIO35: U2.44 (GPIO35)
- new net GPIO36: U2.45 (GPIO36)
- new net GPIO37: U2.46 (GPIO37)
- new net GPIO38: U2.47 (GPIO38)
- new net GPIO39: U2.48 (GPIO39)
- new net GPIO4: U2.1 (GPIO4)
- new net GPIO40_ADC0: U2.49 (GPIO40_ADC0)
- new net GPIO41_ADC1: U2.52 (GPIO41_ADC1)
- new net GPIO42_ADC2: U2.53 (GPIO42_ADC2)
- new net GPIO43_ADC3: U2.54 (GPIO43_ADC3)
- new net GPIO44_ADC4: U2.55 (GPIO44_ADC4)
- new net GPIO45_ADC5: U2.56 (GPIO45_ADC5)
- new net GPIO46_ADC6: U2.57 (GPIO46_ADC6)
- new net GPIO47_ADC7: U2.58 (GPIO47_ADC7)
- new net GPIO5: U2.2 (GPIO5)
- new net GPIO6: U2.3 (GPIO6)
- new net GPIO7: U2.4 (GPIO7)
- new net GPIO8: U2.6 (GPIO8)
- new net GPIO9: U2.7 (GPIO9)
- new net QSPI_SCLK: U2.71 (QSPI_SCLK)
- new net QSPI_SD0: U2.72 (QSPI_SD0)
- new net QSPI_SD1: U2.74 (QSPI_SD1)
- new net QSPI_SD2: U2.73 (QSPI_SD2)
- new net QSPI_SD3: U2.70 (QSPI_SD3)
- new net QSPI_SS: R4.1, U2.75 (QSPI_SS)
- new net RUN: SW2.2, U2.35 (RUN)
- new net SWCLK: J2.1 (Pin_1), U2.33 (SWCLK)
- new net SWD: J2.3 (Pin_3), U2.34 (SWD)
- new net USB_D+: J1.3 (D+), R5.1
- new net USB_D-: J1.2 (D-), R6.1
- new net VBUS: C4.1, J1.1 (VBUS), U1.3 (VI)
- new net VREG_AVDD: C8.1, R3.2, U2.61 (VREG_AVDD)
- new net VREG_LX: L1.2, U2.63 (VREG_LX)
- new net XIN: C1.1, U2.30 (XIN), Y1.1
- new net XOUT: R2.1, U2.31 (XOUT)
- new net ~{USB_BOOT}: R4.2, SW1.2
- no-connect marks 0 -> 1
Other:
- sheet buttons ports: added matrix_C0, matrix_C1, matrix_C2, matrix_C3, matrix_C4, matrix_C5, matrix_C6, matrix_R0, matrix_R1, matrix_R2, matrix_R3, matrix_R4, matrix_R5; removed none
- note added: "12MHz Crystal"
- note added: "JST Debug Connector"
- note added: "Make sure R7 and R8 are close to RP2350"
- note added: "Power"
- note removed: "TODO JOYSTICK"
- moved on the sheet: J3, J4, U3

Commit message: hella footprints and trying out layouts
Parts:
- removed U3: RP2350B, Package_DFN_QFN:QFN-80-1EP_10x10mm_P0.4mm_EP3.4x3.4mm, symbol MCU_RaspberryPi:RP2350B
- J3, J4: footprint ledaw:CUI_SJ-3523-SMT-TR -> Connector_Audio:Jack_3.5mm_CUI_SJ1-3525N_Horizontal
Other:
- moved on the sheet: ENC1, ENC2, ENC3, ENC4, J3, J4, U4A, U4B, U4C

Commit message: more placement
Parts:
- added C50: 10u, Capacitor_SMD:C_0805_2012Metric, symbol Device:C
- renumbered SW1 to SW101, SW2 to SW102
Connections:
- net +3V3: now also C50.1
- net GND: now also C50.2
Other:
- sheet buttons ports: added matrix_C10, matrix_C11, matrix_C12, matrix_C13, matrix_C7, matrix_C8, matrix_C9; removed matrix_R3, matrix_R4, matrix_R5
- note added: "close to 3v3 pin on source"

Commit message: encoder
Parts:
- added C51, C52, C53, C54, C55, C56, C57, C58: 10nF, symbol Device:C_Small
- added R10, R11, R12, R13, R14, R15, R16, R17, R18, R19, R20, R21, R22, R23, R24, R25: 10k, symbol Device:R_Small
Connections:
- net +3V3: now also R10.1, R12.1, R14.1, R16.1, R18.1, R20.1, R22.1, R24.1
- net GND: now also ENC1.C, ENC1.S1, ENC2.C, ENC2.S1, ENC3.C, ENC3.S1, ENC4.C, ENC4.S1, C51.2, C52.2, C53.2, C54.2, C55.2, C56.2, C57.2, C58.2
- net at ENC4.A: now also R22.2, R23.1
- net at ENC4.B: now also R24.2, R25.1
- net ENC4_SW: now reaches ENC4.S2
- net at ENC2.A: now also R14.2, R15.1
- net at ENC2.B: now also R16.2, R17.1
- net ENC2_SW: now reaches ENC2.S2
- net at ENC1.A: now also R10.2, R11.1
- net at ENC1.B: now also R12.2, R13.1
- net ENC1_SW: now reaches ENC1.S2
- net at ENC3.A: now also R18.2, R19.1
- net at ENC3.B: now also R20.2, R21.1
- net ENC3_SW: now reaches ENC3.S2
- new net ENC1_A: C51.1, R11.2
- new net ENC1_B: C52.1, R13.2
- new net ENC2_A: C53.1, R15.2
- new net ENC2_B: C54.1, R17.2
- new net ENC3_A: C55.1, R19.2
- new net ENC3_B: C56.1, R21.2
- new net ENC4_A: C57.1, R23.2
- new net ENC4_B: C58.1, R25.2
Other:
- moved on the sheet: ENC1, J3, J4

Commit message: midi
Parts:
- added C59: 100nF, symbol Device:C_Small
- added D42: LL4148, Diode_SMD:D_MiniMELF, symbol Diode:LL4148
- added R26: 220, symbol Device:R_Small
- added R27: 10, symbol Device:R_Small
- added R28: 33, symbol Device:R_Small
- added U7: TLP2310, Package_SO:SO-5-6_4.55x3.7mm_P1.27mm, symbol Isolator:TLP2310
- added U8: 74AHC1G125, symbol 74xGxx:74AHC1G125
Connections:
- net +3V3: now also U4.VR1_3, U4.VR2_3, C59.1, R28.2, U7.6 (VDD), U8.5 (VCC)
- net GND: now also J3.S, J4.S, U4.C, U4.D, U4.VR1_1, U4.VR2_1, C59.2, U7.4 (GND), U8.1, U8.3 (GND)
- net at J3.R: now also R26.1
- net at J3.T: now also D42.2 (A), U7.3 (K)
- net JOYSTICK_Y: now reaches U4.VR2_2
- net JOYSTICK_SW: now reaches U4.A, U4.B
- net JOYSTICK_X: now reaches U4.VR1_2
- net at J4.R: now also R28.1
- net at J4.T: now also R27.2
- new net: D42.1 (K), R26.2, U7.1 (A)
- new net: R27.1, U8.4
- new net MIDI_IN: U7.5 (VO)
- new net MIDI_OUT: U8.2
Other:
- note added: "4"
- note added: "5"
- note added: "MIDI standard: T: sink R: Source S: Shield https://minimidi.world/"
- note added: "TODO double check joystick orientation. but fixable in code so it doesn't really matter"
- moved on the sheet: J3, J4, U4A, U4B, U4C

Commit message: efuse
Parts:
- removed C4, C7: 10u, Capacitor_SMD:C_0805_2012Metric, symbol Device:C
- removed J1: USB_B_Micro, Connector_USB:USB_Micro-B_Amphenol_10103594-0001LF_Horizontal, symbol Connector:USB_B_Micro
- removed R1, R4: 1k, Resistor_SMD:R_0402_1005Metric, symbol Device:R
- removed R5, R6: 27, Resistor_SMD:R_0402_1005Metric, symbol Device:R
- removed SW101, SW102: SW_Push, Button_Switch_SMD:SW_Push_1P1T_NO_Vertical_Wuerth_434133025816, symbol Switch:SW_Push
- removed U1: NCP1117-3.3_SOT223, Package_TO_SOT_SMD:SOT-223-3_TabPin2, symbol Regulator_Linear:NCP1117-3.3_SOT223
- C51, C52, C53, C54, C55, C56, C57, C58, C59: footprint (none) -> Capacitor_SMD:C_0805_2012Metric
- R10, R11, R12, R13, R14, R15, R16, R17, R18, R19, R20, R21, R22, R23, R24, R25, R26, R27, R28: footprint (none) -> Resistor_SMD:R_0805_2012Metric
Connections:
- net GPIO23 is gone; now on net ENC1_A: U2.23 (GPIO23)
- net GPIO24 is gone; now on net ENC1_B: U2.25 (GPIO24)
- net GPIO25 is gone; now on net ENC2_A: U2.26 (GPIO25)
- net GPIO26 is gone; now on net ENC2_B: U2.27 (GPIO26)
- net GPIO27 is gone; now on net ENC3_A: U2.28 (GPIO27)
- net GPIO28 is gone; now on net ENC3_B: U2.36 (GPIO28)
- net GPIO29 is gone; now on net ENC4_A: U2.37 (GPIO29)
- net GPIO30 is gone; now on net ENC4_B: U2.38 (GPIO30)
- net GPIO31 is gone; now on net ENC1_SW: U2.39 (GPIO31)
- net GPIO32 is gone; now on net ENC2_SW: U2.40 (GPIO32)
- net GPIO33 is gone; now on net ENC3_SW: U2.42 (GPIO33)
- net GPIO34 is gone; now on net ENC4_SW: U2.43 (GPIO34)
- net GPIO35 is gone; now on net JOYSTICK_SW: U2.44 (GPIO35)
- net GPIO40_ADC0 is gone; now on net JOYSTICK_X: U2.49 (GPIO40_ADC0)
- net GPIO41_ADC1 is gone; now on net JOYSTICK_Y: U2.52 (GPIO41_ADC1)
- net MIDI_IN is gone; now on net MIDI_RX: U7.5 (VO)
- net MIDI_OUT is gone; now on net MIDI_TX: U8.2
- net GPIO0 renamed MIDI_TX
- net GPIO1 renamed MIDI_RX
- net GPIO10 renamed matrix_C1
- net GPIO11 renamed matrix_C2
- net GPIO12 renamed matrix_C3
- net GPIO13 renamed matrix_C4
- net GPIO14 renamed matrix_C5
- net GPIO15 renamed matrix_C6
- net GPIO16 renamed matrix_C7
- net GPIO17 renamed matrix_C8
- net GPIO18 renamed matrix_C9
- net GPIO19 renamed matrix_C10
- net GPIO20 renamed matrix_C11
- net GPIO21 renamed matrix_C12
- net GPIO22 renamed matrix_C13
- net GPIO36: no longer names the net of U2.45 (GPIO36)
- net GPIO37: no longer names the net of U2.46 (GPIO37)
- net GPIO38: no longer names the net of U2.47 (GPIO38)
- net GPIO39: no longer names the net of U2.48 (GPIO39)
- net GPIO4 renamed CM4_TX
- net GPIO42_ADC2: no longer names the net of U2.53 (GPIO42_ADC2)
- net GPIO43_ADC3: no longer names the net of U2.54 (GPIO43_ADC3)
- net GPIO44_ADC4: no longer names the net of U2.55 (GPIO44_ADC4)
- net GPIO45_ADC5: no longer names the net of U2.56 (GPIO45_ADC5)
- net GPIO46_ADC6: no longer names the net of U2.57 (GPIO46_ADC6)
- net GPIO47_ADC7: no longer names the net of U2.58 (GPIO47_ADC7)
- net GPIO5 renamed CM5_TX
- net GPIO6 renamed matrix_R0
- net GPIO7 renamed matrix_R1
- net GPIO8 renamed matrix_R2
- net GPIO9 renamed matrix_C0
- no-connect marks 1 -> 2
Other:
- note removed: "Make sure R7 and R8 are close to RP2350"
- note removed: "Power"

Commit message: wip usb
Connections:
- net CM4_TX renamed MCU_RX
- net CM5_TX renamed MCU_TX
Other:
- note added: "from CM4 perspective so MCU_RX goes to UART1 TX"
Changed lines of the file:
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@@
 		)
 	)
+	(text "from CM4 perspective\nso MCU_RX goes to UART1 TX"
+		(exclude_from_sim no)
+		(at 197.612 85.344 0)
+		(effects
+			(font
+				(size 1.27 1.27)
+			)
+			(justify left)
+		)
+	)
 	(junction
 		(at 342.9 107.95)
@@
 		)
 	)
-	(label "SWD"
-		(at 129.54 250.19 0)
-		(effects
-			(font
-				(size 1.27 1.27)
-			)
-			(justify left bottom)
-		)
-	)
 	(label "MIDI_RX"
 		(at 299.72 267.97 180)
@@
 		)
 	)
-	(label "SWCLK"
-		(at 129.54 245.11 0)
-		(effects
-			(font
-				(size 1.27 1.27)
-			)
-			(justify left bottom)
-		)
-	)
 	(label "matrix_C10"
 		(at 194.31 127 180)
@@
 		)
 	)
-	(hierarchical_label "CM5_TX"
+	(hierarchical_label "MCU_TX"
 		(shape input)
 		(at 194.31 91.44 0)
@@
 		)
 	)
-	(hierarchical_label "CM4_TX"
+	(hierarchical_label "SWD"
+		(shape input)
+		(at 129.54 250.19 180)
+		(effects
+			(font
+				(size 1.27 1.27)
+			)
+			(justify right)
+		)
+	)
+	(hierarchical_label "MCU_RX"
 		(shape input)
 		(at 194.31 88.9 0)
@@
 		)
 	)
+	(hierarchical_label "SWCLK"
+		(shape input)
+		(at 129.58 245.11 180)
+		(effects
+			(font
+				(size 1.27 1.27)
+			)
+			(justify right)
+		)
+	)
