File: hardware/board/mcu.kicad_sch (KiCad schematic)
At the start: 62 parts, among them J2 SM03B-SRSS-TB, J3 MidiIn, J4 MidiOut, U2 RP2350_80QFN, U4 THB001P, U7 TLP2310, U8 74AHC1G125, Y1 ABM8-272-T3

Commit message: finish assignment
Parts:
- U8: value 74AHC1G125 -> 74AHC1G125DCKR; footprint (none) -> Package_TO_SOT_SMD:SOT-353_SC-70-5
Changed lines of the file:
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@@
 		(fields_autoplaced yes)
 		(property "Reference" "U8"
-			(at 264.16 304.7298 0)
+			(at 266.7 304.7298 0)
 			(show_name no)
 			(do_not_autoplace no)
@@
 			)
 		)
-		(property "Value" "74AHC1G125"
-			(at 264.16 307.2698 0)
+		(property "Value" "74AHC1G125DCKR"
+			(at 266.7 307.2698 0)
 			(show_name no)
 			(do_not_autoplace no)
@@
 			)
 		)
-		(property "Footprint" ""
+		(property "Footprint" "Package_TO_SOT_SMD:SOT-353_SC-70-5"
 			(at 251.46 311.15 0)
 			(hide yes)

Commit message: connecting main
Connections:
- net FUSE_ILM: now reaches U2.58 (GPIO47_ADC7)
Changed lines of the file:
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@@
+	(wire
+		(pts
+			(xy 179.07 200.66) (xy 187.96 200.66)
+		)
+		(stroke
+			(width 0)
+			(type default)
+		)
+	)
 	(wire
 		(pts
@@
 		)
 	)
+	(hierarchical_label "FUSE_ILM"
+		(shape input)
+		(at 187.96 200.66 0)
+		(effects
+			(font
+				(size 1.27 1.27)
+			)
+			(justify left)
+		)
+	)

Commit message: cleanup paper
Parts:
- removed J2: SM03B-SRSS-TB, Connector_JST:JST_SH_SM03B-SRSS-TB_1x03-1MP_P1.00mm_Horizontal, symbol Connector_Generic_MountingPin:Conn_01x03_MountingPin
Other:
- note removed: "JST Debug Connector"

Commit message: LeMatrix
Connections:
- net GPIO2 is gone; now on net ENC1_SW: U2.79 (GPIO2)
- net GPIO3 is gone; now on net ENC2_SW: U2.80 (GPIO3)
- net ENC1_A: now also U2.3 (GPIO6); no longer U2.23 (GPIO23)
- net ENC1_B: now also U2.4 (GPIO7); no longer U2.25 (GPIO24)
- net ENC1_SW: no longer U2.39 (GPIO31)
- net ENC2_A: now also U2.6 (GPIO8); no longer U2.26 (GPIO25)
- net ENC2_B: now also U2.7 (GPIO9); no longer U2.27 (GPIO26)
- net ENC2_SW: no longer U2.40 (GPIO32)
- net ENC3_A: now also U2.43 (GPIO34); no longer U2.28 (GPIO27)
- net ENC3_B: now also U2.44 (GPIO35); no longer U2.36 (GPIO28)
- net ENC3_SW: now also U2.47 (GPIO38); no longer U2.42 (GPIO33)
- net ENC4_A: now also U2.45 (GPIO36); no longer U2.37 (GPIO29)
- net ENC4_B: now also U2.46 (GPIO37); no longer U2.38 (GPIO30)
- net ENC4_SW: now also U2.48 (GPIO39); no longer U2.43 (GPIO34)
- net JOYSTICK_SW: now also U2.8 (GPIO10); no longer U2.44 (GPIO35)
- net JOYSTICK_X: now also U2.56 (GPIO45_ADC5); no longer U2.49 (GPIO40_ADC0)
- net JOYSTICK_Y: now also U2.57 (GPIO46_ADC6); no longer U2.52 (GPIO41_ADC1)
- net MCU_RX: now also U2.77 (GPIO0); no longer U2.1 (GPIO4)
- net MCU_TX: now also U2.78 (GPIO1); no longer U2.2 (GPIO5)
- net MIDI_RX: now also U2.2 (GPIO5); no longer U2.78 (GPIO1)
- net MIDI_TX: now also U2.1 (GPIO4); no longer U2.77 (GPIO0)
- net matrix_C0: now also U2.40 (GPIO32); no longer U2.7 (GPIO9)
- net matrix_C1: now also U2.39 (GPIO31); no longer U2.8 (GPIO10)
- net matrix_C10: now also U2.22 (GPIO22); no longer U2.19 (GPIO19)
- net matrix_C11: now also U2.21 (GPIO21); no longer U2.20 (GPIO20)
- net matrix_C12: now also U2.20 (GPIO20); no longer U2.21 (GPIO21)
- net matrix_C13: now also U2.19 (GPIO19); no longer U2.22 (GPIO22)
- net matrix_C2: now also U2.38 (GPIO30); no longer U2.9 (GPIO11)
- net matrix_C3: now also U2.37 (GPIO29); no longer U2.11 (GPIO12)
- net matrix_C4: now also U2.36 (GPIO28); no longer U2.12 (GPIO13)
- net matrix_C5: now also U2.28 (GPIO27); no longer U2.13 (GPIO14)
- net matrix_C6: now also U2.27 (GPIO26); no longer U2.14 (GPIO15)
- net matrix_C7: now also U2.26 (GPIO25); no longer U2.16 (GPIO16)
- net matrix_C8: now also U2.25 (GPIO24); no longer U2.17 (GPIO17)
- net matrix_C9: now also U2.23 (GPIO23); no longer U2.18 (GPIO18)
- net matrix_R0: now also U2.16 (GPIO16); no longer U2.3 (GPIO6)
- net matrix_R1: now also U2.17 (GPIO17); no longer U2.4 (GPIO7)
- net matrix_R2: now also U2.18 (GPIO18); no longer U2.6 (GPIO8)

Commit message: reannoation with good linkage?
Parts:
- renumbered C6 to C301, C9 to C302, C10 to C303, C11 to C304, C12 to C305, C13 to C306, C14 to C307, C15 to C308, C16 to C309, C17 to C310, C18 to C311, C19 to C312, C50 to C313, C8 to C314, C3 to C315, C5 to C316, C51 to C317, C52 to C318, C53 to C319, C54 to C320, C55 to C321, C56 to C322, C57 to C323, C58 to C324, C1 to C325, C2 to C326, C59 to C327, D42 to D301, ENC1 to ENC301, ENC2 to ENC302, ENC3 to ENC303, ENC4 to ENC304, J3 to J301, J4 to J302, L1 to L301, R3 to R301, R10 to R302, R12 to R303, R14 to R304, R16 to R305, R18 to R306, R20 to R307, R22 to R308, R24 to R309, R11 to R310, R13 to R311, R15 to R312, R17 to R313, R19 to R314, R21 to R315, R23 to R316, R25 to R317, R2 to R318, R26 to R319, R28 to R320, R27 to R321, U2 to U301, U4 to U302, U7 to U303, U8 to U304, Y1 to Y301

Commit message: big routing board
Connections:
- net ENC1_A: now also U301.44 (GPIO35); no longer U301.3 (GPIO6)
- net ENC1_B: now also U301.45 (GPIO36); no longer U301.4 (GPIO7)
- net ENC1_SW: now also U301.42 (GPIO33); no longer U301.79 (GPIO2)
- net ENC2_A: now also U301.46 (GPIO37); no longer U301.6 (GPIO8)
- net ENC2_B: now also U301.47 (GPIO38); no longer U301.7 (GPIO9)
- net ENC2_SW: now also U301.43 (GPIO34); no longer U301.80 (GPIO3)
- net ENC3_A: now also U301.3 (GPIO6); no longer U301.43 (GPIO34)
- net ENC3_B: now also U301.4 (GPIO7); no longer U301.44 (GPIO35)
- net ENC3_SW: now also U301.79 (GPIO2); no longer U301.47 (GPIO38)
- net ENC4_A: now also U301.6 (GPIO8); no longer U301.45 (GPIO36)
- net ENC4_B: now also U301.7 (GPIO9); no longer U301.46 (GPIO37)
- net ENC4_SW: now also U301.80 (GPIO3); no longer U301.48 (GPIO39)
- net JOYSTICK_X: now also U301.52 (GPIO41_ADC1); no longer U301.56 (GPIO45_ADC5)
- net JOYSTICK_Y: now also U301.53 (GPIO42_ADC2); no longer U301.57 (GPIO46_ADC6)

Commit message: loose ends
Connections:
- net FUSE_ILM: now also U301.52 (GPIO41_ADC1); no longer U301.58 (GPIO47_ADC7)
- net JOYSTICK_X: now also U301.58 (GPIO47_ADC7); no longer U301.52 (GPIO41_ADC1)
- net JOYSTICK_Y: now also U301.57 (GPIO46_ADC6); no longer U301.53 (GPIO42_ADC2)
Changed lines of the file:
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@@
 	(wire
 		(pts
-			(xy 179.07 187.96) (xy 194.31 187.96)
-		)
-		(stroke
-			(width 0)
-			(type default)
-		)
-	)
-	(wire
-		(pts
 			(xy 260.35 262.89) (xy 261.62 262.89)
 		)
@@
 	(wire
 		(pts
+			(xy 179.07 200.66) (xy 194.31 200.66)
+		)
+		(stroke
+			(width 0)
+			(type default)
+		)
+	)
+	(wire
+		(pts
 			(xy 172.72 29.21) (xy 172.72 27.94)
 		)
@@
 	(wire
 		(pts
+			(xy 179.07 185.42) (xy 187.96 185.42)
+		)
+		(stroke
+			(width 0)
+			(type default)
+		)
+	)
+	(wire
+		(pts
 			(xy 227.33 510.54) (xy 242.57 510.54)
 		)
@@
 	(wire
 		(pts
-			(xy 179.07 185.42) (xy 194.31 185.42)
-		)
-		(stroke
-			(width 0)
-			(type default)
-		)
-	)
-	(wire
-		(pts
 			(xy 378.46 107.95) (xy 368.3 107.95)
 		)
@@
 	(wire
 		(pts
+			(xy 179.07 198.12) (xy 194.31 198.12)
+		)
+		(stroke
+			(width 0)
+			(type default)
+		)
+	)
+	(wire
+		(pts
 			(xy 384.81 80.01) (xy 384.81 83.82)
 		)
@@
 	(wire
 		(pts
-			(xy 179.07 200.66) (xy 187.96 200.66)
-		)
-		(stroke
-			(width 0)
-			(type default)
-		)
-	)
-	(wire
-		(pts
 			(xy 218.44 39.37) (xy 207.01 39.37)
 		)
@@
 		)
 	)
+	(label "JOYSTICK_X"
+		(at 194.31 200.66 180)
+		(effects
+			(font
+				(size 1.27 1.27)
+			)
+			(justify right bottom)
+		)
+	)
 	(label "ENC4_SW"
 		(at 421.64 80.01 180)
@@
 		)
 	)
-	(label "JOYSTICK_Y"
-		(at 194.31 187.96 180)
-		(effects
-			(font
-				(size 1.27 1.27)
-			)
-			(justify right bottom)
-		)
-	)
 	(label "QSPI_SCLK"
 		(at 96.52 105.41 0)
@@
 		)
 	)
+	(label "JOYSTICK_Y"
+		(at 194.31 198.12 180)
+		(effects
+			(font
+				(size 1.27 1.27)
+			)
+			(justify right bottom)
+		)
+	)
 	(label "ENC2_A"
 		(at 284.48 107.95 0)
@@
 		)
 	)
-	(label "JOYSTICK_X"
-		(at 194.31 185.42 180)
-		(effects
-			(font
-				(size 1.27 1.27)
-			)
-			(justify right bottom)
-		)
-	)
 	(label "ENC1_A"
 		(at 236.22 107.95 0)
@@
 	(hierarchical_label "FUSE_ILM"
 		(shape input)
-		(at 187.96 200.66 0)
+		(at 187.96 185.42 0)
 		(effects
 			(font

Commit message: wire encoder sw 3/4 and some cleanup
Connections:
- net ENC3_SW: now also U301.9 (GPIO11); no longer U301.79 (GPIO2)
- net ENC4_SW: now also U301.11 (GPIO12); no longer U301.80 (GPIO3)
Changed lines of the file:
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@@
 	(wire
 		(pts
-			(xy 179.07 86.36) (xy 194.31 86.36)
-		)
-		(stroke
-			(width 0)
-			(type default)
-		)
-	)
-	(wire
-		(pts
 			(xy 342.9 99.06) (xy 353.06 99.06)
 		)
@@
 	(wire
 		(pts
+			(xy 179.07 109.22) (xy 194.31 109.22)
+		)
+		(stroke
+			(width 0)
+			(type default)
+		)
+	)
+	(wire
+		(pts
 			(xy 179.07 101.6) (xy 194.31 101.6)
 		)
@@
 	(wire
 		(pts
+			(xy 179.07 106.68) (xy 194.31 106.68)
+		)
+		(stroke
+			(width 0)
+			(type default)
+		)
+	)
+	(wire
+		(pts
 			(xy 406.4 83.82) (xy 406.4 80.01)
 		)
@@
 	(wire
 		(pts
-			(xy 179.07 83.82) (xy 194.31 83.82)
-		)
-		(stroke
-			(width 0)
-			(type default)
-		)
-	)
-	(wire
-		(pts
 			(xy 287.02 175.26) (xy 300.99 175.26)
 		)
@@
 		)
 	)
-	(label "ENC4_SW"
-		(at 194.31 86.36 180)
+	(label "ENC3_SW"
+		(at 194.31 106.68 180)
 		(effects
 			(font
@@
 		)
 	)
+	(label "ENC4_SW"
+		(at 194.31 109.22 180)
+		(effects
+			(font
+				(size 1.27 1.27)
+			)
+			(justify right bottom)
+		)
+	)
 	(label "JOYSTICK_SW"
 		(at 194.31 104.14 180)
@@
 		(effects
 			(font
-				(size 1.27 1.27)
-			)
-			(justify right bottom)
-		)
-	)
-	(label "ENC3_SW"
-		(at 194.31 83.82 180)
-		(effects
-			(font
