File: hardware/board/board.kicad_pcb (KiCad board)
At the start: 2 copper layers, 300 x 120 mm, 192 parts, among them J1 USB_B_Micro, J2 SM03B-SRSS-TB, J3 MidiIn, J4 MidiOut, J5 LineIn, J6 LineOut, J7 Headphone, SW1 SW_Push, SW10 SW_Push, SW11 SW_Push, SW12 SW_Push, SW13 SW_Push, SW14 SW_Push, SW15 SW_Push, SW16 SW_Push, SW17 SW_Push, SW18 SW_Push, SW19 SW_Push, SW2 SW_Push, SW20 SW_Push, SW21 SW_Push, SW22 SW_Push, SW23 SW_Push, SW24 SW_Push, SW25 SW_Push, SW26 SW_Push, SW27 SW_Push, SW28 SW_Push, SW29 SW_Push, SW3 SW_Push, SW30 SW_Push, SW31 SW_Push, SW32 SW_Push, SW33 SW_Push, SW34 SW_Push, SW35 SW_Push, SW36 SW_Push, SW37 SW_Push, SW38 SW_Push, SW39 SW_Push, SW4 SW_Push, SW40 SW_Push, SW41 SW_Push, SW42 SW_Push, SW43 SW_Push, SW5 SW_Push, SW6 SW_Push, SW7 SW_Push, SW8 SW_Push, SW9 SW_Push, U1 NCP1117-3.3_SOT223, U2 RP2350_80QFN, U3 Oled, U4 CNK_THB001P, U5 TPS7A20xxxDBV, U6 QFN40P700X700X80-57N, Y1 ABM8-272-T3, Y2 12.288MHz

Commit message: usb c footprint
Parts:
- added P1: USB_C_Plug_USB2.0, Connector_USB:USB_C_Receptacle_HRO_TYPE-C-31-M-12, B.Cu at (137.5, 88.0)
- added P2: USB_C_Plug_USB2.0, Connector_USB:USB_C_Receptacle_HRO_TYPE-C-31-M-12, B.Cu at (157.5, 88.0)
- U4: value CNK_THB001P -> THB001P
- U6: value QFN40P700X700X80-57N -> MAX98089ETN_T
- moved J4 62.0 mm to (257.5, 88.0)
- moved J3 55.5 mm to (277.5, 88.0)
- moved J6 49.0 mm to (297.5, 88.0)
- moved J5 42.8 mm to (317.5, 88.0)
- turned ENC1 to 90 degrees
- turned ENC2 to 90 degrees
- turned ENC3 to 90 degrees
- turned ENC4 to 90 degrees

Commit message: more placement
Parts:
- removed SW42, SW43: SW_Push, ledaw:ks-33-2.0
- added C50: 10u, Capacitor_SMD:C_0805_2012Metric, F.Cu at (60.0, 255.0)
- added REF**: bf-32-s-8ohm, ledaw:bf-32-s-8ohm, F.Cu at (347.5, 103.5)
- added REF**: bf-32-s-8ohm, ledaw:bf-32-s-8ohm, F.Cu at (87.5, 103.5)
- added SW101: SW_Push, Button_Switch_SMD:SW_Push_1P1T_NO_Vertical_Wuerth_434133025816, F.Cu at (54.4, 255.9)
- added SW102: SW_Push, Button_Switch_SMD:SW_Push_1P1T_NO_Vertical_Wuerth_434133025816, F.Cu at (54.4, 260.6)
- MK1, MK2: moved to B.Cu
- SW1, SW2: footprint Button_Switch_SMD:SW_Push_1P1T_NO_Vertical_Wuerth_434133025816 -> ledaw:ks-33-2.0
- moved MK2 383.6 mm to (287.5, 103.5), turned to 180 degrees
- moved MK1 318.6 mm to (147.5, 103.5), turned to 180 degrees
- moved SW14 230.9 mm to (337.5, 133.5)
- moved LS1 209.5 mm to (149.0, 214.1)
- moved LS2 209.5 mm to (149.0, 226.0)
- moved SW41 200.0 mm to (357.5, 183.5)
- moved SW19 192.4 mm to (127.5, 153.5)
- moved SW27 191.0 mm to (347.5, 153.5)
- moved SW28 186.8 mm to (97.5, 183.5)
- moved SW16 164.9 mm to (77.5, 173.5)
- moved SW26 160.0 mm to (327.5, 153.5)
- moved SW23 153.0 mm to (247.5, 153.5)
- moved SW32 153.0 mm to (177.5, 183.5)
- moved SW8 148.7 mm to (217.5, 133.5)
- moved SW2 141.8 mm to (97.5, 133.5)
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Connections:
- D10 pad 1: /mcu/buttons/matrix_C1 -> /mcu/buttons/matrix_C9
- D11 pad 1: /mcu/buttons/matrix_C1 -> /mcu/buttons/matrix_C10
- D12 pad 1: /mcu/buttons/matrix_C1 -> /mcu/buttons/matrix_C11
- D13 pad 1: /mcu/buttons/matrix_C2 -> /mcu/buttons/matrix_C12
- D14 pad 1: /mcu/buttons/matrix_C2 -> /mcu/buttons/matrix_C13
- D15 pad 1: /mcu/buttons/matrix_C2 -> /mcu/buttons/matrix_C0
- D16 pad 1: /mcu/buttons/matrix_C2 -> /mcu/buttons/matrix_C1
- D18 pad 1: /mcu/buttons/matrix_C2 -> /mcu/buttons/matrix_C3
- D19 pad 1: /mcu/buttons/matrix_C3 -> /mcu/buttons/matrix_C4
- D2 pad 1: /mcu/buttons/matrix_C0 -> /mcu/buttons/matrix_C1
- D20 pad 1: /mcu/buttons/matrix_C3 -> /mcu/buttons/matrix_C5
- D21 pad 1: /mcu/buttons/matrix_C3 -> /mcu/buttons/matrix_C6
- D22 pad 1: /mcu/buttons/matrix_C3 -> /mcu/buttons/matrix_C7
- D23 pad 1: /mcu/buttons/matrix_C3 -> /mcu/buttons/matrix_C8
- D24 pad 1: /mcu/buttons/matrix_C3 -> /mcu/buttons/matrix_C9
- D25 pad 1: /mcu/buttons/matrix_C4 -> /mcu/buttons/matrix_C10
- D26 pad 1: /mcu/buttons/matrix_C4 -> /mcu/buttons/matrix_C11
- D27 pad 1: /mcu/buttons/matrix_C4 -> /mcu/buttons/matrix_C12
- D28 pad 1: /mcu/buttons/matrix_C4 -> /mcu/buttons/matrix_C0
- D29 pad 1: /mcu/buttons/matrix_C4 -> /mcu/buttons/matrix_C1
- D3 pad 1: /mcu/buttons/matrix_C0 -> /mcu/buttons/matrix_C2
- D30 pad 1: /mcu/buttons/matrix_C4 -> /mcu/buttons/matrix_C2
- D31 pad 1: /mcu/buttons/matrix_C5 -> /mcu/buttons/matrix_C3
- D32 pad 1: /mcu/buttons/matrix_C5 -> /mcu/buttons/matrix_C4
- D34 pad 1: /mcu/buttons/matrix_C5 -> /mcu/buttons/matrix_C6
- D35 pad 1: /mcu/buttons/matrix_C5 -> /mcu/buttons/matrix_C7
- D36 pad 1: /mcu/buttons/matrix_C5 -> /mcu/buttons/matrix_C8
- D37 pad 1: /mcu/buttons/matrix_C6 -> /mcu/buttons/matrix_C9
- D38 pad 1: /mcu/buttons/matrix_C6 -> /mcu/buttons/matrix_C10
- D39 pad 1: /mcu/buttons/matrix_C6 -> /mcu/buttons/matrix_C11
- D4 pad 1: /mcu/buttons/matrix_C0 -> /mcu/buttons/matrix_C3
- D40 pad 1: /mcu/buttons/matrix_C6 -> /mcu/buttons/matrix_C12
- D41 pad 1: /mcu/buttons/matrix_C6 -> /mcu/buttons/matrix_C13
- D5 pad 1: /mcu/buttons/matrix_C0 -> /mcu/buttons/matrix_C4
- D6 pad 1: /mcu/buttons/matrix_C0 -> /mcu/buttons/matrix_C5
- D7 pad 1: /mcu/buttons/matrix_C1 -> /mcu/buttons/matrix_C6
- D8 pad 1: /mcu/buttons/matrix_C1 -> /mcu/buttons/matrix_C7
- D9 pad 1: /mcu/buttons/matrix_C1 -> /mcu/buttons/matrix_C8
- SW1 pad 1: GND -> /mcu/buttons/matrix_R0
- SW1 pad 2: /mcu/~{USB_BOOT} -> Net-(D1-A)
- SW10 pad 1: /mcu/buttons/matrix_R1 -> /mcu/buttons/matrix_R0
- SW10 pad 2: Net-(D8-A) -> Net-(D10-A)
- SW11 pad 1: /mcu/buttons/matrix_R2 -> /mcu/buttons/matrix_R0
- SW11 pad 2: Net-(D9-A) -> Net-(D11-A)
- SW12 pad 1: /mcu/buttons/matrix_R3 -> /mcu/buttons/matrix_R0
- SW12 pad 2: Net-(D10-A) -> Net-(D12-A)
- SW13 pad 1: /mcu/buttons/matrix_R4 -> /mcu/buttons/matrix_R0
- SW13 pad 2: Net-(D11-A) -> Net-(D13-A)
- SW14 pad 1: /mcu/buttons/matrix_C6 -> /mcu/buttons/matrix_R0
- SW14 pad 2: Net-(D12-A) -> Net-(D14-A)
- SW15 pad 1: /mcu/buttons/matrix_R0 -> (no net)
- SW15 pad 2: Net-(D13-A) -> (no net)
- SW16 pad 1: /mcu/buttons/matrix_R1 -> (no net)
- SW16 pad 2: Net-(D14-A) -> (no net)
- SW17 pad 1: /mcu/buttons/matrix_R2 -> /mcu/buttons/matrix_R1
- SW17 pad 2: Net-(D15-A) -> Net-(D17-A)
- SW18 pad 1: /mcu/buttons/matrix_R3 -> (no net)
- SW18 pad 2: Net-(D16-A) -> (no net)
- SW19 pad 1: /mcu/buttons/matrix_R4 -> (no net)
- SW19 pad 2: Net-(D17-A) -> (no net)
- SW2 pad 1: Net-(R1-Pad1) -> /mcu/buttons/matrix_R0
- SW2 pad 2: /mcu/RUN -> Net-(D2-A)
- SW20 pad 1: /mcu/buttons/matrix_C6 -> /mcu/buttons/matrix_R1
- SW20 pad 2: Net-(D18-A) -> Net-(D20-A)
- SW21 pad 1: /mcu/buttons/matrix_R0 -> /mcu/buttons/matrix_R1
- SW21 pad 2: Net-(D19-A) -> Net-(D21-A)
- SW22 pad 2: Net-(D20-A) -> Net-(D22-A)
- SW23 pad 1: /mcu/buttons/matrix_R2 -> /mcu/buttons/matrix_R1
- SW23 pad 2: Net-(D21-A) -> Net-(D23-A)
- SW24 pad 1: /mcu/buttons/matrix_R3 -> /mcu/buttons/matrix_R1
- SW24 pad 2: Net-(D22-A) -> Net-(D24-A)
- SW25 pad 1: /mcu/buttons/matrix_R4 -> /mcu/buttons/matrix_R1
- SW25 pad 2: Net-(D23-A) -> Net-(D25-A)
- SW26 pad 1: /mcu/buttons/matrix_C6 -> /mcu/buttons/matrix_R1
- SW26 pad 2: Net-(D24-A) -> Net-(D26-A)
- SW27 pad 1: /mcu/buttons/matrix_R0 -> /mcu/buttons/matrix_R1
- SW27 pad 2: Net-(D25-A) -> Net-(D27-A)
- SW28 pad 1: /mcu/buttons/matrix_R1 -> /mcu/buttons/matrix_R2
- SW28 pad 2: Net-(D26-A) -> Net-(D28-A)
- SW29 pad 2: Net-(D27-A) -> Net-(D29-A)
- SW3 pad 2: Net-(D1-A) -> Net-(D3-A)
- SW30 pad 1: /mcu/buttons/matrix_R3 -> /mcu/buttons/matrix_R2
- SW30 pad 2: Net-(D28-A) -> Net-(D30-A)
- SW31 pad 1: /mcu/buttons/matrix_R4 -> /mcu/buttons/matrix_R2
- SW31 pad 2: Net-(D29-A) -> Net-(D31-A)
- SW32 pad 1: /mcu/buttons/matrix_C6 -> (no net)
- SW32 pad 2: Net-(D30-A) -> (no net)
- SW33 pad 1: /mcu/buttons/matrix_R0 -> (no net)
- SW33 pad 2: Net-(D31-A) -> (no net)
- SW34 pad 1: /mcu/buttons/matrix_R1 -> /mcu/buttons/matrix_R2
- SW34 pad 2: Net-(D32-A) -> Net-(D34-A)
- SW35 pad 2: Net-(D33-A) -> Net-(D35-A)
- SW36 pad 1: /mcu/buttons/matrix_R3 -> /mcu/buttons/matrix_R2
- SW36 pad 2: Net-(D34-A) -> Net-(D36-A)
- SW37 pad 1: /mcu/buttons/matrix_R4 -> (no net)
- SW37 pad 2: Net-(D35-A) -> (no net)
- SW38 pad 1: /mcu/buttons/matrix_C6 -> /mcu/buttons/matrix_R2
- SW38 pad 2: Net-(D36-A) -> Net-(D38-A)
- SW39 pad 1: /mcu/buttons/matrix_R0 -> /mcu/buttons/matrix_R2
- SW39 pad 2: Net-(D37-A) -> Net-(D39-A)
- SW4 pad 1: /mcu/buttons/matrix_R1 -> /mcu/buttons/matrix_R0
- SW4 pad 2: Net-(D2-A) -> Net-(D4-A)
- SW40 pad 1: /mcu/buttons/matrix_R1 -> /mcu/buttons/matrix_R2
- SW40 pad 2: Net-(D38-A) -> Net-(D40-A)
- SW41 pad 2: Net-(D39-A) -> Net-(D41-A)
- SW5 pad 1: /mcu/buttons/matrix_R2 -> /mcu/buttons/matrix_R0
- SW5 pad 2: Net-(D3-A) -> Net-(D5-A)
- SW6 pad 1: /mcu/buttons/matrix_R3 -> /mcu/buttons/matrix_R0
- SW6 pad 2: Net-(D4-A) -> Net-(D6-A)
- SW7 pad 1: /mcu/buttons/matrix_R4 -> /mcu/buttons/matrix_R0
- SW7 pad 2: Net-(D5-A) -> Net-(D7-A)
- SW8 pad 1: /mcu/buttons/matrix_C6 -> /mcu/buttons/matrix_R0
- SW8 pad 2: Net-(D6-A) -> Net-(D8-A)
- SW9 pad 2: Net-(D7-A) -> Net-(D9-A)

Commit message: rp2350 pdf
Parts:
- D1, D10, D11, D12, D13, D14, D15, D16, D17, D18, D19, D2, D20, D21, D22, D23, D24, D25, D26, D27, D28, D29, D30, D31, D32, D33, D34, D35, D36, D37, D38, D39, D40, D41, D5, D6, D7, D8, D9: moved to F.Cu
- LS1, LS2: moved to B.Cu
- moved TP10 58.8 mm to (80.7, 395.6)
- moved TP11 58.8 mm to (80.7, 399.6)
- moved TP12 58.8 mm to (80.7, 403.7)
- moved TP13 58.8 mm to (84.8, 383.4)
- moved TP14 58.8 mm to (84.8, 387.5)
- moved TP15 58.8 mm to (84.8, 391.5)
- moved TP16 58.8 mm to (84.8, 395.6)
- moved TP18 58.8 mm to (84.8, 403.7)
- moved TP7 58.8 mm to (80.7, 383.4)
- moved TP8 58.8 mm to (80.7, 387.5)
- moved TP9 58.8 mm to (80.7, 391.5)
- moved TP1 58.8 mm to (76.7, 383.4)
- moved TP2 58.8 mm to (76.7, 387.5)
- moved TP3 58.8 mm to (76.7, 391.5)
- moved TP4 58.8 mm to (76.7, 395.6)
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
Commit message: efuse
Parts:
- added C51: 10nF, Capacitor_SMD:C_0805_2012Metric, F.Cu at (6.46, 387.5)
- added C52: 10nF, Capacitor_SMD:C_0805_2012Metric, F.Cu at (6.46, 390.5)
- added C53: 10nF, Capacitor_SMD:C_0805_2012Metric, F.Cu at (6.46, 393.5)
- added C54: 10nF, Capacitor_SMD:C_0805_2012Metric, F.Cu at (10.9, 387.5)
- added C55: 10nF, Capacitor_SMD:C_0805_2012Metric, F.Cu at (10.9, 390.5)
- added C56: 10nF, Capacitor_SMD:C_0805_2012Metric, F.Cu at (10.9, 393.5)
- added C57: 10nF, Capacitor_SMD:C_0805_2012Metric, F.Cu at (15.4, 387.5)
- added C58: 10nF, Capacitor_SMD:C_0805_2012Metric, F.Cu at (15.4, 390.5)
- added C59: 100nF, Capacitor_SMD:C_0805_2012Metric, F.Cu at (15.4, 393.5)
- added D42: LL4148, Diode_SMD:D_MiniMELF, F.Cu at (7.45, 401.9)
- added R10: 10k, Resistor_SMD:R_0805_2012Metric, F.Cu at (-6.79, 387.5)
- added R11: 10k, Resistor_SMD:R_0805_2012Metric, F.Cu at (-6.79, 390.4)
- added R12: 10k, Resistor_SMD:R_0805_2012Metric, F.Cu at (-6.79, 393.4)
- added R13: 10k, Resistor_SMD:R_0805_2012Metric, F.Cu at (-6.79, 396.3)
- added R14: 10k, Resistor_SMD:R_0805_2012Metric, F.Cu at (-6.79, 399.3)
- added R15: 10k, Resistor_SMD:R_0805_2012Metric, F.Cu at (-6.79, 402.2)
- added R16: 10k, Resistor_SMD:R_0805_2012Metric, F.Cu at (-6.79, 405.2)
- added R17: 10k, Resistor_SMD:R_0805_2012Metric, F.Cu at (-2.38, 387.5)
- added R18: 10k, Resistor_SMD:R_0805_2012Metric, F.Cu at (-2.38, 390.4)
- added R19: 10k, Resistor_SMD:R_0805_2012Metric, F.Cu at (-2.38, 393.4)
- added R20: 10k, Resistor_SMD:R_0805_2012Metric, F.Cu at (-2.38, 396.3)
- added R21: 10k, Resistor_SMD:R_0805_2012Metric, F.Cu at (-2.38, 399.3)
- added R22: 10k, Resistor_SMD:R_0805_2012Metric, F.Cu at (-2.38, 402.2)
- added R23: 10k, Resistor_SMD:R_0805_2012Metric, F.Cu at (-2.38, 405.2)
- added R24: 10k, Resistor_SMD:R_0805_2012Metric, F.Cu at (2.02, 387.5)
- added R25: 10k, Resistor_SMD:R_0805_2012Metric, F.Cu at (2.02, 390.4)
- added R26: 220, Resistor_SMD:R_0805_2012Metric, F.Cu at (2.02, 393.4)
- added R27: 10, Resistor_SMD:R_0805_2012Metric, F.Cu at (2.02, 396.3)
- added R28: 33, Resistor_SMD:R_0805_2012Metric, F.Cu at (2.02, 399.3)
- added U7: TLP2310, Package_SO:SO-5-6_4.55x3.7mm_P1.27mm, F.Cu at (8.76, 397.7)
Connections:
- net /mcu/GPIO0 renamed /mcu/MIDI_TX
- net /mcu/GPIO4 renamed /mcu/CM4_TX
- net /mcu/GPIO5 renamed /mcu/CM5_TX
- D1 pad 1: /mcu/buttons/matrix_C0 -> /mcu/matrix_C0
- D10 pad 1: /mcu/buttons/matrix_C9 -> /mcu/matrix_C9
- D11 pad 1: /mcu/buttons/matrix_C10 -> /mcu/matrix_C10
- D12 pad 1: /mcu/buttons/matrix_C11 -> /mcu/matrix_C11
- D13 pad 1: /mcu/buttons/matrix_C12 -> /mcu/matrix_C12
- D14 pad 1: /mcu/buttons/matrix_C13 -> /mcu/matrix_C13
- D15 pad 1: /mcu/buttons/matrix_C0 -> /mcu/matrix_C0
- D16 pad 1: /mcu/buttons/matrix_C1 -> /mcu/matrix_C1
- D17 pad 1: /mcu/buttons/matrix_C2 -> /mcu/matrix_C2
- D18 pad 1: /mcu/buttons/matrix_C3 -> /mcu/matrix_C3
- D19 pad 1: /mcu/buttons/matrix_C4 -> /mcu/matrix_C4
- D2 pad 1: /mcu/buttons/matrix_C1 -> /mcu/matrix_C1
- D20 pad 1: /mcu/buttons/matrix_C5 -> /mcu/matrix_C5
- D21 pad 1: /mcu/buttons/matrix_C6 -> /mcu/matrix_C6
- D22 pad 1: /mcu/buttons/matrix_C7 -> /mcu/matrix_C7
- D23 pad 1: /mcu/buttons/matrix_C8 -> /mcu/matrix_C8
- D24 pad 1: /mcu/buttons/matrix_C9 -> /mcu/matrix_C9
- D25 pad 1: /mcu/buttons/matrix_C10 -> /mcu/matrix_C10
- D26 pad 1: /mcu/buttons/matrix_C11 -> /mcu/matrix_C11
- D27 pad 1: /mcu/buttons/matrix_C12 -> /mcu/matrix_C12
- D28 pad 1: /mcu/buttons/matrix_C0 -> /mcu/matrix_C0
- D29 pad 1: /mcu/buttons/matrix_C1 -> /mcu/matrix_C1
- D3 pad 1: /mcu/buttons/matrix_C2 -> /mcu/matrix_C2
- D30 pad 1: /mcu/buttons/matrix_C2 -> /mcu/matrix_C2
- D31 pad 1: /mcu/buttons/matrix_C3 -> /mcu/matrix_C3
- D32 pad 1: /mcu/buttons/matrix_C4 -> /mcu/matrix_C4
- D33 pad 1: /mcu/buttons/matrix_C5 -> /mcu/matrix_C5
- D34 pad 1: /mcu/buttons/matrix_C6 -> /mcu/matrix_C6
- D35 pad 1: /mcu/buttons/matrix_C7 -> /mcu/matrix_C7
- D36 pad 1: /mcu/buttons/matrix_C8 -> /mcu/matrix_C8
- D37 pad 1: /mcu/buttons/matrix_C9 -> /mcu/matrix_C9
- D38 pad 1: /mcu/buttons/matrix_C10 -> /mcu/matrix_C10
- D39 pad 1: /mcu/buttons/matrix_C11 -> /mcu/matrix_C11
- D4 pad 1: /mcu/buttons/matrix_C3 -> /mcu/matrix_C3
- D40 pad 1: /mcu/buttons/matrix_C12 -> /mcu/matrix_C12
- D41 pad 1: /mcu/buttons/matrix_C13 -> /mcu/matrix_C13
- D5 pad 1: /mcu/buttons/matrix_C4 -> /mcu/matrix_C4
- D6 pad 1: /mcu/buttons/matrix_C5 -> /mcu/matrix_C5
- D7 pad 1: /mcu/buttons/matrix_C6 -> /mcu/matrix_C6
- D8 pad 1: /mcu/buttons/matrix_C7 -> /mcu/matrix_C7
- D9 pad 1: /mcu/buttons/matrix_C8 -> /mcu/matrix_C8
- ENC1 pad A: unconnected-(ENC1-PadA) -> Net-(ENC1-PadA)
- ENC1 pad B: unconnected-(ENC1-PadB) -> Net-(ENC1-PadB)
- ENC1 pad C: unconnected-(ENC1-PadC) -> GND
- ENC1 pad S1: unconnected-(ENC1-PadS1) -> GND
- ENC1 pad S2: unconnected-(ENC1-PadS2) -> /mcu/ENC1_SW
- ENC2 pad A: unconnected-(ENC2-PadA) -> Net-(ENC2-PadA)
- ENC2 pad B: unconnected-(ENC2-PadB) -> Net-(ENC2-PadB)
- ENC2 pad C: unconnected-(ENC2-PadC) -> GND
- ENC2 pad S1: unconnected-(ENC2-PadS1) -> GND
- ENC2 pad S2: unconnected-(ENC2-PadS2) -> /mcu/ENC2_SW
- ENC3 pad A: unconnected-(ENC3-PadA) -> Net-(ENC3-PadA)
- ENC3 pad B: unconnected-(ENC3-PadB) -> Net-(ENC3-PadB)
- ENC3 pad C: unconnected-(ENC3-PadC) -> GND
- ENC3 pad S1: unconnected-(ENC3-PadS1) -> GND
- ENC3 pad S2: unconnected-(ENC3-PadS2) -> /mcu/ENC3_SW
- ENC4 pad A: unconnected-(ENC4-PadA) -> Net-(ENC4-PadA)
- ENC4 pad B: unconnected-(ENC4-PadB) -> Net-(ENC4-PadB)
- ENC4 pad C: unconnected-(ENC4-PadC) -> GND
- ENC4 pad S1: unconnected-(ENC4-PadS1) -> GND
- ENC4 pad S2: unconnected-(ENC4-PadS2) -> /mcu/ENC4_SW
- J3 pad R: unconnected-(J3-PadR) -> Net-(J3-PadR)
- J3 pad S: unconnected-(J3-PadS) -> GND
- J3 pad T: unconnected-(J3-PadT) -> Net-(D42-A)
- J4 pad R: unconnected-(J4-PadR) -> Net-(J4-PadR)
- J4 pad S: unconnected-(J4-PadS) -> GND
- J4 pad T: unconnected-(J4-PadT) -> Net-(J4-PadT)
- Module1 pad 101: (no net) -> unconnected-(Module1B-USB_OTG_ID-Pad101)
- Module1 pad 102: (no net) -> unconnected-(Module1B-PCIe_CLK_nREQ-Pad102)
- Module1 pad 103: (no net) -> unconnected-(Module1B-USB2_N-Pad103)
- Module1 pad 104: (no net) -> unconnected-(Module1B-Reserved-Pad104)
- Module1 pad 105: (no net) -> unconnected-(Module1B-USB2_P-Pad105)
- Module1 pad 106: (no net) -> unconnected-(Module1B-Reserved-Pad106)
- Module1 pad 107: (no net) -> unconnected-(Module1B-GND-Pad107)
- Module1 pad 108: (no net) -> unconnected-(Module1B-GND-Pad108)
- Module1 pad 109: (no net) -> unconnected-(Module1B-PCIe_nRST-Pad109)
- Module1 pad 110: (no net) -> unconnected-(Module1B-PCIe_CLK_P-Pad110)
- Module1 pad 111: (no net) -> unconnected-(Module1B-VDAC_COMP-Pad111)
- Module1 pad 112: (no net) -> unconnected-(Module1B-PCIe_CLK_N-Pad112)
- Module1 pad 113: (no net) -> unconnected-(Module1B-GND-Pad113)
- Module1 pad 114: (no net) -> unconnected-(Module1B-GND-Pad114)
- Module1 pad 115: (no net) -> unconnected-(Module1B-CAM1_D0_N-Pad115)
- Module1 pad 116: (no net) -> unconnected-(Module1B-PCIe_RX_P-Pad116)
- Module1 pad 117: (no net) -> unconnected-(Module1B-CAM1_D0_P-Pad117)
- Module1 pad 118: (no net) -> unconnected-(Module1B-PCIe_RX_N-Pad118)
- Module1 pad 119: (no net) -> unconnected-(Module1B-GND-Pad119)
- Module1 pad 120: (no net) -> unconnected-(Module1B-GND-Pad120)
- Module1 pad 121: (no net) -> unconnected-(Module1B-CAM1_D1_N-Pad121)
- Module1 pad 122: (no net) -> unconnected-(Module1B-PCIe_TX_P-Pad122)
- Module1 pad 123: (no net) -> unconnected-(Module1B-CAM1_D1_P-Pad123)
- Module1 pad 124: (no net) -> unconnected-(Module1B-PCIe_TX_N-Pad124)
- Module1 pad 125: (no net) -> unconnected-(Module1B-GND-Pad125)
- Module1 pad 126: (no net) -> unconnected-(Module1B-GND-Pad126)
- Module1 pad 127: (no net) -> unconnected-(Module1B-CAM1_C_N-Pad127)
- Module1 pad 128: (no net) -> unconnected-(Module1B-CAM0_D0_N-Pad128)
- Module1 pad 129: (no net) -> unconnected-(Module1B-CAM1_C_P-Pad129)
- Module1 pad 130: (no net) -> unconnected-(Module1B-CAM0_D0_P-Pad130)
- Module1 pad 131: (no net) -> unconnected-(Module1B-GND-Pad131)
- Module1 pad 132: (no net) -> unconnected-(Module1B-GND-Pad132)
- Module1 pad 133: (no net) -> unconnected-(Module1B-CAM1_D2_N-Pad133)
- Module1 pad 134: (no net) -> unconnected-(Module1B-CAM0_D1_N-Pad134)
- Module1 pad 135: (no net) -> unconnected-(Module1B-CAM1_D2_P-Pad135)
- Module1 pad 136: (no net) -> unconnected-(Module1B-CAM0_D1_P-Pad136)
- Module1 pad 137: (no net) -> unconnected-(Module1B-GND-Pad137)
- Module1 pad 138: (no net) -> unconnected-(Module1B-GND-Pad138)
- Module1 pad 139: (no net) -> unconnected-(Module1B-CAM1_D3_N-Pad139)
- Module1 pad 140: (no net) -> unconnected-(Module1B-CAM0_C_N-Pad140)
- Module1 pad 141: (no net) -> unconnected-(Module1B-CAM1_D3_P-Pad141)
- Module1 pad 142: (no net) -> unconnected-(Module1B-CAM0_C_P-Pad142)
- Module1 pad 143: (no net) -> unconnected-(Module1B-HDMI1_HOTPLUG-Pad143)
- Module1 pad 144: (no net) -> unconnected-(Module1B-GND-Pad144)
- Module1 pad 145: (no net) -> unconnected-(Module1B-HDMI1_SDA-Pad145)
- Module1 pad 146: (no net) -> unconnected-(Module1B-HDMI1_TX2_P-Pad146)
- Module1 pad 147: (no net) -> unconnected-(Module1B-HDMI1_SCL-Pad147)
- Module1 pad 148: (no net) -> unconnected-(Module1B-HDMI1_TX2_N-Pad148)
- Module1 pad 149: (no net) -> unconnected-(Module1B-HDMI1_CEC-Pad149)
- Module1 pad 150: (no net) -> unconnected-(Module1B-GND-Pad150)
- Module1 pad 151: (no net) -> unconnected-(Module1B-HDMI0_CEC-Pad151)
- Module1 pad 152: (no net) -> unconnected-(Module1B-HDMI1_TX1_P-Pad152)
- Module1 pad 153: (no net) -> unconnected-(Module1B-HDMI0_HOTPLUG-Pad153)
- Module1 pad 154: (no net) -> unconnected-(Module1B-HDMI1_TX1_N-Pad154)
- Module1 pad 155: (no net) -> unconnected-(Module1B-GND-Pad155)
- Module1 pad 156: (no net) -> unconnected-(Module1B-GND-Pad156)
- Module1 pad 157: (no net) -> unconnected-(Module1B-DSI0_D0_N-Pad157)
- Module1 pad 158: (no net) -> unconnected-(Module1B-HDMI1_TX0_P-Pad158)
- Module1 pad 159: (no net) -> unconnected-(Module1B-DSI0_D0_P-Pad159)
- Module1 pad 160: (no net) -> unconnected-(Module1B-HDMI1_TX0_N-Pad160)
- Module1 pad 161: (no net) -> unconnected-(Module1B-GND-Pad161)
- Module1 pad 162: (no net) -> unconnected-(Module1B-GND-Pad162)
- Module1 pad 163: (no net) -> unconnected-(Module1B-DSI0_D1_N-Pad163)
- Module1 pad 164: (no net) -> unconnected-(Module1B-HDMI1_CLK_P-Pad164)
- Module1 pad 165: (no net) -> unconnected-(Module1B-DSI0_D1_P-Pad165)
- Module1 pad 166: (no net) -> unconnected-(Module1B-HDMI1_CLK_N-Pad166)
- Module1 pad 167: (no net) -> unconnected-(Module1B-GND-Pad167)
- Module1 pad 168: (no net) -> unconnected-(Module1B-GND-Pad168)
- Module1 pad 169: (no net) -> unconnected-(Module1B-DSI0_C_N-Pad169)
- Module1 pad 170: (no net) -> unconnected-(Module1B-HDMI0_TX2_P-Pad170)
- Module1 pad 171: (no net) -> unconnected-(Module1B-DSI0_C_P-Pad171)
- Module1 pad 172: (no net) -> unconnected-(Module1B-HDMI0_TX2_N-Pad172)
- Module1 pad 173: (no net) -> unconnected-(Module1B-GND-Pad173)
- Module1 pad 174: (no net) -> unconnected-(Module1B-GND-Pad174)
- Module1 pad 175: (no net) -> unconnected-(Module1B-DSI1_D0_N-Pad175)
- Module1 pad 176: (no net) -> unconnected-(Module1B-HDMI0_TX1_P-Pad176)
- Module1 pad 177: (no net) -> unconnected-(Module1B-DSI1_D0_P-Pad177)
- Module1 pad 178: (no net) -> unconnected-(Module1B-HDMI0_TX1_N-Pad178)
- Module1 pad 179: (no net) -> unconnected-(Module1B-GND-Pad179)
- Module1 pad 180: (no net) -> unconnected-(Module1B-GND-Pad180)
- Module1 pad 181: (no net) -> unconnected-(Module1B-DSI1_D1_N-Pad181)
- Module1 pad 182: (no net) -> unconnected-(Module1B-HDMI0_TX0_P-Pad182)
- Module1 pad 183: (no net) -> unconnected-(Module1B-DSI1_D1_P-Pad183)
- Module1 pad 184: (no net) -> unconnected-(Module1B-HDMI0_TX0_N-Pad184)
- Module1 pad 185: (no net) -> unconnected-(Module1B-GND-Pad185)
- Module1 pad 186: (no net) -> unconnected-(Module1B-GND-Pad186)
- Module1 pad 187: (no net) -> unconnected-(Module1B-DSI1_C_N-Pad187)
- Module1 pad 188: (no net) -> unconnected-(Module1B-HDMI0_CLK_P-Pad188)
- Module1 pad 189: (no net) -> unconnected-(Module1B-DSI1_C_P-Pad189)
- Module1 pad 190: (no net) -> unconnected-(Module1B-HDMI0_CLK_N-Pad190)
- Module1 pad 191: (no net) -> unconnected-(Module1B-GND-Pad191)
- Module1 pad 192: (no net) -> unconnected-(Module1B-GND-Pad192)
- Module1 pad 193: (no net) -> unconnected-(Module1B-DSI1_D2_N-Pad193)
- Module1 pad 194: (no net) -> unconnected-(Module1B-DSI1_D3_N-Pad194)
- Module1 pad 195: (no net) -> unconnected-(Module1B-DSI1_D2_P-Pad195)
- Module1 pad 196: (no net) -> unconnected-(Module1B-DSI1_D3_P-Pad196)
- Module1 pad 197: (no net) -> unconnected-(Module1B-GND-Pad197)
- Module1 pad 198: (no net) -> unconnected-(Module1B-GND-Pad198)
- Module1 pad 199: (no net) -> unconnected-(Module1B-HDMI0_SDA-Pad199)
- Module1 pad 200: (no net) -> unconnected-(Module1B-HDMI0_SCL-Pad200)
- SW1 pad 1: /mcu/buttons/matrix_R0 -> /mcu/matrix_R0
- SW10 pad 1: /mcu/buttons/matrix_R0 -> /mcu/matrix_R0
- SW11 pad 1: /mcu/buttons/matrix_R0 -> /mcu/matrix_R0
- SW12 pad 1: /mcu/buttons/matrix_R0 -> /mcu/matrix_R0
- SW13 pad 1: /mcu/buttons/matrix_R0 -> /mcu/matrix_R0
- SW14 pad 1: /mcu/buttons/matrix_R0 -> /mcu/matrix_R0
- SW15 pad 1: (no net) -> /mcu/matrix_R1
- SW15 pad 2: (no net) -> Net-(D15-A)
- SW16 pad 1: (no net) -> /mcu/matrix_R1
- SW16 pad 2: (no net) -> Net-(D16-A)
- SW17 pad 1: /mcu/buttons/matrix_R1 -> /mcu/matrix_R1
- SW18 pad 1: (no net) -> /mcu/matrix_R1
- SW18 pad 2: (no net) -> Net-(D18-A)
- SW19 pad 1: (no net) -> /mcu/matrix_R1
- SW19 pad 2: (no net) -> Net-(D19-A)
- SW2 pad 1: /mcu/buttons/matrix_R0 -> /mcu/matrix_R0
- SW20 pad 1: /mcu/buttons/matrix_R1 -> /mcu/matrix_R1
- SW21 pad 1: /mcu/buttons/matrix_R1 -> /mcu/matrix_R1
- SW22 pad 1: /mcu/buttons/matrix_R1 -> /mcu/matrix_R1
- SW23 pad 1: /mcu/buttons/matrix_R1 -> /mcu/matrix_R1
- SW24 pad 1: /mcu/buttons/matrix_R1 -> /mcu/matrix_R1
- SW25 pad 1: /mcu/buttons/matrix_R1 -> /mcu/matrix_R1
- SW26 pad 1: /mcu/buttons/matrix_R1 -> /mcu/matrix_R1
- SW27 pad 1: /mcu/buttons/matrix_R1 -> /mcu/matrix_R1
- SW28 pad 1: /mcu/buttons/matrix_R2 -> /mcu/matrix_R2
- SW29 pad 1: /mcu/buttons/matrix_R2 -> /mcu/matrix_R2
- SW3 pad 1: /mcu/buttons/matrix_R0 -> /mcu/matrix_R0
- SW30 pad 1: /mcu/buttons/matrix_R2 -> /mcu/matrix_R2
- SW31 pad 1: /mcu/buttons/matrix_R2 -> /mcu/matrix_R2
- SW32 pad 1: (no net) -> /mcu/matrix_R2
- SW32 pad 2: (no net) -> Net-(D32-A)
- SW33 pad 1: (no net) -> /mcu/matrix_R2
- SW33 pad 2: (no net) -> Net-(D33-A)
- SW34 pad 1: /mcu/buttons/matrix_R2 -> /mcu/matrix_R2
- SW35 pad 1: /mcu/buttons/matrix_R2 -> /mcu/matrix_R2
- SW36 pad 1: /mcu/buttons/matrix_R2 -> /mcu/matrix_R2
- SW37 pad 1: (no net) -> /mcu/matrix_R2
- SW37 pad 2: (no net) -> Net-(D37-A)
- SW38 pad 1: /mcu/buttons/matrix_R2 -> /mcu/matrix_R2
- SW39 pad 1: /mcu/buttons/matrix_R2 -> /mcu/matrix_R2
- SW4 pad 1: /mcu/buttons/matrix_R0 -> /mcu/matrix_R0
- SW40 pad 1: /mcu/buttons/matrix_R2 -> /mcu/matrix_R2
- SW41 pad 1: /mcu/buttons/matrix_R2 -> /mcu/matrix_R2
- SW5 pad 1: /mcu/buttons/matrix_R0 -> /mcu/matrix_R0
- SW6 pad 1: /mcu/buttons/matrix_R0 -> /mcu/matrix_R0
- SW7 pad 1: /mcu/buttons/matrix_R0 -> /mcu/matrix_R0
- SW8 pad 1: /mcu/buttons/matrix_R0 -> /mcu/matrix_R0
- SW9 pad 1: /mcu/buttons/matrix_R0 -> /mcu/matrix_R0
- U2 pad 11: /mcu/GPIO12 -> /mcu/matrix_C3
- U2 pad 12: /mcu/GPIO13 -> /mcu/matrix_C4
- U2 pad 13: /mcu/GPIO14 -> /mcu/matrix_C5
- U2 pad 14: /mcu/GPIO15 -> /mcu/matrix_C6
- U2 pad 16: /mcu/GPIO16 -> /mcu/matrix_C7
- U2 pad 17: /mcu/GPIO17 -> /mcu/matrix_C8
- U2 pad 18: /mcu/GPIO18 -> /mcu/matrix_C9
- U2 pad 19: /mcu/GPIO19 -> /mcu/matrix_C10
- U2 pad 20: /mcu/GPIO20 -> /mcu/matrix_C11
- U2 pad 21: /mcu/GPIO21 -> /mcu/matrix_C12
- U2 pad 22: /mcu/GPIO22 -> /mcu/matrix_C13
- U2 pad 23: /mcu/GPIO23 -> /mcu/ENC1_A
- U2 pad 25: /mcu/GPIO24 -> /mcu/ENC1_B
- U2 pad 26: /mcu/GPIO25 -> /mcu/ENC2_A
- U2 pad 27: /mcu/GPIO26 -> /mcu/ENC2_B
- U2 pad 28: /mcu/GPIO27 -> /mcu/ENC3_A
- U2 pad 3: /mcu/GPIO6 -> /mcu/matrix_R0
- U2 pad 36: /mcu/GPIO28 -> /mcu/ENC3_B
- U2 pad 37: /mcu/GPIO29 -> /mcu/ENC4_A
- U2 pad 38: /mcu/GPIO30 -> /mcu/ENC4_B
- U2 pad 39: /mcu/GPIO31 -> /mcu/ENC1_SW
- U2 pad 4: /mcu/GPIO7 -> /mcu/matrix_R1
- U2 pad 40: /mcu/GPIO32 -> /mcu/ENC2_SW
- U2 pad 42: /mcu/GPIO33 -> /mcu/ENC3_SW
- U2 pad 43: /mcu/GPIO34 -> /mcu/ENC4_SW
- U2 pad 44: /mcu/GPIO35 -> /mcu/JOYSTICK_SW
- U2 pad 45: /mcu/GPIO36 -> unconnected-(U2-GPIO36-Pad45)
- U2 pad 46: /mcu/GPIO37 -> unconnected-(U2-GPIO37-Pad46)
- U2 pad 47: /mcu/GPIO38 -> unconnected-(U2-GPIO38-Pad47)
- U2 pad 48: /mcu/GPIO39 -> unconnected-(U2-GPIO39-Pad48)
- U2 pad 49: /mcu/GPIO40_ADC0 -> /mcu/JOYSTICK_X
- U2 pad 52: /mcu/GPIO41_ADC1 -> /mcu/JOYSTICK_Y
- U2 pad 53: /mcu/GPIO42_ADC2 -> unconnected-(U2-GPIO42_ADC2-Pad53)
- U2 pad 54: /mcu/GPIO43_ADC3 -> unconnected-(U2-GPIO43_ADC3-Pad54)
- U2 pad 55: /mcu/GPIO44_ADC4 -> unconnected-(U2-GPIO44_ADC4-Pad55)
- U2 pad 56: /mcu/GPIO45_ADC5 -> unconnected-(U2-GPIO45_ADC5-Pad56)
- U2 pad 57: /mcu/GPIO46_ADC6 -> unconnected-(U2-GPIO46_ADC6-Pad57)
- U2 pad 58: /mcu/GPIO47_ADC7 -> unconnected-(U2-GPIO47_ADC7-Pad58)
- U2 pad 6: /mcu/GPIO8 -> /mcu/matrix_R2
- U2 pad 66: Net-(U2-USB_DM) -> unconnected-(U2-USB_DM-Pad66)
- U2 pad 67: Net-(U2-USB_DP) -> unconnected-(U2-USB_DP-Pad67)
- U2 pad 7: /mcu/GPIO9 -> /mcu/matrix_C0
- U2 pad 78: /mcu/GPIO1 -> /mcu/MIDI_RX
- U2 pad 8: /mcu/GPIO10 -> /mcu/matrix_C1
- U2 pad 9: /mcu/GPIO11 -> /mcu/matrix_C2
- U4 pad A: Net-(U4-PadA) -> /mcu/JOYSTICK_SW
- U4 pad B: Net-(U4-PadA) -> /mcu/JOYSTICK_SW
- U4 pad C: Net-(U4-PadC) -> GND
- U4 pad D: Net-(U4-PadC) -> GND
- U4 pad VR1_1: unconnected-(U4-PadVR1_1) -> GND
- U4 pad VR1_2: unconnected-(U4-PadVR1_2) -> /mcu/JOYSTICK_X
- U4 pad VR1_3: unconnected-(U4-PadVR1_3) -> +3V3
- U4 pad VR2_1: unconnected-(U4-PadVR2_1) -> GND
- U4 pad VR2_2: unconnected-(U4-PadVR2_2) -> /mcu/JOYSTICK_Y
- U4 pad VR2_3: unconnected-(U4-PadVR2_3) -> +3V3

Commit message: finish usb?
Parts:
- added U10: AP22653W6, Package_TO_SOT_SMD:SOT-23-6, F.Cu at (33.6, 174.9)
- C4: value 10u -> 1uF
- C7: value 10u -> 0.1uF
- J1: value USB_B_Micro -> USB_C_Receptacle_PowerOnly_6P
- R1, R4: value 1k -> 5.1k
- R5: value 27 -> 1M
- R6: value 27 -> 390k
- U1: value NCP1117-3.3_SOT223 -> TPS259531DSGR
Connections:
- net /mcu/CM4_TX renamed /mcu/MCU_RX
- net /mcu/CM5_TX renamed /mcu/MCU_TX
- C4 pad 1: VBUS -> +5V
- C7 pad 1: +3V3 -> Net-(C7-Pad1)
- J1 pad 1: VBUS -> (no net)
- J1 pad 2: /mcu/USB_D- -> (no net)
- J1 pad 3: /mcu/USB_D+ -> (no net)
- J1 pad 4: unconnected-(J1-ID-Pad4) -> (no net)
- J1 pad 5: GND -> (no net)
- J1 pad 6: GND -> (no net)
- J1 pad SH: (no net) -> GND
- Module1 pad 77: unconnected-(Module1A-+5v_(Input)-Pad77) -> +5V
- Module1 pad 79: unconnected-(Module1A-+5v_(Input)-Pad79) -> +5V
- Module1 pad 81: unconnected-(Module1A-+5v_(Input)-Pad81) -> +5V
- Module1 pad 83: unconnected-(Module1A-+5v_(Input)-Pad83) -> +5V
- Module1 pad 85: unconnected-(Module1A-+5v_(Input)-Pad85) -> +5V
- Module1 pad 87: unconnected-(Module1A-+5v_(Input)-Pad87) -> +5V
- P1 pad A1: Net-(P1-GND-PadA1) -> GND
- P1 pad A12: Net-(P1-GND-PadA1) -> GND
- P1 pad A5: unconnected-(P1-CC-PadA5) -> Net-(P1-CC)
- P1 pad A6: unconnected-(P1-D+-PadA6) -> Net-(P1-D+)
- P1 pad A7: unconnected-(P1-D--PadA7) -> Net-(P1-D-)
- P1 pad B1: Net-(P1-GND-PadA1) -> GND
- P1 pad B12: Net-(P1-GND-PadA1) -> GND
- P1 pad B5: unconnected-(P1-VCONN-PadB5) -> Net-(P1-VCONN)
- P1 pad SH: unconnected-(P1-SHIELD-PadSH) -> GND
- R1 pad 1: Net-(R1-Pad1) -> Net-(J1-CC2)
- R4 pad 1: /mcu/QSPI_SS -> Net-(J1-CC1)
- R4 pad 2: /mcu/~{USB_BOOT} -> GND
- R5 pad 1: /mcu/USB_D+ -> Net-(C7-Pad1)
- R5 pad 2: Net-(U2-USB_DP) -> Net-(U1-EN/UVLO)
- R6 pad 1: /mcu/USB_D- -> Net-(U1-EN/UVLO)
- R6 pad 2: Net-(U2-USB_DM) -> GND
- U1 pad 1: GND -> Net-(U1-DVDT)
- U1 pad 2: +3V3 -> Net-(U1-EN/UVLO)
- U1 pad 3: VBUS -> Net-(C7-Pad1)

Commit message: finish assignment
Parts:
- removed the J1 at (17.8, 279.3)
- removed SW101, SW102: SW_Push, Button_Switch_SMD:SW_Push_1P1T_NO_Vertical_Wuerth_434133025816
- added C60: 3.3nF, Capacitor_SMD:C_0805_2012Metric, F.Cu at (105.2, 274.3)
- added C61: 47uF, Capacitor_SMD:C_0805_2012Metric, F.Cu at (105.2, 277.3)
- added C62: 0.1uF, Capacitor_SMD:C_0805_2012Metric, F.Cu at (116.9, 265.5)
- added C63: 10uF, Capacitor_SMD:C_0805_2012Metric, F.Cu at (116.9, 268.5)
- added J8: USB_B_Micro, CM4IO:USB_Micro-B_EDAC_UCON00686, B.Cu at (257.5, 85.2)
- added R29: 681 @ 1%, Resistor_SMD:R_0805_2012Metric, F.Cu at (109.7, 274.2)
- added R30: 10k, Resistor_SMD:R_0805_2012Metric, F.Cu at (109.7, 277.2)
- added R31: 2.2k @ 1%, Resistor_SMD:R_0805_2012Metric, F.Cu at (105.2, 257.5)
- added R32: 49.9k @ 1%, Resistor_SMD:R_0805_2012Metric, F.Cu at (105.2, 260.4)
- added R33: 10k, Resistor_SMD:R_0805_2012Metric, F.Cu at (105.2, 263.4)
- added R34: 56k, Resistor_SMD:R_0805_2012Metric, F.Cu at (105.2, 266.3)
- added R35: 56k, Resistor_SMD:R_0805_2012Metric, F.Cu at (105.2, 269.3)
- added U8: 74AHC1G125DCKR, Package_TO_SOT_SMD:SOT-353_SC-70-5, F.Cu at (115.8, 274.6)
- added U9: FSUSB42MX, Package_SO:MSOP-10_3x3mm_P0.5mm, F.Cu at (111.0, 266.3)
- J1: renamed from P2; value USB_C_Plug_USB2.0 -> USB_C_Receptacle_PowerOnly_6P
- R1, R4, R5, R6: footprint Resistor_SMD:R_0402_1005Metric -> Resistor_SMD:R_0805_2012Metric
- U1: footprint Package_TO_SOT_SMD:SOT-223-3_TabPin2 -> ledaw:SON50P200X200X80-9N
Connections:
- J1 pad A1: Net-(P2-GND-PadA1) -> (no net)
- J1 pad A12: Net-(P2-GND-PadA1) -> GND
- J1 pad A4: Net-(P2-VBUS-PadA4) -> (no net)
- J1 pad A5: unconnected-(P2-CC-PadA5) -> Net-(J1-CC1)
- J1 pad A6: unconnected-(P2-D+-PadA6) -> (no net)
- J1 pad A7: unconnected-(P2-D--PadA7) -> (no net)
- J1 pad A9: Net-(P2-VBUS-PadA4) -> Net-(C7-Pad1)
- J1 pad B1: Net-(P2-GND-PadA1) -> (no net)
- J1 pad B12: Net-(P2-GND-PadA1) -> GND
- J1 pad B4: Net-(P2-VBUS-PadA4) -> (no net)
- J1 pad B5: unconnected-(P2-VCONN-PadB5) -> Net-(J1-CC2)
- J1 pad B9: Net-(P2-VBUS-PadA4) -> Net-(C7-Pad1)
- J1 pad SH: unconnected-(P2-SHIELD-PadSH) -> GND

Commit message: make key courtyard smaller
Parts:
- D3, D4, LS1, LS2: moved to F.Cu
- moved R10 201.3 mm to (127.9, 237.9)
- moved R11 201.3 mm to (127.9, 240.8)
- moved R12 201.3 mm to (127.9, 243.8)
- moved R15 201.3 mm to (127.9, 252.6)
- moved R16 201.3 mm to (127.9, 255.6)
- moved R17 201.3 mm to (132.3, 237.9)
- moved R18 201.3 mm to (132.3, 240.8)
- moved R19 201.3 mm to (132.3, 243.8)
- moved R22 201.3 mm to (132.3, 252.6)
- moved R23 201.3 mm to (132.3, 255.6)
- moved R24 201.3 mm to (136.7, 237.9)
- moved R25 201.3 mm to (136.7, 240.8)
- moved R26 201.3 mm to (136.7, 243.8)
- moved R13 201.3 mm to (127.9, 246.7)
- moved R14 201.3 mm to (127.9, 249.7)
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