File: hardware/board/board.kicad_pcb (KiCad board)
At the start: 2 copper layers, 300 x 120 mm, 239 parts, among them J1 USB_C_Receptacle_PowerOnly_6P, J2 SM03B-SRSS-TB, J3 MidiIn, J4 MidiOut, J5 LineIn, J6 LineOut, J7 Headphone, J8 USB_B_Micro, P1 USB_C_Plug_USB2.0, SW1 SW_Push, SW10 SW_Push, SW11 SW_Push, SW12 SW_Push, SW13 SW_Push, SW14 SW_Push, SW15 SW_Push, SW16 SW_Push, SW17 SW_Push, SW18 SW_Push, SW19 SW_Push, SW2 SW_Push, SW20 SW_Push, SW21 SW_Push, SW22 SW_Push, SW23 SW_Push, SW24 SW_Push, SW25 SW_Push, SW26 SW_Push, SW27 SW_Push, SW28 SW_Push, SW29 SW_Push, SW3 SW_Push, SW30 SW_Push, SW31 SW_Push, SW32 SW_Push, SW33 SW_Push, SW34 SW_Push, SW35 SW_Push, SW36 SW_Push, SW37 SW_Push, SW38 SW_Push, SW39 SW_Push, SW4 SW_Push, SW40 SW_Push, SW41 SW_Push, SW5 SW_Push, SW6 SW_Push, SW7 SW_Push, SW8 SW_Push, SW9 SW_Push, U1 TPS259531DSGR, U10 AP22653W6, U2 RP2350_80QFN, U3 Oled, U4 THB001P, U5 TPS7A20xxxDBV, U6 MAX98089ETN_T, U7 TLP2310, U8 74AHC1G125DCKR, U9 FSUSB42MX, Y1 ABM8-272-T3, Y2 12.288MHz

Commit message: connecting main
Parts:
- U4: value THB001P -> CNK_THB001P
- U6: value MAX98089ETN_T -> QFN40P700X700X80-57N
- moved TP12 261.5 mm to (311.3, 112.5)
- moved D14 259.1 mm to (342.3, 143.4), turned to 90 degrees
- moved TP10 258.0 mm to (314.6, 114.3)
- moved TP5 254.8 mm to (290.7, 99.5)
- moved TP3 254.5 mm to (289.7, 90.9)
- moved TP11 254.2 mm to (293.9, 99.4)
- moved TP4 250.8 mm to (291.4, 102.3)
- moved TP6 249.2 mm to (285.8, 106.6)
- moved C24 247.0 mm to (296.7, 112.1), turned to -90 degrees
- moved D27 246.8 mm to (349.4, 162.1)
- moved D43 243.6 mm to (306.8, 114.0), turned to 90 degrees
- moved C27 242.1 mm to (290.3, 96.2), turned to -90 degrees
- moved C26 239.5 mm to (293.9, 102.7), turned to -90 degrees
- moved TP14 239.3 mm to (285.4, 95.7)
- moved D13 239.2 mm to (322.3, 143.4), turned to 90 degrees
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
Commit message: matrix
Parts:
- removed J2: SM03B-SRSS-TB, Connector_JST:JST_SH_SM03B-SRSS-TB_1x03-1MP_P1.00mm_Horizontal
- D1, D10, D11, D12, D13, D14, D15, D16, D17, D18, D19, D2, D20, D21, D22, D23, D24, D25, D26, D27, D28, D29, D3, D30, D31, D32, D33, D34, D35, D36, D37, D38, D39, D4, D40, D41, D5, D6, D7, D8, D9: moved to B.Cu
- U4: value CNK_THB001P -> THB001P
- U6: value QFN40P700X700X80-57N -> MAX98089ETN_T
- moved TP12 321.3 mm to (142.3, 385.7)
- moved TP5 320.7 mm to (138.2, 381.7)
- moved TP3 320.7 mm to (138.2, 373.6)
- moved TP11 320.4 mm to (142.3, 381.7)
- moved TP6 315.8 mm to (138.2, 385.7)
- moved TP4 315.0 mm to (138.2, 377.6)
- moved TP10 314.7 mm to (142.3, 377.6)
- moved TP14 307.1 mm to (146.3, 369.5)
- moved D43 304.0 mm to (150.9, 375.1), turned to 0 degrees
- moved C24 300.0 mm to (126.2, 358.9), turned to 0 degrees
- moved C27 299.7 mm to (130.7, 349.9), turned to 0 degrees
- moved TP13 298.8 mm to (146.3, 365.5)
- moved TP16 298.5 mm to (146.3, 377.6)
- moved TP8 297.6 mm to (142.3, 369.5)
- moved LS2 296.8 mm to (127.6, 381.5)
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Connections:
- net /FUSE_FAULT renamed /usb/FUSE_~{FLT}
- Module1 pad 1: unconnected-(Module1A-GND-Pad1) -> GND
- Module1 pad 101: unconnected-(Module1B-USB_OTG_ID-Pad101) -> /USB2_OTG_ID
- Module1 pad 103: unconnected-(Module1B-USB2_N-Pad103) -> /USB2_N
- Module1 pad 105: unconnected-(Module1B-USB2_P-Pad105) -> /USB2_P
- Module1 pad 107: unconnected-(Module1B-GND-Pad107) -> GND
- Module1 pad 108: unconnected-(Module1B-GND-Pad108) -> GND
- Module1 pad 113: unconnected-(Module1B-GND-Pad113) -> GND
- Module1 pad 114: unconnected-(Module1B-GND-Pad114) -> GND
- Module1 pad 119: unconnected-(Module1B-GND-Pad119) -> GND
- Module1 pad 120: unconnected-(Module1B-GND-Pad120) -> GND
- Module1 pad 125: unconnected-(Module1B-GND-Pad125) -> GND
- Module1 pad 126: unconnected-(Module1B-GND-Pad126) -> GND
- Module1 pad 13: unconnected-(Module1A-GND-Pad13) -> GND
- Module1 pad 131: unconnected-(Module1B-GND-Pad131) -> GND
- Module1 pad 132: unconnected-(Module1B-GND-Pad132) -> GND
- Module1 pad 137: unconnected-(Module1B-GND-Pad137) -> GND
- Module1 pad 138: unconnected-(Module1B-GND-Pad138) -> GND
- Module1 pad 14: unconnected-(Module1A-GND-Pad14) -> GND
- Module1 pad 143: unconnected-(Module1B-HDMI1_HOTPLUG-Pad143) -> GND
- Module1 pad 144: unconnected-(Module1B-GND-Pad144) -> GND
- Module1 pad 149: unconnected-(Module1B-HDMI1_CEC-Pad149) -> GND
- Module1 pad 150: unconnected-(Module1B-GND-Pad150) -> GND
- Module1 pad 155: unconnected-(Module1B-GND-Pad155) -> GND
- Module1 pad 156: unconnected-(Module1B-GND-Pad156) -> GND
- Module1 pad 161: unconnected-(Module1B-GND-Pad161) -> GND
- Module1 pad 162: unconnected-(Module1B-GND-Pad162) -> GND
- Module1 pad 167: unconnected-(Module1B-GND-Pad167) -> GND
- Module1 pad 168: unconnected-(Module1B-GND-Pad168) -> GND
- Module1 pad 173: unconnected-(Module1B-GND-Pad173) -> GND
- Module1 pad 174: unconnected-(Module1B-GND-Pad174) -> GND
- Module1 pad 179: unconnected-(Module1B-GND-Pad179) -> GND
- Module1 pad 180: unconnected-(Module1B-GND-Pad180) -> GND
- Module1 pad 185: unconnected-(Module1B-GND-Pad185) -> GND
- Module1 pad 186: unconnected-(Module1B-GND-Pad186) -> GND
- Module1 pad 191: unconnected-(Module1B-GND-Pad191) -> GND
- Module1 pad 192: unconnected-(Module1B-GND-Pad192) -> GND
- Module1 pad 197: unconnected-(Module1B-GND-Pad197) -> GND
- Module1 pad 198: unconnected-(Module1B-GND-Pad198) -> GND
- Module1 pad 2: unconnected-(Module1A-GND-Pad2) -> GND
- Module1 pad 22: unconnected-(Module1A-GND-Pad22) -> GND
- Module1 pad 23: unconnected-(Module1A-GND-Pad23) -> GND
- Module1 pad 24: unconnected-(Module1A-GPIO26-Pad24) -> /USB2_~{FAULT}
- Module1 pad 25: unconnected-(Module1A-GPIO21-Pad25) -> /PCM_DOUT
- Module1 pad 26: unconnected-(Module1A-GPIO19-Pad26) -> /PCM_FS
- Module1 pad 27: unconnected-(Module1A-GPIO20-Pad27) -> /PCM_DIN
- Module1 pad 28: unconnected-(Module1A-GPIO13-Pad28) -> /SWD
- Module1 pad 30: unconnected-(Module1A-GPIO6-Pad30) -> /DC
- Module1 pad 31: unconnected-(Module1A-GPIO12-Pad31) -> /SWCLK
- Module1 pad 32: unconnected-(Module1A-GND-Pad32) -> GND
- Module1 pad 33: unconnected-(Module1A-GND-Pad33) -> GND
- Module1 pad 34: unconnected-(Module1A-GPIO5-Pad34) -> /RST
- Module1 pad 38: unconnected-(Module1A-GPIO11-Pad38) -> /SPI0_SCLK
- Module1 pad 39: unconnected-(Module1A-GPIO8-Pad39) -> /SPI0_CE0
- Module1 pad 41: unconnected-(Module1A-GPIO25-Pad41) -> /CODEC_~{IRQ}
- Module1 pad 42: unconnected-(Module1A-GND-Pad42) -> GND
- Module1 pad 43: unconnected-(Module1A-GND-Pad43) -> GND
- Module1 pad 44: unconnected-(Module1A-GPIO10-Pad44) -> /SPI0_MOSI
- Module1 pad 45: unconnected-(Module1A-GPIO24-Pad45) -> /USBH_EN
- Module1 pad 46: unconnected-(Module1A-GPIO22-Pad46) -> /CODEC_1V8EN
- Module1 pad 47: unconnected-(Module1A-GPIO23-Pad47) -> /CODEC_CLKEN
- Module1 pad 48: unconnected-(Module1A-GPIO27-Pad48) -> /RUN
- Module1 pad 49: unconnected-(Module1A-GPIO18-Pad49) -> /PCM_CLK
- Module1 pad 51: unconnected-(Module1A-GPIO15-Pad51) -> /UART0_RX
- Module1 pad 52: unconnected-(Module1A-GND-Pad52) -> GND
- Module1 pad 53: unconnected-(Module1A-GND-Pad53) -> GND
- Module1 pad 55: unconnected-(Module1A-GPIO14-Pad55) -> /UART0_TX
- Module1 pad 56: unconnected-(Module1A-GPIO3-Pad56) -> /I2C1_SCL
- Module1 pad 58: unconnected-(Module1A-GPIO2-Pad58) -> /I2C1_SDA
- Module1 pad 59: unconnected-(Module1A-GND-Pad59) -> GND
- Module1 pad 60: unconnected-(Module1A-GND-Pad60) -> GND
- Module1 pad 65: unconnected-(Module1A-GND-Pad65) -> GND
- Module1 pad 66: unconnected-(Module1A-GND-Pad66) -> GND
- Module1 pad 7: unconnected-(Module1A-GND-Pad7) -> GND
- Module1 pad 71: unconnected-(Module1A-GND-Pad71) -> GND
- Module1 pad 74: unconnected-(Module1A-GND-Pad74) -> GND
- Module1 pad 8: unconnected-(Module1A-GND-Pad8) -> GND
- Module1 pad 98: unconnected-(Module1A-GND-Pad98) -> GND
- R29 pad 1: /FUSE_VILM -> /mcu/FUSE_ILM
- R31 pad 2: /usb/USB_OTG -> /USB2_OTG_ID
- R33 pad 2: /usb/USBH_~{FAULT} -> /USB2_~{FAULT}
- R7 pad 1: /audio/CODEC_1V8EN -> /CODEC_1V8EN
- R8 pad 1: /audio/CODEC_~{IRQ} -> /CODEC_~{IRQ}
- U1 pad 7: /FUSE_VILM -> /mcu/FUSE_ILM
- U10 pad 3: /usb/USBH_EN -> /USBH_EN
- U10 pad 4: /usb/USBH_~{FAULT} -> /USB2_~{FAULT}
- U2 pad 1: /mcu/MCU_RX -> /UART0_RX
- U2 pad 2: /mcu/MCU_TX -> /UART0_TX
- U2 pad 33: /mcu/SWCLK -> /MCU_SWCLK
- U2 pad 34: /mcu/SWD -> /MCU_SWD
- U2 pad 35: /mcu/RUN -> /RUN
- U2 pad 58: unconnected-(U2-GPIO47_ADC7-Pad58) -> /mcu/FUSE_ILM
- U5 pad 3: /audio/CODEC_1V8EN -> /CODEC_1V8EN
- U6 pad 10: /audio/CODEC_LRCLKS1 -> /PCM_DIN
- U6 pad 51: /audio/CODEC_SCL -> /I2C1_SCL
- U6 pad 52: /audio/CODEC_SDA -> /I2C1_SDA
- U6 pad 56: /audio/CODEC_~{IRQ} -> /CODEC_~{IRQ}
- U6 pad 7: /audio/CODEC_SDOUTS1 -> /PCM_FS
- U6 pad 8: /audio/CODEC_BCLKS1 -> /PCM_CLK
- U6 pad 9: /audio/CODEC_SDINS1 -> /PCM_DOUT
- U9 pad 2: /usb/USB_OTG -> /USB2_OTG_ID
- U9 pad 3: /usb/USB_P -> /USB2_P
- U9 pad 4: /usb/USB_N -> /USB2_N
- Y2 pad 1: /audio/CODEC_CLKEN -> /CODEC_CLKEN
Routing:
- net /mcu/matrix_R1: track 0.00 -> 322.7 mm
- net /mcu/matrix_R0: track 0.00 -> 273.5 mm
- net /mcu/matrix_R2: track 0.00 -> 273.5 mm
- net /mcu/matrix_C2: track 0.00 -> 127.9 mm
- net /mcu/matrix_C1: track 0.00 -> 111.5 mm
- net /mcu/matrix_C3: track 0.00 -> 106.6 mm
- net /mcu/matrix_C4: track 0.00 -> 99.2 mm
- net /mcu/matrix_C0: track 0.00 -> 82.2 mm
- net /mcu/matrix_C11: track 0.00 -> 79.7 mm
- net /mcu/matrix_C12: track 0.00 -> 74.9 mm
- net /mcu/matrix_C5: track 0.00 -> 73.3 mm
- net /mcu/matrix_C7: track 0.00 -> 72.4 mm
- net /mcu/matrix_C6: track 0.00 -> 69.0 mm
- net /mcu/matrix_C9: track 0.00 -> 58.3 mm
- net /mcu/matrix_C8: track 0.00 -> 58.3 mm
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
Commit message: LeMatrix
Parts:
- C1, C10, C2, C3, C5, C6, C8, C9, D42, D43, L1, R2, R3, U1, U10, U2, U5, U6, U7, U9, Y1: moved to B.Cu
- moved D43 326.7 mm to (323.1, 97.5), turned to 180 degrees
- moved U5 291.6 mm to (284.6, 120.5), turned to 180 degrees
- moved U6 288.2 mm to (291.5, 115.0), turned to 90 degrees
- moved U7 268.8 mm to (183.5, 100.5), turned to 180 degrees
- moved D42 266.1 mm to (181.5, 105.0), turned to 180 degrees
- moved U8 255.2 mm to (152.5, 99.0)
- moved U1 245.8 mm to (114.0, 94.2), turned to 180 degrees
- moved U10 238.7 mm to (130.5, 93.5), turned to 180 degrees
- moved U9 230.7 mm to (142.0, 95.0), turned to 180 degrees
- moved R3 226.2 mm to (223.4, 149.0), turned to -90 degrees
- moved C8 220.9 mm to (223.4, 151.0), turned to -90 degrees
- moved C5 217.7 mm to (226.4, 150.9), turned to 180 degrees
- moved C6 215.4 mm to (237.6, 157.8)
- moved C3 214.8 mm to (226.4, 151.9), turned to 180 degrees
- moved L1 209.9 mm to (226.4, 149.2), turned to 180 degrees
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Connections:
- U2 pad 1: /UART0_RX -> /mcu/MIDI_TX
- U2 pad 11: /mcu/matrix_C3 -> unconnected-(U2-GPIO12-Pad11)
- U2 pad 12: /mcu/matrix_C4 -> unconnected-(U2-GPIO13-Pad12)
- U2 pad 13: /mcu/matrix_C5 -> unconnected-(U2-GPIO14-Pad13)
- U2 pad 14: /mcu/matrix_C6 -> unconnected-(U2-GPIO15-Pad14)
- U2 pad 16: /mcu/matrix_C7 -> /mcu/matrix_R0
- U2 pad 17: /mcu/matrix_C8 -> /mcu/matrix_R1
- U2 pad 18: /mcu/matrix_C9 -> /mcu/matrix_R2
- U2 pad 19: /mcu/matrix_C10 -> /mcu/matrix_C13
- U2 pad 2: /UART0_TX -> /mcu/MIDI_RX
- U2 pad 20: /mcu/matrix_C11 -> /mcu/matrix_C12
- U2 pad 21: /mcu/matrix_C12 -> /mcu/matrix_C11
- U2 pad 22: /mcu/matrix_C13 -> /mcu/matrix_C10
- U2 pad 23: /mcu/ENC1_A -> /mcu/matrix_C9
- U2 pad 25: /mcu/ENC1_B -> /mcu/matrix_C8
- U2 pad 26: /mcu/ENC2_A -> /mcu/matrix_C7
- U2 pad 27: /mcu/ENC2_B -> /mcu/matrix_C6
- U2 pad 28: /mcu/ENC3_A -> /mcu/matrix_C5
- U2 pad 3: /mcu/matrix_R0 -> /mcu/ENC1_A
- U2 pad 36: /mcu/ENC3_B -> /mcu/matrix_C4
- U2 pad 37: /mcu/ENC4_A -> /mcu/matrix_C3
- U2 pad 38: /mcu/ENC4_B -> /mcu/matrix_C2
- U2 pad 39: /mcu/ENC1_SW -> /mcu/matrix_C1
- U2 pad 4: /mcu/matrix_R1 -> /mcu/ENC1_B
- U2 pad 40: /mcu/ENC2_SW -> /mcu/matrix_C0
- U2 pad 42: /mcu/ENC3_SW -> unconnected-(U2-GPIO33-Pad42)
- U2 pad 43: /mcu/ENC4_SW -> /mcu/ENC3_A
- U2 pad 44: /mcu/JOYSTICK_SW -> /mcu/ENC3_B
- U2 pad 45: unconnected-(U2-GPIO36-Pad45) -> /mcu/ENC4_A
- U2 pad 46: unconnected-(U2-GPIO37-Pad46) -> /mcu/ENC4_B
- U2 pad 47: unconnected-(U2-GPIO38-Pad47) -> /mcu/ENC3_SW
- U2 pad 48: unconnected-(U2-GPIO39-Pad48) -> /mcu/ENC4_SW
- U2 pad 49: /mcu/JOYSTICK_X -> unconnected-(U2-GPIO40_ADC0-Pad49)
- U2 pad 52: /mcu/JOYSTICK_Y -> unconnected-(U2-GPIO41_ADC1-Pad52)
- U2 pad 56: unconnected-(U2-GPIO45_ADC5-Pad56) -> /mcu/JOYSTICK_X
- U2 pad 57: unconnected-(U2-GPIO46_ADC6-Pad57) -> /mcu/JOYSTICK_Y
- U2 pad 6: /mcu/matrix_R2 -> /mcu/ENC2_A
- U2 pad 7: /mcu/matrix_C0 -> /mcu/ENC2_B
- U2 pad 77: /mcu/MIDI_TX -> /UART0_RX
- U2 pad 78: /mcu/MIDI_RX -> /UART0_TX
- U2 pad 79: /mcu/GPIO2 -> /mcu/ENC1_SW
- U2 pad 8: /mcu/matrix_C1 -> /mcu/JOYSTICK_SW
- U2 pad 80: /mcu/GPIO3 -> /mcu/ENC2_SW
- U2 pad 9: /mcu/matrix_C2 -> unconnected-(U2-GPIO11-Pad9)
Routing:
- net /mcu/matrix_C0: track 82.2 -> 218.7 mm
- net /mcu/matrix_C13: track 58.3 -> 194.0 mm
- net /mcu/matrix_C12: track 74.9 -> 201.3 mm, vias 0 -> 2
- net /mcu/matrix_C1: track 111.5 -> 226.5 mm, vias 0 -> 2
- net /mcu/matrix_C11: track 79.7 -> 183.9 mm, vias 0 -> 2
- net /mcu/matrix_C2: track 127.9 -> 219.7 mm, vias 0 -> 2
- net /mcu/matrix_C10: track 58.3 -> 143.1 mm, vias 0 -> 2
- net /mcu/matrix_C3: track 106.6 -> 183.3 mm, vias 0 -> 2
- net /mcu/matrix_C9: track 58.3 -> 125.1 mm, vias 0 -> 4
- net /mcu/matrix_R0: track 273.5 -> 330.9 mm
- net /mcu/matrix_C4: track 99.2 -> 147.5 mm, vias 0 -> 2
- net /UART0_TX: track 0.00 -> 46.2 mm, vias 0 -> 2
- net /mcu/matrix_C8: track 58.3 -> 103.6 mm, vias 0 -> 4
- net /UART0_RX: track 0.00 -> 44.8 mm
- net /mcu/matrix_C5: track 73.3 -> 114.2 mm, vias 0 -> 2
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- added copper zone on In1.Cu, net (none)
- added copper zone on B.Cu, net +1V1
- added copper zone on B.Cu, net +3V3
- added copper zone on B.Cu, net /mcu/VREG_LX
- added copper zone on B.Cu, net GND
Other:
- copper layers 2 -> 4

Commit message: start audio codec
Parts:
- moved U5 8.03 mm to (282.8, 112.8), turned to 0 degrees
Changed lines of the file:
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@@
 	(footprint "Package_TO_SOT_SMD:SOT-23-5"
 		(layer "B.Cu")
-		(at 284.6375 120.55 180)
+		(at 282.75 112.75)
 		(descr "SOT, 5 Pin (JEDEC MO-178 Var AA https://www.jedec.org/document_search?search_api_views_fulltext=MO-178)")
 		(tags "SOT TO_SOT_SMD")
@@
 		)
 		(property "LCSC" "C2862740"
-			(at 0 0 0)
+			(at 0 0 180)
 			(unlocked yes)
 			(layer "B.Fab")
@@
 		(duplicate_pad_numbers_are_jumpers no)
 		(fp_line
-			(start 0.91 1.56)
-			(end 0.91 1.51)
+			(start -0.91 -1.56)
+			(end -0.91 -1.51)
 			(stroke
 				(width 0.12)
@@
 		)
 		(fp_line
-			(start 0.91 0.39)
-			(end 0.91 -0.39)
+			(start -0.91 1.51)
+			(end -0.91 1.56)
 			(stroke
 				(width 0.12)
@@
 		)
 		(fp_line
-			(start 0.91 -1.51)
-			(end 0.91 -1.56)
+			(start -0.91 1.56)
+			(end 0.91 1.56)
 			(stroke
 				(width 0.12)
@@
 		)
 		(fp_line
-			(start -0.91 1.56)
-			(end 0.91 1.56)
+			(start 0.91 -1.51)
+			(end 0.91 -1.56)
 			(stroke
 				(width 0.12)
@@
 		)
 		(fp_line
-			(start -0.91 1.51)
-			(end -0.91 1.56)
+			(start 0.91 0.39)
+			(end 0.91 -0.39)
 			(stroke
 				(width 0.12)
@@
 		)
 		(fp_line
-			(start -0.91 -1.56)
-			(end -0.91 -1.51)
+			(start 0.91 1.56)
+			(end 0.91 1.51)
 			(stroke
 				(width 0.12)
@@
 		)
 		(fp_line
-			(start 2.05 1.5)
-			(end 2.05 0.39)
+			(start -2.05 -1.5)
+			(end -2.05 1.5)
 			(stroke
 				(width 0.05)
@@
 		)
 		(fp_line
-			(start 2.05 0.39)
-			(end 1.05 0.39)
+			(start -2.05 1.5)
+			(end -1.05 1.5)
 			(stroke
 				(width 0.05)
@@
 		)
 		(fp_line
-			(start 2.05 -0.39)
-			(end 2.05 -1.5)
+			(start -1.05 -1.7)
+			(end -1.05 -1.5)
 			(stroke
 				(width 0.05)
@@
 		)
 		(fp_line
-			(start 2.05 -1.5)
-			(end 1.05 -1.5)
+			(start -1.05 -1.5)
+			(end -2.05 -1.5)
 			(stroke
 				(width 0.05)
@@
 		)
 		(fp_line
-			(start 1.05 1.7)
-			(end 1.05 1.5)
+			(start -1.05 1.5)
+			(end -1.05 1.7)
 			(stroke
 				(width 0.05)
@@
 		)
 		(fp_line
-			(start 1.05 1.5)
-			(end 2.05 1.5)
+			(start -1.05 1.7)
+			(end 1.05 1.7)
 			(stroke
 				(width 0.05)
@@
 		)
 		(fp_line
-			(start 1.05 0.39)
-			(end 1.05 -0.39)
+			(start 1.05 -1.7)
+			(end -1.05 -1.7)
 			(stroke
 				(width 0.05)
@@
 		)
 		(fp_line
-			(start 1.05 -0.39)
-			(end 2.05 -0.39)
+			(start 1.05 -1.5)
+			(end 1.05 -1.7)
 			(stroke
 				(width 0.05)
@@
 		)
 		(fp_line
-			(start 1.05 -1.5)
-			(end 1.05 -1.7)
+			(start 1.05 -0.39)
+			(end 2.05 -0.39)
 			(stroke
 				(width 0.05)
@@
 		)
 		(fp_line
-			(start 1.05 -1.7)
-			(end -1.05 -1.7)
+			(start 1.05 0.39)
+			(end 1.05 -0.39)
 			(stroke
 				(width 0.05)
@@
 		)
 		(fp_line
-			(start -1.05 1.7)
-			(end 1.05 1.7)
+			(start 1.05 1.5)
+			(end 2.05 1.5)
 			(stroke
 				(width 0.05)
@@
 		)
 		(fp_line
-			(start -1.05 1.5)
-			(end -1.05 1.7)
+			(start 1.05 1.7)
+			(end 1.05 1.5)
 			(stroke
 				(width 0.05)
@@
 		)
 		(fp_line
-			(start -1.05 -1.5)
-			(end -2.05 -1.5)
+			(start 2.05 -1.5)
+			(end 1.05 -1.5)
 			(stroke
 				(width 0.05)
@@
 		)
 		(fp_line
-			(start -1.05 -1.7)
-			(end -1.05 -1.5)
+			(start 2.05 -0.39)
+			(end 2.05 -1.5)
 			(stroke
 				(width 0.05)
@@
 		)
 		(fp_line
-			(start -2.05 1.5)
-			(end -1.05 1.5)
+			(start 2.05 0.39)
+			(end 1.05 0.39)
 			(stroke
 				(width 0.05)
@@
 		)
 		(fp_line
-			(start -2.05 -1.5)
-			(end -2.05 1.5)
+			(start 2.05 1.5)
+			(end 2.05 0.39)
 			(stroke
 				(width 0.05)
@@
 		)
 		(pad "1" smd roundrect
-			(at -1.1375 0.95 180)
+			(at -1.1375 0.95)
 			(size 1.325 0.6)
 			(layers "B.Cu" "B.Mask" "B.Paste")
@@
 		)
 		(pad "2" smd roundrect
-			(at -1.1375 0 180)
+			(at -1.1375 0)
 			(size 1.325 0.6)
 			(layers "B.Cu" "B.Mask" "B.Paste")
@@
 		)
 		(pad "3" smd roundrect
-			(at -1.1375 -0.95 180)
+			(at -1.1375 -0.95)
 			(size 1.325 0.6)
 			(layers "B.Cu" "B.Mask" "B.Paste")
@@
 		)
 		(pad "4" smd roundrect
-			(at 1.1375 -0.95 180)
+			(at 1.1375 -0.95)
 			(size 1.325 0.6)
 			(layers "B.Cu" "B.Mask" "B.Paste")
@@
 		)
 		(pad "5" smd roundrect
-			(at 1.1375 0.95 180)
+			(at 1.1375 0.95)
 			(size 1.325 0.6)
 			(layers "B.Cu" "B.Mask" "B.Paste")
@@
 	)
 	(segment
-		(start 231.5 150.766667)
-		(end 231.5 128.6)
-		(width 0.2)
-		(layer "B.Cu")
-		(net "/UART0_TX")
-	)
-	(segment
 		(start 232.366667 151)
 		(end 232.466667 150.9)
@@
 	)
 	(segment
-		(start 231.5 128.6)
-		(end 227.1 124.2)
+		(start 231.466667 150.8)
+		(end 231.5 150.766667)
 		(width 0.2)
 		(layer "B.Cu")
@@
 	)
 	(segment
-		(start 231.466667 150.8)
-		(end 231.5 150.766667)
+		(start 231.5 150.766667)
+		(end 231.5 128.6)
 		(width 0.2)
 		(layer "B.Cu")
@@
 	)
 	(segment
-		(start 215.3 124.2)
+		(start 215.1 124)
 		(end 214 122.9)
 		(width 0.2)
@@
 	)
 	(segment
-		(start 227.1 124.2)
-		(end 215.3 124.2)
+		(start 226.9 124)
+		(end 215.1 124)
+		(width 0.2)
+		(layer "B.Cu")
+		(net "/UART0_TX")
+	)
+	(segment
+		(start 231.5 128.6)
+		(end 226.9 124)
 		(width 0.2)
 		(layer "B.Cu")

Commit message: fix hpmic / linein mixup
Parts:
- added C10: 1uF, Capacitor_SMD:C_0805_2012Metric, B.Cu at (185.5, 245.7)
- added C11: 1uF, Capacitor_SMD:C_0805_2012Metric, B.Cu at (183.3, 245.7)
- added C12: 100nF, Capacitor_SMD:C_0805_2012Metric, F.Cu at (184.4, 262.4)
- added C13: 1uF, Capacitor_SMD:C_0805_2012Metric, F.Cu at (191.0, 257.1)
- added C14: 10uF, Capacitor_SMD:C_0805_2012Metric, F.Cu at (174.3, 252.9)
- added C15: 1uF, Capacitor_SMD:C_0805_2012Metric, F.Cu at (176.5, 252.9)
- added C16: 1uF, Capacitor_SMD:C_0805_2012Metric, F.Cu at (194.7, 257.1)
- added C17: 10uF, Capacitor_SMD:C_0805_2012Metric, F.Cu at (178.0, 261.1)
- added C18: 1uF, Capacitor_SMD:C_0805_2012Metric, F.Cu at (178.0, 256.7)
- added C19: 1uF, Capacitor_SMD:C_0805_2012Metric, F.Cu at (179.9, 249.9)
- added C20: 1uF, Capacitor_SMD:C_0805_2012Metric, F.Cu at (178.7, 252.9)
- added C21: 1uF, Capacitor_SMD:C_0805_2012Metric, F.Cu at (178.0, 258.9)
- added C22: 1uF, Capacitor_SMD:C_0805_2012Metric, F.Cu at (183.5, 249.9)
- added C23: 100nF, Capacitor_SMD:C_0805_2012Metric, F.Cu at (191.0, 259.3)
- added C24: 1uF, Capacitor_SMD:C_0805_2012Metric, F.Cu at (191.0, 254.9)
- added C25: 2.2uF, Capacitor_SMD:C_0805_2012Metric, F.Cu at (194.7, 254.9)
- added C26: 10uF, Capacitor_SMD:C_0805_2012Metric, B.Cu at (176.5, 249.2)
- added C27: 10uF, Capacitor_SMD:C_0805_2012Metric, B.Cu at (174.3, 249.2)
- added C3: 1uF, Capacitor_SMD:C_0805_2012Metric, B.Cu at (176.8, 263.4)
- added C6: 100nF, Capacitor_SMD:C_0805_2012Metric, B.Cu at (192.9, 262.5)
- added FB1: 600Ohm@100MHz, Inductor_SMD:L_0805_2012Metric, B.Cu at (190.8, 262.5)
- added R1: 10k, Resistor_SMD:R_0805_2012Metric, B.Cu at (176.8, 265.6)
- added R4: 10k, Resistor_SMD:R_0805_2012Metric, F.Cu at (194.7, 259.3)
- added R5: 2.2k, Resistor_SMD:R_0805_2012Metric, F.Cu at (191.0, 252.7)
- added U2: TPS7A20xxxDBV, Package_TO_SOT_SMD:SOT-23-5, B.Cu at (180.5, 264.5)
- added U4: MAX98089ETN_T, footprints:MAX98089ETN_T, B.Cu at (184.5, 255.6)
- added Y1: 12.288MHz, Oscillator:Oscillator_SMD_SeikoEpson_SG210-4Pin_2.5x2.0mm, B.Cu at (187.8, 262.1)
Routing:
- net /GPIO3/SCL1: track 0.00 -> 36.6 mm, vias 0 -> 1
- net /GPIO2/SDA1: track 0.00 -> 36.3 mm, vias 0 -> 1
- net GND: track 3.53 -> 39.3 mm, vias 5 -> 30
- net /codec/DIGMICDATA: track 0.00 -> 29.8 mm, vias 0 -> 1
- net +1V8: track 0.00 -> 28.7 mm, vias 0 -> 5
- net /codec/DIGMICCLK: track 0.00 -> 28.7 mm, vias 0 -> 1
- net /codec/JackS: track 0.00 -> 23.1 mm, vias 0 -> 2
- net /GPIO25: track 0.00 -> 15.6 mm, vias 0 -> 2
- net Net-(U4-MIC2N): track 0.00 -> 15.0 mm
- net Net-(U4-INA1/EXTMICP): track 0.00 -> 13.1 mm, vias 0 -> 2
- net Net-(U4-MIC2P): track 0.00 -> 13.1 mm
- net /GPIO18/PCM.CLK: track 0.00 -> 12.5 mm, vias 0 -> 1
- net /GPIO19/PCM.FS: track 0.00 -> 11.0 mm, vias 0 -> 1
- net /GPIO21/PCM.DOUT: track 0.00 -> 10.6 mm, vias 0 -> 1
- net Net-(U4-INA2/EXTMICN): track 0.00 -> 10.3 mm, vias 0 -> 2
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- added copper zone on B.Cu, net +5V
Other:
- board text added: "headphone"
- board text added: "i2s"
- board text added: "linein"
- board text added: "lineout"
- board text added: "speaker"
