File: hardware/board/board.kicad_pcb (KiCad board)
At the start: 4 copper layers, 300 x 120 mm, 265 parts, among them J1 USB_C_Receptacle_PowerOnly_6P, J3 MidiIn, J4 MidiOut, J5 LineIn, J6 LineOut, J7 Headphone, J8 USB_B_Micro, P1 USB_C_Plug_USB2.0, SW1 SW_Push, SW10 SW_Push, SW11 SW_Push, SW12 SW_Push, SW13 SW_Push, SW14 SW_Push, SW15 SW_Push, SW16 SW_Push, SW17 SW_Push, SW18 SW_Push, SW19 SW_Push, SW2 SW_Push, SW20 SW_Push, SW21 SW_Push, SW22 SW_Push, SW23 SW_Push, SW24 SW_Push, SW25 SW_Push, SW26 SW_Push, SW27 SW_Push, SW28 SW_Push, SW29 SW_Push, SW3 SW_Push, SW30 SW_Push, SW31 SW_Push, SW32 SW_Push, SW33 SW_Push, SW34 SW_Push, SW35 SW_Push, SW36 SW_Push, SW37 SW_Push, SW38 SW_Push, SW39 SW_Push, SW4 SW_Push, SW40 SW_Push, SW41 SW_Push, SW5 SW_Push, SW6 SW_Push, SW7 SW_Push, SW8 SW_Push, SW9 SW_Push, U1 TPS259531DSGR, U10 AP22653W6, U2 RP2350_80QFN, U2 TPS7A20xxxDBV, U3 Oled, U4 MAX98089ETN_T, U4 THB001P, U5 TPS7A20xxxDBV, U6 MAX98089ETN_T, U7 TLP2310, U8 74AHC1G125DCKR, U9 FSUSB42MX, Y1 12.288MHz, Y1 ABM8-272-T3, Y2 12.288MHz

Commit message: wip doing the copy from hat
Parts:
- removed the C11 at (186.6, 362.5)
- removed C12, C13, C16: 100n, Capacitor_SMD:C_0402_1005Metric
- removed the C14 at (186.6, 368.4)
- removed the C15 at (189.5, 358.5)
- removed the C17 at (189.5, 362.5)
- removed the C18 at (189.5, 364.4)
- removed the C19 at (189.5, 366.4)
- removed C20, C22 (x2), C24, C28, C29, C33, C36, C37, C38, C39, C4, C40, C42: 1uF, Capacitor_SMD:C_0805_2012Metric
- removed C20, C41, C59: 100nF, Capacitor_SMD:C_0805_2012Metric
- removed the C21 at (126.2, 349.9)
- removed the C23 at (126.2, 355.9)
- removed the C23 at (191.0, 259.3)
- removed C24: 47pF, Capacitor_SMD:C_0805_2012Metric
- removed the C25 at (126.2, 361.9)
- removed the C25 at (194.7, 254.9)
- removed the C26 at (130.7, 346.9)
- removed the C27 at (130.7, 349.9)
- removed the C30 at (130.7, 358.9)
- removed the C31 at (130.7, 361.9)
- removed C32, C35, C44, C45, C63: 10uF, Capacitor_SMD:C_0805_2012Metric
- removed the C34 at (135.1, 352.9)
- removed C43: 2.2uF, Capacitor_SMD:C_0805_2012Metric
- removed C46, C47, C48, C49: 470pF, Capacitor_SMD:C_0805_2012Metric
- removed C50: 10u, Capacitor_SMD:C_0805_2012Metric
- removed C51, C52, C53, C54, C55, C56, C57, C58: 10nF, Capacitor_SMD:C_0805_2012Metric
- removed C60: 3.3nF, Capacitor_SMD:C_0805_2012Metric
- removed C61: 47uF, Capacitor_SMD:C_0805_2012Metric
- removed C62, C7: 0.1uF, Capacitor_SMD:C_0805_2012Metric
- removed D43: ESDA6V1BC6, Package_TO_SOT_SMD:SOT-23-6
- removed the FB1 at (148.5, 346.8)
- removed FB2, FB3, FB4, FB5, FB6: 600Ohm@100MHz, Inductor_SMD:L_0805_2012Metric
- removed LS1: SpeakerL, TerminalBlock_Phoenix:TerminalBlock_Phoenix_MKDS-1,5-2-5.08_1x02_P5.08mm_Horizontal
- removed LS2: SpeakerR, TerminalBlock_Phoenix:TerminalBlock_Phoenix_MKDS-1,5-2-5.08_1x02_P5.08mm_Horizontal
- removed R1, R4: 5.1k, Resistor_SMD:R_0805_2012Metric
- removed R10, R11, R12, R13, R14, R15, R16, R17, R18, R19, R20, R21, R22, R23, R24, R25, R30, R33: 10k, Resistor_SMD:R_0805_2012Metric
- removed R26: 220, Resistor_SMD:R_0805_2012Metric
- removed R27: 10, Resistor_SMD:R_0805_2012Metric
- removed R28: 33, Resistor_SMD:R_0805_2012Metric
- removed R29: 681 @ 1%, Resistor_SMD:R_0805_2012Metric
- removed R31: 2.2k @ 1%, Resistor_SMD:R_0805_2012Metric
- removed R32: 49.9k @ 1%, Resistor_SMD:R_0805_2012Metric
- removed R34, R35: 56k, Resistor_SMD:R_0805_2012Metric
- removed the R5 at (166.6, 327.4)
- removed R6: 390k, Resistor_SMD:R_0805_2012Metric
- removed the R7 at (153.0, 350.9)
- removed the R8 at (153.0, 353.9)
- removed R9: 2.2k, Resistor_SMD:R_0805_2012Metric
- removed TP1: LDO_IN, TestPoint:TestPoint_Pad_D2.0mm
- removed TP10: HPR, TestPoint:TestPoint_Pad_D2.0mm
- removed TP11: HPL, TestPoint:TestPoint_Pad_D2.0mm
- removed TP12: JACKSENSE, TestPoint:TestPoint_Pad_D2.0mm
- removed TP13: RECP, TestPoint:TestPoint_Pad_D2.0mm
- removed TP14: RECN, TestPoint:TestPoint_Pad_D2.0mm
- removed TP15: SPKLP, TestPoint:TestPoint_Pad_D2.0mm
- removed TP16: SPKLN, TestPoint:TestPoint_Pad_D2.0mm
- removed TP17: SPKRP, TestPoint:TestPoint_Pad_D2.0mm
- removed TP18: SPKRN, TestPoint:TestPoint_Pad_D2.0mm
- removed TP2: LDO_OUT, TestPoint:TestPoint_Pad_D2.0mm
- removed TP3: MICBIAS, TestPoint:TestPoint_Pad_D2.0mm
- removed TP4: INA1, TestPoint:TestPoint_Pad_D2.0mm
- removed TP5: INA2, TestPoint:TestPoint_Pad_D2.0mm
- removed TP6: CODEC_MCLK, TestPoint:TestPoint_Pad_D2.0mm
- removed TP7: MIC2P, TestPoint:TestPoint_Pad_D2.0mm
- removed TP8: MIC2N, TestPoint:TestPoint_Pad_D2.0mm
- removed TP9: HPSNS, TestPoint:TestPoint_Pad_D2.0mm
- removed the U5 at (282.8, 112.8)
- removed U6: MAX98089ETN_T, ledaw:MAX98089ETN_T
- removed Y2: 12.288MHz, Oscillator:Oscillator_SMD_SeikoEpson_SG210-4Pin_2.5x2.0mm
- moved J5 0.51 mm to (297.2, 88.0)
- moved J6 0.50 mm to (277.5, 88.0)
- renumbered C6 to C23, C3 to C25, C12 to C30, C13 to C31, C16 to C34, R1 to R7, R4 to R8, U2 to U5

Commit message: reannoation with good linkage?
Parts:
- removed C10, C11, C15, C18, C19, C21, C25, C31, C34: 1uF, Capacitor_SMD:C_0805_2012Metric
- removed C14, C17, C26, C27: 10uF, Capacitor_SMD:C_0805_2012Metric
- removed C23, C30: 100nF, Capacitor_SMD:C_0805_2012Metric
- removed FB1: 600Ohm@100MHz, Inductor_SMD:L_0805_2012Metric
- removed R5: 2.2k, Resistor_SMD:R_0805_2012Metric
- removed R7, R8: 10k, Resistor_SMD:R_0805_2012Metric
- removed U4: MAX98089ETN_T, footprints:MAX98089ETN_T
- removed U5: TPS7A20xxxDBV, Package_TO_SOT_SMD:SOT-23-5
- removed Y1: 12.288MHz, Oscillator:Oscillator_SMD_SeikoEpson_SG210-4Pin_2.5x2.0mm
- added C101: 47uF, Capacitor_SMD:C_0805_2012Metric, F.Cu at (236.6, 261.1)
- added C201: 10uF, Capacitor_SMD:C_0805_2012Metric, F.Cu at (213.8, 239.6)
- added C202: 100nF, Capacitor_SMD:C_0805_2012Metric, F.Cu at (209.4, 227.5)
- added C203: 10uF, Capacitor_SMD:C_0805_2012Metric, F.Cu at (213.8, 230.5)
- added C204: 100nF, Capacitor_SMD:C_0805_2012Metric, F.Cu at (213.8, 224.5)
- added C205: 1uF, Capacitor_SMD:C_0805_2012Metric, F.Cu at (213.8, 227.5)
- added C206: 1uF, Capacitor_SMD:C_0805_2012Metric, F.Cu at (213.8, 233.6)
- added C207: 1uF, Capacitor_SMD:C_0805_2012Metric, F.Cu at (213.8, 236.6)
- added C208: 1uF, Capacitor_SMD:C_0805_2012Metric, F.Cu at (218.3, 218.5)
- added C209: 1uF, Capacitor_SMD:C_0805_2012Metric, F.Cu at (218.3, 227.5)
- added C210: 100nF, Capacitor_SMD:C_0805_2012Metric, F.Cu at (218.3, 233.6)
- added C211: 470pF, Capacitor_SMD:C_0805_2012Metric, F.Cu at (222.7, 224.5)
- added C212: 100nF, Capacitor_SMD:C_0805_2012Metric, F.Cu at (209.4, 218.5)
- added C213: 10uF, Capacitor_SMD:C_0805_2012Metric, F.Cu at (222.7, 218.5)
- added C214: 470pF, Capacitor_SMD:C_0805_2012Metric, F.Cu at (222.7, 227.5)
- added C215: 10uF, Capacitor_SMD:C_0805_2012Metric, F.Cu at (222.7, 221.5)
- added C216: 1uF, Capacitor_SMD:C_0805_2012Metric, F.Cu at (222.7, 236.6)
- added C217: 100nF, Capacitor_SMD:C_0805_2012Metric, F.Cu at (209.4, 221.5)
- added C218: 1uF, Capacitor_SMD:C_0805_2012Metric, F.Cu at (209.4, 236.6)
- added C219: 1uF, Capacitor_SMD:C_0805_2012Metric, F.Cu at (209.4, 239.6)
- added C220: 470pF, Capacitor_SMD:C_0805_2012Metric, F.Cu at (222.7, 230.5)
- added C221: 1uF, Capacitor_SMD:C_0805_2012Metric, F.Cu at (213.8, 218.5)
- added C222: 1uF, Capacitor_SMD:C_0805_2012Metric, F.Cu at (213.8, 221.5)
- added C223: 470pF, Capacitor_SMD:C_0805_2012Metric, F.Cu at (222.7, 233.6)
- added C224: 1uF, Capacitor_SMD:C_0805_2012Metric, F.Cu at (218.3, 236.6)
- added C225: 2.2uF, Capacitor_SMD:C_0805_2012Metric, F.Cu at (218.3, 239.6)
- added C226: 1uF, Capacitor_SMD:C_0805_2012Metric, F.Cu at (218.3, 221.5)
- added C227: 1uF, Capacitor_SMD:C_0805_2012Metric, F.Cu at (218.3, 224.5)
- added C228: 1uF, Capacitor_SMD:C_0805_2012Metric, F.Cu at (218.3, 230.5)
- added C229: 1uF, Capacitor_SMD:C_0805_2012Metric, F.Cu at (209.4, 224.5)
- added C230: 1uF, Capacitor_SMD:C_0805_2012Metric, F.Cu at (209.4, 233.6)
- added C231: 47pF, Capacitor_SMD:C_0805_2012Metric, F.Cu at (209.4, 230.5)
- added C304: 100n, Capacitor_SMD:C_0402_1005Metric, F.Cu at (209.7, 275.6)
- added C305: 100n, Capacitor_SMD:C_0402_1005Metric, F.Cu at (209.7, 277.6)
- added C306: 100n, Capacitor_SMD:C_0402_1005Metric, F.Cu at (209.7, 279.6)
- added C307: 100n, Capacitor_SMD:C_0402_1005Metric, F.Cu at (212.5, 275.6)
- added C308: 100n, Capacitor_SMD:C_0402_1005Metric, F.Cu at (212.5, 277.6)
- added C309: 100n, Capacitor_SMD:C_0402_1005Metric, F.Cu at (212.5, 279.6)
- added C310: 100n, Capacitor_SMD:C_0402_1005Metric, F.Cu at (215.4, 275.6)
- added C311: 100n, Capacitor_SMD:C_0402_1005Metric, F.Cu at (215.4, 277.6)
- added C312: 100n, Capacitor_SMD:C_0402_1005Metric, F.Cu at (215.4, 279.6)
- added C313: 10u, Capacitor_SMD:C_0805_2012Metric, F.Cu at (210.5, 261.1)
- added C317: 10nF, Capacitor_SMD:C_0805_2012Metric, F.Cu at (210.5, 264.1)
- added C318: 10nF, Capacitor_SMD:C_0805_2012Metric, F.Cu at (210.5, 267.1)
- added C319: 10nF, Capacitor_SMD:C_0805_2012Metric, F.Cu at (210.5, 270.1)
- added C320: 10nF, Capacitor_SMD:C_0805_2012Metric, F.Cu at (210.5, 273.1)
- added C321: 10nF, Capacitor_SMD:C_0805_2012Metric, F.Cu at (214.9, 261.1)
- added C322: 10nF, Capacitor_SMD:C_0805_2012Metric, F.Cu at (214.9, 264.1)
- added C323: 10nF, Capacitor_SMD:C_0805_2012Metric, F.Cu at (214.9, 267.1)
- added C324: 10nF, Capacitor_SMD:C_0805_2012Metric, F.Cu at (214.9, 270.1)
- added C327: 100nF, Capacitor_SMD:C_0805_2012Metric, F.Cu at (214.9, 273.1)
- added C501: 10uF, Capacitor_SMD:C_0805_2012Metric, F.Cu at (230.2, 273.1)
- added C502: 0.1uF, Capacitor_SMD:C_0805_2012Metric, F.Cu at (230.2, 270.1)
- added C503: 0.1uF, Capacitor_SMD:C_0805_2012Metric, F.Cu at (230.2, 264.1)
- added C504: 1uF, Capacitor_SMD:C_0805_2012Metric, F.Cu at (230.2, 261.1)
- added C505: 3.3nF, Capacitor_SMD:C_0805_2012Metric, F.Cu at (230.2, 267.1)
- added D201: ESDA6V1BC6, Package_TO_SOT_SMD:SOT-23-6, F.Cu at (224.1, 243.5)
- added FB201: 600Ohm@100MHz, Inductor_SMD:L_0805_2012Metric, F.Cu at (209.4, 242.5)
- added FB202: 600Ohm@100MHz, Inductor_SMD:L_0805_2012Metric, F.Cu at (209.4, 248.0)
- added FB203: 600Ohm@100MHz, Inductor_SMD:L_0805_2012Metric, F.Cu at (209.4, 250.7)
- added FB204: 600Ohm@100MHz, Inductor_SMD:L_0805_2012Metric, F.Cu at (209.4, 253.5)
- added FB205: 600Ohm@100MHz, Inductor_SMD:L_0805_2012Metric, F.Cu at (209.4, 256.2)
- added FB206: 600Ohm@100MHz, Inductor_SMD:L_0805_2012Metric, F.Cu at (209.4, 245.2)
- added LS201: SpeakerL, TerminalBlock_Phoenix:TerminalBlock_Phoenix_MKDS-1,5-2-5.08_1x02_P5.08mm_Horizontal, F.Cu at (228.5, 223.2)
- added LS202: SpeakerR, TerminalBlock_Phoenix:TerminalBlock_Phoenix_MKDS-1,5-2-5.08_1x02_P5.08mm_Horizontal, F.Cu at (228.5, 235.1)
- added R201: 10k, Resistor_SMD:R_0805_2012Metric, F.Cu at (228.9, 245.5)
- added R202: 2.2k, Resistor_SMD:R_0805_2012Metric, F.Cu at (228.9, 248.5)
- added R203: 10k, Resistor_SMD:R_0805_2012Metric, F.Cu at (228.9, 242.6)
- added R302: 10k, Resistor_SMD:R_0805_2012Metric, F.Cu at (197.2, 261.1)
- added R303: 10k, Resistor_SMD:R_0805_2012Metric, F.Cu at (197.2, 267.0)
- added R304: 10k, Resistor_SMD:R_0805_2012Metric, F.Cu at (197.2, 272.9)
- added R305: 10k, Resistor_SMD:R_0805_2012Metric, F.Cu at (197.2, 278.8)
- added R306: 10k, Resistor_SMD:R_0805_2012Metric, F.Cu at (201.6, 264.0)
- added R307: 10k, Resistor_SMD:R_0805_2012Metric, F.Cu at (201.6, 269.9)
- added R308: 10k, Resistor_SMD:R_0805_2012Metric, F.Cu at (201.6, 275.8)
- added R309: 10k, Resistor_SMD:R_0805_2012Metric, F.Cu at (206.0, 261.1)
- added R310: 10k, Resistor_SMD:R_0805_2012Metric, F.Cu at (197.2, 264.0)
- added R311: 10k, Resistor_SMD:R_0805_2012Metric, F.Cu at (197.2, 269.9)
- added R312: 10k, Resistor_SMD:R_0805_2012Metric, F.Cu at (197.2, 275.8)
- added R313: 10k, Resistor_SMD:R_0805_2012Metric, F.Cu at (201.6, 261.1)
- added R314: 10k, Resistor_SMD:R_0805_2012Metric, F.Cu at (201.6, 267.0)
- added R315: 10k, Resistor_SMD:R_0805_2012Metric, F.Cu at (201.6, 272.9)
- added R316: 10k, Resistor_SMD:R_0805_2012Metric, F.Cu at (201.6, 278.8)
- added R317: 10k, Resistor_SMD:R_0805_2012Metric, F.Cu at (206.0, 264.0)
- added R319: 220, Resistor_SMD:R_0805_2012Metric, F.Cu at (206.0, 267.0)
- added R320: 33, Resistor_SMD:R_0805_2012Metric, F.Cu at (206.0, 272.9)
- added R321: 10, Resistor_SMD:R_0805_2012Metric, F.Cu at (206.0, 269.9)
- added R501: 56k, Resistor_SMD:R_0805_2012Metric, F.Cu at (225.7, 269.9)
- added R502: 49.9k @ 1%, Resistor_SMD:R_0805_2012Metric, F.Cu at (225.7, 264.0)
- added R503: 56k, Resistor_SMD:R_0805_2012Metric, F.Cu at (225.7, 272.9)
- added R504: 10k, Resistor_SMD:R_0805_2012Metric, F.Cu at (225.7, 267.0)
- added R505: 2.2k @ 1%, Resistor_SMD:R_0805_2012Metric, F.Cu at (225.7, 261.1)
- added R506: 10k, Resistor_SMD:R_0805_2012Metric, F.Cu at (221.3, 275.8)
- added R507: 1M, Resistor_SMD:R_0805_2012Metric, F.Cu at (221.3, 267.0)
- added R508: 390k, Resistor_SMD:R_0805_2012Metric, F.Cu at (221.3, 269.9)
- added R509: 681 @ 1%, Resistor_SMD:R_0805_2012Metric, F.Cu at (221.3, 272.9)
- added R510: 5.1k, Resistor_SMD:R_0805_2012Metric, F.Cu at (221.3, 261.1)
- added R511: 5.1k, Resistor_SMD:R_0805_2012Metric, F.Cu at (221.3, 264.0)
- added TP201: CODEC_MCLK, TestPoint:TestPoint_Pad_D2.0mm, F.Cu at (197.0, 239.3)
- added TP202: SPKLP, TestPoint:TestPoint_Pad_D2.0mm, F.Cu at (205.1, 227.1)
- added TP203: JACKSENSE, TestPoint:TestPoint_Pad_D2.0mm, F.Cu at (201.1, 239.3)
- added TP204: RECP, TestPoint:TestPoint_Pad_D2.0mm, F.Cu at (205.1, 219.0)
- added TP205: SPKLN, TestPoint:TestPoint_Pad_D2.0mm, F.Cu at (205.1, 231.2)
- added TP206: RECN, TestPoint:TestPoint_Pad_D2.0mm, F.Cu at (205.1, 223.1)
- added TP207: MICBIAS, TestPoint:TestPoint_Pad_D2.0mm, F.Cu at (197.0, 227.1)
- added TP208: INA1, TestPoint:TestPoint_Pad_D2.0mm, F.Cu at (197.0, 231.2)
- added TP209: HPR, TestPoint:TestPoint_Pad_D2.0mm, F.Cu at (201.1, 231.2)
- added TP210: SPKRP, TestPoint:TestPoint_Pad_D2.0mm, F.Cu at (205.1, 235.2)
- added TP211: INA2, TestPoint:TestPoint_Pad_D2.0mm, F.Cu at (197.0, 235.2)
- added TP212: HPL, TestPoint:TestPoint_Pad_D2.0mm, F.Cu at (201.1, 235.2)
- added TP213: INA1, TestPoint:TestPoint_Pad_D2.0mm, F.Cu at (201.1, 219.0)
- added TP214: HPSNS, TestPoint:TestPoint_Pad_D2.0mm, F.Cu at (201.1, 227.1)
- added TP215: INA2, TestPoint:TestPoint_Pad_D2.0mm, F.Cu at (201.1, 223.1)
- added TP216: SPKRN, TestPoint:TestPoint_Pad_D2.0mm, F.Cu at (205.1, 239.3)
- added TP217: LDO_IN, TestPoint:TestPoint_Pad_D2.0mm, F.Cu at (197.0, 219.0)
- added TP218: LDO_OUT, TestPoint:TestPoint_Pad_D2.0mm, F.Cu at (197.0, 223.1)
- added U201: MAX98089ETN_T, ledaw:MAX98089ETN_T, F.Cu at (216.9, 245.7)
- added U202: TPS7A20xxxDBV, Package_TO_SOT_SMD:SOT-23-5, F.Cu at (224.1, 248.1)
- added Y201: 12.288MHz, Oscillator:Oscillator_SMD_SeikoEpson_SG210-4Pin_2.5x2.0mm, F.Cu at (233.4, 243.1)
- renumbered C6 to C301, C9 to C302, C10 to C303, C8 to C314, C3 to C315, C5 to C316, C1 to C325, C2 to C326, D42 to D301, D1 to D401, D2 to D402, D3 to D403, D4 to D404, D5 to D405, D6 to D406, D7 to D407, D8 to D408, D9 to D409, D10 to D410, D11 to D411, D12 to D412, D13 to D413, D14 to D414, D15 to D415, D16 to D416, D17 to D417, D18 to D418, D19 to D419, D20 to D420, D21 to D421, D22 to D422, D23 to D423, D24 to D424, D25 to D425, D26 to D426, D27 to D427, D28 to D428, D29 to D429, D30 to D430, D31 to D431, D32 to D432, D33 to D433, D34 to D434, D35 to D435, D36 to D436, D37 to D437, D38 to D438, D39 to D439, D40 to D440, D41 to D441, ENC1 to ENC301, ENC2 to ENC302, ENC3 to ENC303, ENC4 to ENC304, J6 to J201, J7 to J202, J5 to J203, J3 to J301, J4 to J302, J8 to J501, J1 to J502, L1 to L301, MK1 to MK201, MK2 to MK202, Module1 to Module101, P1 to P501, R3 to R301, R2 to R318, SW1 to SW401, SW2 to SW402, SW3 to SW403, SW4 to SW404, SW5 to SW405, SW6 to SW406, SW7 to SW407, SW8 to SW408, SW9 to SW409, SW10 to SW410, SW11 to SW411, SW12 to SW412, SW13 to SW413, SW14 to SW414, SW15 to SW415, SW16 to SW416, SW17 to SW417, SW18 to SW418, SW19 to SW419, SW20 to SW420, SW21 to SW421, SW22 to SW422, SW23 to SW423, SW24 to SW424, SW25 to SW425, SW26 to SW426, SW27 to SW427, SW28 to SW428, SW29 to SW429, SW30 to SW430, SW31 to SW431, SW32 to SW432, SW33 to SW433, SW34 to SW434, SW35 to SW435, SW36 to SW436, SW37 to SW437, SW38 to SW438, SW39 to SW439, SW40 to SW440, SW41 to SW441, U3 to U101, U2 to U301, U4 to U302, U7 to U303, U8 to U304, U10 to U501, U9 to U502, U1 to U503, Y1 to Y301
Connections:
- J202 pad S: /audio/JackS -> /audio/JACKSENSE
Routing:
- net /GPIO3/SCL1: track 36.6 -> 0.00 mm, vias 1 -> 0
- net /GPIO2/SDA1: track 36.3 -> 0.00 mm, vias 1 -> 0
- net GND: track 39.3 -> 3.53 mm, vias 30 -> 5
- net /codec/DIGMICDATA: track 29.8 -> 0.00 mm, vias 1 -> 0
- net +1V8: track 28.7 -> 0.00 mm, vias 5 -> 0
- net /codec/DIGMICCLK: track 28.7 -> 0.00 mm, vias 1 -> 0
- net /codec/JackS: track 23.1 -> 0.00 mm, vias 2 -> 0
- net /GPIO25: track 15.6 -> 0.00 mm, vias 2 -> 0
- net Net-(U4-MIC2N): track 15.0 -> 0.00 mm
- net Net-(U4-INA1/EXTMICP): track 13.1 -> 0.00 mm, vias 2 -> 0
- net Net-(U4-MIC2P): track 13.1 -> 0.00 mm
- net /GPIO18/PCM.CLK: track 12.5 -> 0.00 mm, vias 1 -> 0
- net /GPIO19/PCM.FS: track 11.0 -> 0.00 mm, vias 1 -> 0
- net /GPIO21/PCM.DOUT: track 10.6 -> 0.00 mm, vias 1 -> 0
- net Net-(U4-INA2/EXTMICN): track 10.3 -> 0.00 mm, vias 2 -> 0
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- removed copper zone on B.Cu, net +5V

Commit message: successfully got hat in?
Parts:
- added J101: CM4_DEBUG, Connector_PinSocket_2.54mm:PinSocket_2x20_P2.54mm_Vertical, B.Cu at (191.5, 221.9)
- added J102: DEBUG_PORT, Connector_PinHeader_2.54mm:PinHeader_1x03_P2.54mm_Vertical, F.Cu at (186.7, 227.9)
- added J201: LineOut, Connector_Audio:Jack_3.5mm_CUI_SJ-3523-SMT_Horizontal, F.Cu at (200.1, 263.6)
- added J202: LineIn, Connector_Audio:Jack_3.5mm_CUI_SJ-3523-SMT_Horizontal, F.Cu at (223.1, 263.6)
- added J203: Headphone, footprints:CUI_SJ-43514-SMT-TR, F.Cu at (215.2, 270.5)
- added JP101: ID_WP, Jumper:SolderJumper-2_P1.3mm_Open_RoundedPad1.0x1.5mm, B.Cu at (231.7, 240.2)
- added MH1: MountingHole_2.7mm_M2.5, MountingHole:MountingHole_2.7mm_M2.5, F.Cu at (186.6, 220.6)
- added MH2: MountingHole_2.7mm_M2.5, MountingHole:MountingHole_2.7mm_M2.5, F.Cu at (244.6, 220.6)
- added MH3: MountingHole_2.7mm_M2.5, MountingHole:MountingHole_2.7mm_M2.5, F.Cu at (186.6, 269.6)
- added MH4: MountingHole_2.7mm_M2.5, MountingHole:MountingHole_2.7mm_M2.5, F.Cu at (244.6, 269.6)
- added MK201: MicL, Sensor_Audio:Knowles_LGA-5_3.5x2.65mm, F.Cu at (245.1, 233.6)
- added MK202: MicR, Sensor_Audio:Knowles_LGA-5_3.5x2.65mm, F.Cu at (245.1, 257.6)
- added R101: 3.9k, Resistor_SMD:R_0805_2012Metric, F.Cu at (231.7, 236.3)
- added R102: 3.9k, Resistor_SMD:R_0805_2012Metric, F.Cu at (231.7, 234.2)
- added TP101: 5V, TestPoint:TestPoint_THTPad_1.5x1.5mm_Drill0.7mm, F.Cu at (196.8, 226.8)
- added TP102: GND, TestPoint:TestPoint_THTPad_1.5x1.5mm_Drill0.7mm, F.Cu at (196.8, 229.5)
- added U101: Oled, Connector_PinHeader_2.54mm:PinHeader_1x07_P2.54mm_Vertical, F.Cu at (239.5, 241.8)
- added U102: CAT24C256, Package_SO:SOIC-8_3.9x4.9mm_P1.27mm, F.Cu at (231.7, 240.2)
- C201, C203, C204, C205, C206, C207, C208, C209, C210, C224, C225, C226, C227, C228, R201, R202: moved to B.Cu
- moved R316 92.6 mm to (272.8, 219.5)
- moved C501 85.6 mm to (296.9, 219.5)
- moved R312 85.5 mm to (268.4, 228.3)
- moved R509 85.5 mm to (292.5, 225.4)
- moved R507 85.5 mm to (292.5, 219.5)
- moved R508 85.5 mm to (292.5, 222.4)
- moved R311 83.9 mm to (268.4, 225.4)
- moved R305 83.7 mm to (264.0, 228.3)
- moved R310 82.4 mm to (268.4, 222.4)
- moved C502 82.0 mm to (296.9, 222.5)
- moved R304 81.9 mm to (264.0, 225.4)
- moved R320 80.2 mm to (272.8, 228.3)
- moved R303 80.2 mm to (264.0, 222.4)
- moved R501 80.2 mm to (288.1, 219.5)
- moved C231 79.2 mm to (288.1, 239.2)
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Routing:
- net GND: track 3.53 -> 93.5 mm, vias 5 -> 46
- net /codec/JackS: track 0.00 -> 63.6 mm
- net Net-(D201-TVS1): track 0.00 -> 60.5 mm, vias 0 -> 2
- net /audio/DIGMICDATA: track 0.00 -> 55.9 mm, vias 0 -> 3
- net /audio/DIGMICCLK: track 0.00 -> 55.8 mm, vias 0 -> 2
- net Net-(D201-TVS2): track 0.00 -> 47.1 mm
- net /GPIO2/SDA1: track 0.00 -> 44.7 mm
- net /I2C1_SCL: track 0.00 -> 44.1 mm, vias 0 -> 1
- net +3V3: track 0.00 -> 42.3 mm, vias 0 -> 7
- net /PCM_DOUT: track 0.00 -> 37.2 mm, vias 0 -> 4
- net +1V8: track 0.00 -> 34.9 mm, vias 0 -> 7
- net /PCM_FS: track 0.00 -> 33.4 mm, vias 0 -> 2
- net /GPIO10/SPI0.MOSI: track 0.00 -> 31.3 mm, vias 0 -> 1
- net /PCM_DIN: track 0.00 -> 30.5 mm, vias 0 -> 2
- net Net-(C215-Pad2): track 0.00 -> 28.4 mm
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- added copper zone on In2.Cu, net +1V8
- added copper zone on In2.Cu, net +3V3
- added copper zone on F.Cu, net +5V
- added copper zone on In2.Cu, net +5V
Other:
- board size 300 x 120 mm -> 300 x 189.6 mm
- board text added: "PoE"
- board text added: "RJ45"
