File: hardware/board/board.kicad_sch (KiCad schematic)
At the start: 6 parts, among them J101 CM4_DEBUG, J102 DEBUG_PORT, J103 UART, U101 Oled

Commit message: i think this is finally right
Parts:
- renumbered J103 to J101, J101 to J102, J102 to J103
Changed lines of the file:
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@@
 		(in_pos_files yes)
 		(dnp no)
-		(property "Reference" "J103"
+		(property "Reference" "J101"
 			(at 257.302 97.536 0)
 			(show_name no)
@@
 			(project "board"
 				(path "/dd13fd41-39ab-4435-9074-5024f1786746"
-					(reference "J103")
+					(reference "J101")
 					(unit 1)
 				)
@@
 		(in_pos_files yes)
 		(dnp no)
-		(property "Reference" "J101"
+		(property "Reference" "J102"
 			(at 266.192 115.316 0)
 			(show_name no)
@@
 			(project "board"
 				(path "/dd13fd41-39ab-4435-9074-5024f1786746"
-					(reference "J101")
+					(reference "J102")
 					(unit 1)
 				)
@@
 		(dnp no)
 		(fields_autoplaced yes)
-		(property "Reference" "J102"
+		(property "Reference" "J103"
 			(at 266.065 133.35 0)
 			(show_name no)
@@
 			(project "board"
 				(path "/dd13fd41-39ab-4435-9074-5024f1786746"
-					(reference "J102")
+					(reference "J103")
 					(unit 1)
 				)

Commit message: progress on audio
Connections:
- net CODEC_~{IRQ}: now also Module101.54 (GPIO4); no longer Module101.41 (GPIO25)
Changed lines of the file:
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@@
+	(wire
+		(pts
+			(xy 138.43 113.03) (xy 152.4 113.03)
+		)
+		(stroke
+			(width 0)
+			(type default)
+		)
+	)
 	(wire
 		(pts
@@
 		(pts
 			(xy 31.75 170.18) (xy 31.75 175.26)
-		)
-		(stroke
-			(width 0)
-			(type default)
-		)
-	)
-	(wire
-		(pts
-			(xy 227.33 97.79) (xy 213.36 97.79)
 		)
 		(stroke
@@
 		)
 	)
-	(label "CODEC_~{IRQ}"
-		(at 227.33 97.79 180)
-		(effects
-			(font
-				(size 1.27 1.27)
-			)
-			(justify right bottom)
-		)
-	)
 	(label "USB2_P"
 		(at 111.76 53.34 180)
@@
 		)
 	)
+	(label "CODEC_~{IRQ}"
+		(at 138.43 113.03 0)
+		(effects
+			(font
+				(size 1.27 1.27)
+			)
+			(justify left bottom)
+		)
+	)

Commit message: big routing board
Parts:
- J101, J102, J103: footprint (none) -> Connector_PinHeader_1.27mm:PinHeader_1x03_P1.27mm_Vertical
Changed lines of the file:
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@@
 			)
 		)
-		(property "Footprint" ""
+		(property "Footprint" "Connector_PinHeader_1.27mm:PinHeader_1x03_P1.27mm_Vertical"
 			(at 260.35 105.41 0)
 			(hide yes)
@@
 			)
 		)
-		(property "Footprint" ""
+		(property "Footprint" "Connector_PinHeader_1.27mm:PinHeader_1x03_P1.27mm_Vertical"
 			(at 269.24 123.19 0)
 			(hide yes)
@@
 			)
 		)
-		(property "Footprint" ""
+		(property "Footprint" "Connector_PinHeader_1.27mm:PinHeader_1x03_P1.27mm_Vertical"
 			(at 265.43 140.97 0)
 			(hide yes)

Commit message: usb
Parts:
- added C102, C103: 22uF X5R 16V, Capacitor_SMD:C_1206_3216Metric, symbol Device:C_Small
- C101: value 47uF -> 22uF X5R 16V; footprint Capacitor_SMD:C_0805_2012Metric -> Capacitor_SMD:C_1206_3216Metric
Connections:
- net +5V: now also C102.1, C103.1
- net GND: now also C102.2, C103.2
Other:
- moved on the sheet: C101

Commit message: loose ends
Parts:
- added JP101: Jumper_SWCLK_Open, Jumper:SolderJumper-2_P1.3mm_Open_TrianglePad1.0x1.5mm, symbol Jumper:Jumper_2_Open
- added JP102: Jumper_SWD_Open, Jumper:SolderJumper-2_P1.3mm_Open_TrianglePad1.0x1.5mm, symbol Jumper:Jumper_2_Open
Connections:
- net MCU_SWCLK: now also JP101.1 (A)
- net MCU_SWD: now also JP102.1 (A)
- net SWCLK: now also JP101.2 (B)
- net SWD: now also JP102.2 (B)
Other:
- moved on the sheet: J102, J103

Commit message: swd swclk run
Connections:
- net MCU_SWCLK: now also JP101.2 (B); no longer JP101.1 (A)
- net MCU_SWD: now also JP102.2 (B); no longer JP102.1 (A)
- net SWCLK: now also JP101.1 (A); no longer JP101.2 (B)
- net SWD: now also JP102.1 (A); no longer JP102.2 (B)
Other:
- moved on the sheet: JP101, JP102
Changed lines of the file:
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@@
 		(lib_id "Jumper:Jumper_2_Open")
 		(at 276.86 128.27 0)
-		(mirror y)
+		(mirror x)
 		(unit 1)
 		(body_style 1)
@@
 		(dnp no)
 		(property "Reference" "JP102"
-			(at 276.86 130.556 0)
+			(at 276.86 134.874 0)
 			(show_name no)
 			(do_not_autoplace no)
@@
 		)
 		(property "Value" "Jumper_SWD_Open"
-			(at 276.86 133.096 0)
+			(at 276.86 132.334 0)
 			(show_name no)
 			(do_not_autoplace no)
@@
 	(symbol
 		(lib_id "Jumper:Jumper_2_Open")
-		(at 276.86 123.19 180)
+		(at 276.86 123.19 0)
 		(unit 1)
 		(body_style 1)
@@
 		(dnp no)
 		(property "Reference" "JP101"
-			(at 276.86 117.602 0)
+			(at 276.86 113.792 0)
 			(show_name no)
 			(do_not_autoplace no)
@@
 		)
 		(property "Value" "Jumper_SWCLK_Open"
-			(at 276.86 115.316 0)
-			(show_name no)
-			(do_not_autoplace no)
+			(at 276.86 116.078 0)
+			(show_name no)
+			(do_not_autoplace no)

Commit message: finish swd, usb status, starting uart out and rp2350 remap?
Connections:
- net RST: now also Module101.36 (ID_SD)
- net USBH_EN: now also Module101.40 (GPIO9); no longer Module101.45 (GPIO24)
Changed lines of the file:
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@@
+	(wire
+		(pts
+			(xy 139.7 90.17) (xy 152.4 90.17)
+		)
+		(stroke
+			(width 0)
+			(type default)
+		)
+	)
 	(wire
 		(pts
@@
 	(wire
 		(pts
+			(xy 138.43 95.25) (xy 152.4 95.25)
+		)
+		(stroke
+			(width 0)
+			(type default)
+		)
+	)
+	(wire
+		(pts
 			(xy 213.36 143.51) (xy 218.44 143.51)
 		)
@@
 		(pts
 			(xy 247.65 167.64) (xy 260.35 167.64)
-		)
-		(stroke
-			(width 0)
-			(type default)
-		)
-	)
-	(wire
-		(pts
-			(xy 227.33 102.87) (xy 213.36 102.87)
 		)
 		(stroke
@@
 		)
 	)
+	(label "USBH_EN"
+		(at 138.43 95.25 0)
+		(effects
+			(font
+				(size 1.27 1.27)
+			)
+			(justify left bottom)
+		)
+	)
 	(label "MCU_SWCLK"
 		(at 304.8 123.19 180)
@@
 		)
 	)
+	(label "RST"
+		(at 139.7 90.17 0)
+		(effects
+			(font
+				(size 1.27 1.27)
+			)
+			(justify left bottom)
+		)
+	)
 	(label "I2C1_SDA"
 		(at 139.7 118.11 0)
@@
 		(effects
 			(font
-				(size 1.27 1.27)
-			)
-			(justify right bottom)
-		)
-	)
-	(label "USBH_EN"
-		(at 227.33 102.87 180)
-		(effects
-			(font
