File: hardware/board/buttons.kicad_sch (KiCad schematic)
At the start: 84 parts, among them SW10 SW_Push, SW11 SW_Push, SW12 SW_Push, SW13 SW_Push, SW14 SW_Push, SW15 SW_Push, SW16 SW_Push, SW17 SW_Push, SW18 SW_Push, SW19 SW_Push, SW20 SW_Push, SW21 SW_Push, SW22 SW_Push, SW23 SW_Push, SW24 SW_Push, SW25 SW_Push, SW26 SW_Push, SW27 SW_Push, SW28 SW_Push, SW29 SW_Push, SW30 SW_Push, SW31 SW_Push, SW32 SW_Push, SW33 SW_Push, SW34 SW_Push, SW35 SW_Push, SW36 SW_Push, SW37 SW_Push, SW38 SW_Push, SW39 SW_Push, SW40 SW_Push, SW41 SW_Push, SW42 SW_Push, SW43 SW_Push, SW44 SW_Push, SW45 SW_Push, SW46 SW_Push, SW5 SW_Push, SW6 SW_Push, SW7 SW_Push, SW8 SW_Push, SW9 SW_Push

Commit message: add hella parts
Parts:
- SW10: renamed from SW8; footprint Button_Switch_THT:SW_PUSH-12mm -> ledaw:ks-33-2.0
- SW11: footprint Button_Switch_THT:SW_PUSH-12mm -> ledaw:ks-33-2.0
- SW12: renamed from SW16; footprint Button_Switch_THT:SW_PUSH-12mm -> ledaw:ks-33-2.0
- SW13: renamed from SW21; footprint Button_Switch_THT:SW_PUSH-12mm -> ledaw:ks-33-2.0
- SW14: renamed from SW41; footprint Button_Switch_THT:SW_PUSH-12mm -> ledaw:ks-33-2.0
- SW15: renamed from SW9; footprint Button_Switch_THT:SW_PUSH-12mm -> ledaw:ks-33-2.0
- SW16: renamed from SW12; footprint Button_Switch_THT:SW_PUSH-12mm -> ledaw:ks-33-2.0
- SW17: renamed from SW13; footprint Button_Switch_THT:SW_PUSH-12mm -> ledaw:ks-33-2.0
- SW18: renamed from SW17; footprint Button_Switch_THT:SW_PUSH-12mm -> ledaw:ks-33-2.0
- SW19: renamed from SW22; footprint Button_Switch_THT:SW_PUSH-12mm -> ledaw:ks-33-2.0
- SW20: renamed from SW42; footprint Button_Switch_THT:SW_PUSH-12mm -> ledaw:ks-33-2.0
- SW21: renamed from SW14; footprint Button_Switch_THT:SW_PUSH-12mm -> ledaw:ks-33-2.0
- SW22: renamed from SW18; footprint Button_Switch_THT:SW_PUSH-12mm -> ledaw:ks-33-2.0
- SW23: renamed from SW19; footprint Button_Switch_THT:SW_PUSH-12mm -> ledaw:ks-33-2.0
- SW24: renamed from SW23; footprint Button_Switch_THT:SW_PUSH-12mm -> ledaw:ks-33-2.0
- SW25: renamed from SW24; footprint Button_Switch_THT:SW_PUSH-12mm -> ledaw:ks-33-2.0
- SW26: renamed from SW43; footprint Button_Switch_THT:SW_PUSH-12mm -> ledaw:ks-33-2.0
- SW27: renamed from SW25; footprint Button_Switch_THT:SW_PUSH-12mm -> ledaw:ks-33-2.0
- SW28: renamed from SW26; footprint Button_Switch_THT:SW_PUSH-12mm -> ledaw:ks-33-2.0
- SW29: renamed from SW27; footprint Button_Switch_THT:SW_PUSH-12mm -> ledaw:ks-33-2.0
- SW3: renamed from SW5; footprint Button_Switch_THT:SW_PUSH-12mm -> ledaw:ks-33-2.0
- SW30: renamed from SW28; footprint Button_Switch_THT:SW_PUSH-12mm -> ledaw:ks-33-2.0
- SW31: renamed from SW29; footprint Button_Switch_THT:SW_PUSH-12mm -> ledaw:ks-33-2.0
- SW32: renamed from SW44; footprint Button_Switch_THT:SW_PUSH-12mm -> ledaw:ks-33-2.0
- SW33: renamed from SW30; footprint Button_Switch_THT:SW_PUSH-12mm -> ledaw:ks-33-2.0
- SW34: renamed from SW31; footprint Button_Switch_THT:SW_PUSH-12mm -> ledaw:ks-33-2.0
- SW35: renamed from SW32; footprint Button_Switch_THT:SW_PUSH-12mm -> ledaw:ks-33-2.0
- SW36: renamed from SW33; footprint Button_Switch_THT:SW_PUSH-12mm -> ledaw:ks-33-2.0
- SW37: renamed from SW34; footprint Button_Switch_THT:SW_PUSH-12mm -> ledaw:ks-33-2.0
- SW38: renamed from SW45; footprint Button_Switch_THT:SW_PUSH-12mm -> ledaw:ks-33-2.0
- SW39: renamed from SW35; footprint Button_Switch_THT:SW_PUSH-12mm -> ledaw:ks-33-2.0
- SW4: renamed from SW6; footprint Button_Switch_THT:SW_PUSH-12mm -> ledaw:ks-33-2.0
- SW40: renamed from SW36; footprint Button_Switch_THT:SW_PUSH-12mm -> ledaw:ks-33-2.0
- SW41: renamed from SW37; footprint Button_Switch_THT:SW_PUSH-12mm -> ledaw:ks-33-2.0
- SW42: renamed from SW38; footprint Button_Switch_THT:SW_PUSH-12mm -> ledaw:ks-33-2.0
- SW43: renamed from SW39; footprint Button_Switch_THT:SW_PUSH-12mm -> ledaw:ks-33-2.0
- SW44: renamed from SW46; footprint Button_Switch_THT:SW_PUSH-12mm -> ledaw:ks-33-2.0
- SW5: renamed from SW10; footprint Button_Switch_THT:SW_PUSH-12mm -> ledaw:ks-33-2.0
- SW6: renamed from SW15; footprint Button_Switch_THT:SW_PUSH-12mm -> ledaw:ks-33-2.0
- SW7: renamed from SW20; footprint Button_Switch_THT:SW_PUSH-12mm -> ledaw:ks-33-2.0
- SW8: renamed from SW40; footprint Button_Switch_THT:SW_PUSH-12mm -> ledaw:ks-33-2.0
- SW9: renamed from SW7; footprint Button_Switch_THT:SW_PUSH-12mm -> ledaw:ks-33-2.0
- renumbered D16 to D10, D21 to D11, D37 to D12, D3 to D13, D7 to D14, D12 to D15, D17 to D16, D22 to D17, D38 to D18, D4 to D19, D5 to D2, D8 to D20, D13 to D21, D18 to D22, D39 to D24, D9 to D25, D14 to D26, D19 to D27, D24 to D28, D25 to D29, D10 to D3, D40 to D30, D26 to D31, D27 to D32, D28 to D33, D29 to D34, D30 to D35, D41 to D36, D31 to D37, D32 to D38, D33 to D39, D15 to D4, D34 to D40, D35 to D41, D20 to D5, D36 to D6, D2 to D7, D6 to D8, D11 to D9
Connections:
- net io_C0 renamed matrix_C0
- net io_C1 renamed matrix_C1
- net io_C2 renamed matrix_C2
- net io_C3 renamed matrix_C3
- net io_C4 renamed matrix_C4
- net io_C5 renamed matrix_C5
- net io_C6 renamed matrix_C6
- net io_R0 renamed matrix_R0
- net io_R1 renamed matrix_R1
- net io_R2 renamed matrix_R2
- net io_R3 renamed matrix_R3
- net io_R4 renamed matrix_R4
- net io_R5 renamed matrix_R5

Commit message: hella footprints and trying out layouts
Parts:
- removed D42: LL4148, Diode_SMD:D_MiniMELF, symbol Diode:LL4148
- removed SW44: SW_Push, ledaw:ks-33-2.0, symbol Switch:SW_Push
Connections:
- net matrix_R5 is gone; now on net matrix_C6: SW14.1, SW20.1, SW26.1, SW32.1, SW38.1, SW8.1
Changed lines of the file:
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@@
 	)
 	(junction
+		(at 250.19 124.46)
+		(diameter 0)
+		(color 0 0 0 0)
+	)
+	(junction
 		(at 250.19 81.28)
 		(diameter 0)
@@
 	)
 	(junction
-		(at 250.19 124.46)
-		(diameter 0)
-		(color 0 0 0 0)
-	)
-	(junction
 		(at 86.36 85.09)
 		(diameter 0)
@@
 	(wire
 		(pts
+			(xy 250.19 124.46) (xy 250.19 129.54)
+		)
+		(stroke
+			(width 0)
+			(type default)
+		)
+	)
+	(wire
+		(pts
 			(xy 58.42 109.22) (xy 59.69 109.22)
 		)
@@
 	(wire
 		(pts
-			(xy 226.06 129.54) (xy 198.12 129.54)
+			(xy 198.12 129.54) (xy 250.19 129.54)
 		)
 		(stroke
@@
 	(wire
 		(pts
-			(xy 226.06 139.7) (xy 226.06 129.54)
-		)
-		(stroke
-			(width 0)
-			(type default)
-		)
-	)
-	(wire
-		(pts
 			(xy 191.77 124.46) (xy 194.31 124.46)
 		)
@@
 	(wire
 		(pts
-			(xy 247.65 139.7) (xy 250.19 139.7)
-		)
-		(stroke
-			(width 0)
-			(type default)
-		)
-	)
-	(wire
-		(pts
 			(xy 170.18 95.25) (xy 170.18 85.09)
 		)
@@
 	(wire
 		(pts
-			(xy 227.33 139.7) (xy 226.06 139.7)
-		)
-		(stroke
-			(width 0)
-			(type default)
-		)
-	)
-	(wire
-		(pts
 			(xy 114.3 95.25) (xy 114.3 85.09)
 		)
@@
 	(wire
 		(pts
-			(xy 250.19 124.46) (xy 250.19 139.7)
-		)
-		(stroke
-			(width 0)
-			(type default)
-		)
-	)
-	(wire
-		(pts
 			(xy 198.12 71.12) (xy 198.12 81.28)
 		)
@@
 	(wire
 		(pts
-			(xy 237.49 139.7) (xy 240.03 139.7)
-		)
-		(stroke
-			(width 0)
-			(type default)
-		)
-	)
-	(wire
-		(pts
 			(xy 191.77 81.28) (xy 194.31 81.28)
 		)
@@
 	(symbol
 		(lib_id "Diode:LL4148")
-		(at 243.84 139.7 180)
-		(unit 1)
-		(body_style 1)
-		(exclude_from_sim no)
-		(in_bom yes)
-		(on_board yes)
-		(in_pos_files yes)
-		(dnp no)
-		(fields_autoplaced yes)
-		(property "Reference" "D42"
-			(at 243.84 133.096 0)
-			(show_name no)
-			(do_not_autoplace no)
-			(effects
-				(font
-					(size 1.27 1.27)
-				)
-			)
-		)
-		(property "Value" "LL4148"
-			(at 243.84 135.636 0)
-			(show_name no)
-			(do_not_autoplace no)
-			(effects
-				(font
-					(size 1.27 1.27)
-				)
-			)
-		)
-		(property "Footprint" "Diode_SMD:D_MiniMELF"
-			(at 243.84 135.255 0)
-			(hide yes)
-			(show_name no)
-			(do_not_autoplace no)
-			(effects
-				(font
-					(size 1.27 1.27)
-				)
-			)
-		)
-		(property "Datasheet" "http://www.vishay.com/docs/85557/ll4148.pdf"
-			(at 243.84 139.7 0)
-			(hide yes)
-			(show_name no)
-			(do_not_autoplace no)
-			(effects
-				(font
-					(size 1.27 1.27)
-				)
-			)
-		)
-		(property "Description" ""
-			(at 243.84 139.7 0)
-			(show_name no)
-			(do_not_autoplace no)
-			(effects
-				(font
-					(size 1.27 1.27)
-				)
-			)
-		)
-		(property "Sim.Device" "D"
-			(at 243.84 139.7 0)
-			(hide yes)
-			(show_name no)
-			(do_not_autoplace no)
-			(effects
-				(font
-					(size 1.27 1.27)
-				)
-			)
-		)
-		(property "Sim.Pins" "1=K 2=A"
-			(at 243.84 139.7 0)
-			(hide yes)
-			(show_name no)
-			(do_not_autoplace no)
-			(effects
-				(font
-					(size 1.27 1.27)
-				)
-			)
-		)
-		(pin "1"
-		)
-		(pin "2"
-		)
-		(instances
-			(project "board"
-				(path "/dd13fd41-39ab-4435-9074-5024f1786746/c4d314f2-7502-4a7f-ae5f-cbca93031f6d/983efcc0-de63-4ee6-a137-eccfc1685d0f"
-					(reference "D42")
-					(unit 1)
-				)
-			)
-		)
-	)
-	(symbol
-		(lib_id "Diode:LL4148")
 		(at 243.84 81.28 180)
 		(unit 1)
@@
 					(unit 1)
 				)
-			)
-		)
-	)
-	(symbol
-		(lib_id "Switch:SW_Push")
-		(at 232.41 139.7 0)
-		(unit 1)
-		(body_style 1)
-		(exclude_from_sim no)
-		(in_bom yes)
-		(on_board yes)
-		(in_pos_files yes)
-		(dnp no)
-		(fields_autoplaced yes)
-		(property "Reference" "SW44"
-			(at 232.41 132.08 0)
-			(show_name no)
-			(do_not_autoplace no)
-			(effects
-				(font
-					(size 1.27 1.27)
-				)
-			)
-		)
-		(property "Value" "SW_Push"
-			(at 232.41 134.62 0)
-			(show_name no)
-			(do_not_autoplace no)
-			(effects
-				(font
-					(size 1.27 1.27)
-				)
-			)
-		)
-		(property "Footprint" "ledaw:ks-33-2.0"
-			(at 232.41 134.62 0)
-			(hide yes)
-			(show_name no)
-			(do_not_autoplace no)
-			(effects
-				(font
-					(size 1.27 1.27)
-				)
-			)
-		)
-		(property "Datasheet" ""
-			(at 232.41 134.62 0)
-			(hide yes)
-			(show_name no)
-			(do_not_autoplace no)
-			(effects
-				(font
-					(size 1.27 1.27)
-				)
-			)
-		)
-		(property "Description" ""
-			(at 232.41 139.7 0)
-			(show_name no)
-			(do_not_autoplace no)
-			(effects
-				(font
-					(size 1.27 1.27)
-				)
-			)
-		)
-		(pin "1"
-		)
-		(pin "2"
-		)
-		(instances
-			(project "board"
-				(path "/dd13fd41-39ab-4435-9074-5024f1786746/c4d314f2-7502-4a7f-ae5f-cbca93031f6d/983efcc0-de63-4ee6-a137-eccfc1685d0f"
-					(reference "SW44")
-					(unit 1)
-				)

Commit message: more placement
Parts:
- removed D30, D36: LL4148, Diode_SMD:D_MiniMELF, symbol Diode:LL4148
- removed SW32, SW38, SW43: SW_Push, ledaw:ks-33-2.0, symbol Switch:SW_Push
- added D39, D40: LL4148, Diode_SMD:D_MiniMELF, symbol Diode:LL4148
- added SW39, SW40, SW41: SW_Push, ledaw:ks-33-2.0, symbol Switch:SW_Push
- renumbered D14 to D10, D20 to D11, D26 to D12, D32 to D13, D38 to D14, D3 to D15, D9 to D16, D15 to D17, D21 to D18, D27 to D19, D7 to D2, D33 to D20, D39 to D21, D5 to D22, D11 to D23, D17 to D24, D23 to D25, D29 to D26, D35 to D27, D4 to D28, D10 to D29, D13 to D3, D16 to D30, D22 to D31, D28 to D32, D34 to D33, D40 to D34, D6 to D35, D12 to D36, D18 to D37, D24 to D38, D19 to D4, D25 to D5, D31 to D6, D37 to D7, D2 to D8, D8 to D9, SW3 to SW1, SW16 to SW10, SW22 to SW11, SW28 to SW12, SW34 to SW13, SW40 to SW14, SW5 to SW15, SW11 to SW16, SW23 to SW18, SW29 to SW19, SW9 to SW2, SW35 to SW20, SW41 to SW21, SW7 to SW22, SW13 to SW23, SW19 to SW24, SW31 to SW26, SW37 to SW27, SW6 to SW28, SW12 to SW29, SW15 to SW3, SW18 to SW30, SW24 to SW31, SW30 to SW32, SW36 to SW33, SW42 to SW34, SW8 to SW35, SW14 to SW36, SW20 to SW37, SW26 to SW38, SW21 to SW4, SW27 to SW5, SW33 to SW6, SW39 to SW7, SW4 to SW8, SW10 to SW9
Connections:
- net matrix_R3 is gone; now on net matrix_R2: SW28.1, SW29.1, SW30.1, SW31.1, SW32.1, SW33.1, SW34.1
- net matrix_R4 is gone; now on net matrix_R1: SW22.1, SW23.1, SW24.1, SW25.1, SW26.1, SW27.1
- net matrix_C0: no longer D22.1 (K), D35.1 (K), D8.1 (K)
- net matrix_C1: no longer D23.1 (K), D36.1 (K), D9.1 (K)
- net matrix_C2: no longer D10.1 (K), D24.1 (K), D37.1 (K)
- net matrix_C3: no longer D11.1 (K), D25.1 (K), D38.1 (K)
- net matrix_C4: no longer D12.1 (K), D26.1 (K)
- net matrix_C5: no longer D13.1 (K), D27.1 (K)
- net matrix_C6: no longer D14.1 (K), D41.1 (K), SW35.1, SW36.1, SW37.1, SW38.1
- net matrix_R0: now also SW10.1, SW11.1, SW12.1, SW13.1, SW14.1, SW8.1, SW9.1
- net matrix_R1: now also SW15.1, SW16.1, SW17.1, SW18.1, SW19.1, SW20.1, SW21.1; no longer SW10.1, SW11.1, SW12.1, SW13.1, SW14.1, SW8.1, SW9.1
- net matrix_R2: now also SW35.1, SW36.1, SW37.1, SW38.1, SW39.1, SW40.1, SW41.1; no longer SW15.1, SW16.1, SW17.1, SW18.1, SW19.1, SW20.1, SW21.1
- net at D41.2 (A): now also SW41.2
- new net: D39.2 (A), SW39.2
- new net: D40.2 (A), SW40.2
- new net matrix_C10: D11.1 (K), D25.1 (K), D38.1 (K)
- new net matrix_C11: D12.1 (K), D26.1 (K), D39.1 (K)
- new net matrix_C12: D13.1 (K), D27.1 (K), D40.1 (K)
- new net matrix_C13: D14.1 (K), D41.1 (K)
- new net matrix_C7: D22.1 (K), D35.1 (K), D8.1 (K)
- new net matrix_C8: D23.1 (K), D36.1 (K), D9.1 (K)
- new net matrix_C9: D10.1 (K), D24.1 (K), D37.1 (K)
Other:
- moved on the sheet: D10, D11, D12, D13, D14, D15, D16, D17, D18, D19, D20, D21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

Commit message: reannoation with good linkage?
Parts:
- renumbered D1 to D401, D2 to D402, D3 to D403, D4 to D404, D5 to D405, D6 to D406, D7 to D407, D8 to D408, D9 to D409, D10 to D410, D11 to D411, D12 to D412, D13 to D413, D14 to D414, D15 to D415, D16 to D416, D17 to D417, D18 to D418, D19 to D419, D20 to D420, D21 to D421, D22 to D422, D23 to D423, D24 to D424, D25 to D425, D26 to D426, D27 to D427, D28 to D428, D29 to D429, D30 to D430, D31 to D431, D32 to D432, D33 to D433, D34 to D434, D35 to D435, D36 to D436, D37 to D437, D38 to D438, D39 to D439, D40 to D440, D41 to D441, SW1 to SW401, SW2 to SW402, SW3 to SW403, SW4 to SW404, SW5 to SW405, SW6 to SW406, SW7 to SW407, SW8 to SW408, SW9 to SW409, SW10 to SW410, SW11 to SW411, SW12 to SW412, SW13 to SW413, SW14 to SW414, SW15 to SW415, SW16 to SW416, SW17 to SW417, SW18 to SW418, SW19 to SW419, SW20 to SW420, SW21 to SW421, SW22 to SW422, SW23 to SW423, SW24 to SW424, SW25 to SW425, SW26 to SW426, SW27 to SW427, SW28 to SW428, SW29 to SW429, SW30 to SW430, SW31 to SW431, SW32 to SW432, SW33 to SW433, SW34 to SW434, SW35 to SW435, SW36 to SW436, SW37 to SW437, SW38 to SW438, SW39 to SW439, SW40 to SW440, SW41 to SW441

Commit message: fillout LCSC and swap micro usb
Parts:
- D401, D402, D403, D404, D405, D406, D407, D408, D409, D410, D411, D412, D413, D414, D415, D416, D417, D418, D419, D420, D421, D422, D423, D424, D425, D426, D427, D428, D429, D430, D431, D432, D433, D434, D435, D436, D437, D438, D439, D440, D441: LCSC (none) -> C78608
- SW401, SW402, SW403, SW404, SW405, SW406, SW407, SW408, SW409, SW410, SW411, SW412, SW413, SW414, SW415, SW416, SW417, SW418, SW419, SW420, SW421, SW422, SW423, SW424, SW425, SW426, SW427, SW428, SW429, SW430, SW431, SW432, SW433, SW434, SW435, SW436, SW437, SW438, SW439, SW440, SW441: now not fitted
