File: hardware/board/audio.kicad_sch (KiCad schematic)
At the start: 67 parts, among them J201 LineOut, J202 Headphone, J203 LineIn, U201 MAX98089ETN_T, U202 TPS7A20xxxDBV, Y201 12.288MHz

Commit message: drc
Parts:
- added T201: TerminalL, TerminalBlock_Phoenix:TerminalBlock_Phoenix_MKDS-1,5-2-5.08_1x02_P5.08mm_Horizontal, symbol Connector:Screw_Terminal_01x02
- added T202: TerminalR, TerminalBlock_Phoenix:TerminalBlock_Phoenix_MKDS-1,5-2-5.08_1x02_P5.08mm_Horizontal, symbol Connector:Screw_Terminal_01x02
- LS201, LS202: footprint TerminalBlock_Phoenix:TerminalBlock_Phoenix_MKDS-1,5-2-5.08_1x02_P5.08mm_Horizontal -> ledaw:bf-32-s-8ohm; now fitted
Connections:
- net at C211.1, FB202.2, TP202.1: now also T201.1 (Pin_1); no longer LS201.1
- net at C214.1, FB203.2, TP205.1: now also T201.2 (Pin_2); no longer LS201.2
- net at C222.1, FB205.2, TP216.1: now also T202.1 (Pin_1); no longer LS202.1
- net at C219.1, FB204.2, TP210.1: now also T202.2 (Pin_2); no longer LS202.2
- no-connect marks 5 -> 9

Commit message: fillout LCSC and swap micro usb
Parts:
- J201, J203, LS201, LS202, TP201, TP202, TP203, TP204, TP205, TP206, TP207, TP208, TP209, TP210, TP211, TP212, TP213, TP214, TP215, TP216, TP217, TP218: now not fitted
- J202: LCSC C4992301 -> C20182909
- T201, T202: LCSC (none) -> C5183929
Changed lines of the file:
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@@
 		(on_board yes)
 		(in_pos_files yes)
-		(dnp no)
+		(dnp yes)
 		(property "Reference" "J201"
 			(at 214.63 86.9951 0)
@@
 			)
 		)
+		(property "LCSC" "C5183929"
+			(at 260.35 115.57 0)
+			(hide yes)
+			(show_name no)
+			(do_not_autoplace no)
+			(effects
+				(font
+					(size 1.27 1.27)
+				)
+			)
+		)
 		(pin "2"
 		)
@@
 		(on_board yes)
 		(in_pos_files yes)
-		(dnp no)
+		(dnp yes)
 		(property "Reference" "TP206"
 			(at 194.31 90.9321 0)
@@
 		(on_board yes)
 		(in_pos_files yes)
-		(dnp no)
+		(dnp yes)
 		(fields_autoplaced yes)
 		(property "Reference" "TP204"
@@
 		(on_board yes)
 		(in_pos_files yes)
-		(dnp no)
+		(dnp yes)
 		(property "Reference" "TP214"
 			(at 175.006 124.714 0)
@@
 		(on_board yes)
 		(in_pos_files yes)
-		(dnp no)
+		(dnp yes)
 		(property "Reference" "TP201"
 			(at 95.25 60.198 0)
@@
 		(on_board yes)
 		(in_pos_files yes)
-		(dnp no)
+		(dnp yes)
 		(property "Reference" "TP217"
 			(at 49.784 149.352 0)
@@
 			)
 		)
-		(property "LCSC" "C4992301"
+		(property "LCSC" "C20182909"
 			(at 207.01 107.95 0)
 			(hide yes)
@@
 		(on_board yes)
 		(in_pos_files yes)
-		(dnp no)
+		(dnp yes)
 		(property "Reference" "TP205"
 			(at 243.586 75.946 0)
@@
 		(on_board yes)
 		(in_pos_files yes)
-		(dnp no)
+		(dnp yes)
 		(property "Reference" "TP208"
 			(at 93.98 109.474 0)
@@
 		(on_board yes)
 		(in_pos_files yes)
-		(dnp no)
+		(dnp yes)
 		(property "Reference" "LS202"
 			(at 274.32 115.5701 0)
@@
 		(on_board yes)
 		(in_pos_files yes)
-		(dnp no)
+		(dnp yes)
 		(property "Reference" "TP218"
 			(at 67.564 160.02 0)
@@
 		(on_board yes)
 		(in_pos_files yes)
-		(dnp no)
+		(dnp yes)
 		(property "Reference" "TP216"
 			(at 243.586 114.046 0)
@@
 		(on_board yes)
 		(in_pos_files yes)
-		(dnp no)
+		(dnp yes)
 		(property "Reference" "TP213"
 			(at 90.424 120.904 0)
@@
 		(on_board yes)
 		(in_pos_files yes)
-		(dnp no)
+		(dnp yes)
 		(property "Reference" "TP210"
 			(at 243.586 100.076 0)
@@
 			)
 		)
+		(property "LCSC" "C5183929"
+			(at 260.35 76.2 0)
+			(hide yes)
+			(show_name no)
+			(do_not_autoplace no)
+			(effects
+				(font
+					(size 1.27 1.27)
+				)
+			)
+		)
 		(pin "2"
 		)
@@
 		(on_board yes)
 		(in_pos_files yes)
-		(dnp no)
+		(dnp yes)
 		(property "Reference" "LS201"
 			(at 274.32 76.1999 0)
@@
 		(on_board yes)
 		(in_pos_files yes)
-		(dnp no)
+		(dnp yes)
 		(property "Reference" "J203"
 			(at 64.77 122.5551 0)
@@
 		(on_board yes)
 		(in_pos_files yes)
-		(dnp no)
+		(dnp yes)
 		(property "Reference" "TP212"
 			(at 181.61 118.618 0)
@@
 		(on_board yes)
 		(in_pos_files yes)
-		(dnp no)
+		(dnp yes)
 		(fields_autoplaced yes)
 		(property "Reference" "TP203"
@@
 		(on_board yes)
 		(in_pos_files yes)
-		(dnp no)
+		(dnp yes)
 		(property "Reference" "TP207"
 			(at 87.63 92.202 0)
@@
 		(on_board yes)
 		(in_pos_files yes)
-		(dnp no)
+		(dnp yes)
 		(property "Reference" "TP209"
 			(at 180.848 99.822 0)
@@
 		(on_board yes)
 		(in_pos_files yes)
-		(dnp no)
+		(dnp yes)
 		(property "Reference" "TP202"
 			(at 243.586 61.722 0)
@@
 		(on_board yes)
 		(in_pos_files yes)
-		(dnp no)
+		(dnp yes)
 		(property "Reference" "TP215"
 			(at 90.424 125.476 0)
@@
 		(on_board yes)
 		(in_pos_files yes)
-		(dnp no)
+		(dnp yes)
 		(property "Reference" "TP211"
 			(at 93.98 114.554 0)

Commit message: finish LCSC
Parts:
- C201, C203, C213, C215: LCSC C15850 -> C1713
Changed lines of the file:
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@@
 			)
 		)
-		(property "LCSC" "C15850"
+		(property "LCSC" "C1713"
 			(at 175.26 83.82 90)
 			(hide yes)
@@
 			)
 		)
-		(property "LCSC" "C15850"
+		(property "LCSC" "C1713"
 			(at 175.26 87.63 90)
 			(hide yes)
@@
 			)
 		)
-		(property "LCSC" "C15850"
+		(property "LCSC" "C1713"
 			(at 139.7 31.75 0)
 			(hide yes)
@@
 			)
 		)
-		(property "LCSC" "C15850"
+		(property "LCSC" "C1713"
 			(at 121.92 36.83 90)
 			(hide yes)

Commit message: use 1v8 audio LDO
Parts:
- U202: value TPS7A20xxxDBV -> TPS7A2018PDBVR; LCSC C2862740 -> C963430
Changed lines of the file:
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@@
 			)
 		)
-		(property "Value" "TPS7A20xxxDBV"
+		(property "Value" "TPS7A2018PDBVR"
 			(at 60.96 153.67 0)
 			(show_name no)
@@
 			)
 		)
-		(property "LCSC" "C2862740"
+		(property "LCSC" "C963430"
 			(at 60.96 161.29 0)
 			(hide yes)

Commit message: giga test points
Parts:
- TP217: value LDO_IN -> AUDIO_LDO_IN; now fitted
- TP218: value LDO_OUT -> AUDIO_LDO_OUT; now fitted
Other:
- moved on the sheet: C229
Changed lines of the file:
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@@
 	)
 	(junction
+		(at 241.3 69.85)
+		(diameter 0)
+		(color 0 0 0 0)
+	)
+	(junction
 		(at 152.4 29.21)
 		(diameter 0)
@@
 	)
 	(junction
+		(at 90.17 158.75)
+		(diameter 0)
+		(color 0 0 0 0)
+	)
+	(junction
 		(at 143.51 46.99)
 		(diameter 0)
@@
 	)
 	(junction
-		(at 50.8 158.75)
-		(diameter 0)
-		(color 0 0 0 0)
-	)
-	(junction
 		(at 134.62 46.99)
 		(diameter 0)
@@
 	)
 	(junction
-		(at 173.99 142.24)
+		(at 246.38 69.85)
 		(diameter 0)
 		(color 0 0 0 0)
 	)
 	(junction
-		(at 119.38 140.97)
+		(at 173.99 142.24)
 		(diameter 0)
 		(color 0 0 0 0)
 	)
 	(junction
-		(at 241.3 69.85)
+		(at 119.38 140.97)
 		(diameter 0)
 		(color 0 0 0 0)
@@
 	)
 	(junction
-		(at 73.66 158.75)
-		(diameter 0)
-		(color 0 0 0 0)
-	)
-	(junction
 		(at 193.04 110.49)
 		(diameter 0)
@@
 	)
 	(junction
-		(at 246.38 69.85)
-		(diameter 0)
-		(color 0 0 0 0)
-	)
-	(junction
 		(at 72.39 105.41)
 		(diameter 0)
@@
 	(wire
 		(pts
-			(xy 60.96 170.18) (xy 73.66 170.18)
+			(xy 60.96 170.18) (xy 90.17 170.18)
 		)
 		(stroke
@@
 	(wire
 		(pts
-			(xy 53.34 158.75) (xy 50.8 158.75)
-		)
-		(stroke
-			(width 0)
-			(type default)
-		)
-	)
-	(wire
-		(pts
 			(xy 82.55 116.84) (xy 82.55 119.38)
 		)
@@
 	(wire
 		(pts
-			(xy 50.8 158.75) (xy 45.72 158.75)
-		)
-		(stroke
-			(width 0)
-			(type default)
-		)
-	)
-	(wire
-		(pts
 			(xy 152.4 36.83) (xy 152.4 46.99)
 		)
@@
 	(wire
 		(pts
-			(xy 73.66 158.75) (xy 73.66 162.56)
+			(xy 90.17 158.75) (xy 90.17 162.56)
 		)
 		(stroke
@@
 	(wire
 		(pts
-			(xy 69.85 158.75) (xy 73.66 158.75)
+			(xy 69.85 158.75) (xy 90.17 158.75)
 		)
 		(stroke
@@
 	(wire
 		(pts
+			(xy 40.64 158.75) (xy 53.34 158.75)
+		)
+		(stroke
+			(width 0)
+			(type default)
+		)
+	)
+	(wire
+		(pts
 			(xy 74.93 99.06) (xy 74.93 105.41)
 		)
@@
 	(wire
 		(pts
-			(xy 233.68 121.92) (xy 246.38 121.92)
+			(xy 241.3 69.85) (xy 246.38 69.85)
 		)
 		(stroke
@@
 	(wire
 		(pts
-			(xy 223.52 121.92) (xy 223.52 102.87)
+			(xy 233.68 121.92) (xy 246.38 121.92)
 		)
 		(stroke
@@
 	(wire
 		(pts
-			(xy 92.71 105.41) (xy 99.06 105.41)
+			(xy 223.52 121.92) (xy 223.52 102.87)
 		)
 		(stroke
@@
 	(wire
 		(pts
-			(xy 110.49 46.99) (xy 110.49 48.26)
+			(xy 92.71 105.41) (xy 99.06 105.41)
 		)
 		(stroke
@@
 	(wire
 		(pts
-			(xy 45.72 158.75) (xy 45.72 162.56)
+			(xy 110.49 46.99) (xy 110.49 48.26)
 		)
 		(stroke
@@
 	(wire
 		(pts
-			(xy 232.41 69.85) (xy 246.38 69.85)
+			(xy 45.72 158.75) (xy 45.72 162.56)
 		)
 		(stroke
@@
 	(wire
 		(pts
-			(xy 73.66 167.64) (xy 73.66 170.18)
+			(xy 90.17 167.64) (xy 90.17 170.18)
 		)
 		(stroke
@@
 	(wire
 		(pts
+			(xy 232.41 69.85) (xy 241.3 69.85)
+		)
+		(stroke
+			(width 0)
+			(type default)
+		)
+	)
+	(wire
+		(pts
 			(xy 170.18 72.39) (xy 179.07 72.39)
 		)
@@
 	(wire
 		(pts
-			(xy 73.66 156.21) (xy 73.66 158.75)
+			(xy 90.17 156.21) (xy 90.17 158.75)
 		)
 		(stroke
@@
 	(symbol
 		(lib_id "power:+1V8")
-		(at 73.66 156.21 0)
+		(at 90.17 156.21 0)
 		(unit 1)
 		(body_style 1)
@@
 		(fields_autoplaced yes)
 		(property "Reference" "#PWR0241"
-			(at 73.66 160.02 0)
+			(at 90.17 160.02 0)
 			(hide yes)
 			(show_name no)
@@
 		)
 		(property "Value" "+1V8"
-			(at 73.66 151.13 0)
+			(at 90.17 151.13 0)
 			(show_name no)
 			(do_not_autoplace no)
@@
 		)
 		(property "Footprint" ""
-			(at 73.66 156.21 0)
+			(at 90.17 156.21 0)
 			(hide yes)
 			(show_name no)
@@
 		)
 		(property "Datasheet" ""
-			(at 73.66 156.21 0)
+			(at 90.17 156.21 0)
 			(hide yes)
 			(show_name no)
@@
 		)
 		(property "Description" "Power symbol creates a global label with name \"+1V8\""
-			(at 73.66 156.21 0)
+			(at 90.17 156.21 0)
 			(hide yes)
 			(show_name no)
@@
 	(symbol
 		(lib_id "Connector:TestPoint")
-		(at 50.8 158.75 0)
+		(at 40.64 158.75 0)
+		(mirror y)
 		(unit 1)
 		(body_style 1)
@@
 		(on_board yes)
 		(in_pos_files yes)
-		(dnp yes)
+		(dnp no)
 		(property "Reference" "TP217"
-			(at 49.784 149.352 0)
+			(at 41.656 149.352 0)
 			(show_name no)
 			(do_not_autoplace no)
@@
 			)
 		)
-		(property "Value" "LDO_IN"
-			(at 49.784 151.892 0)
+		(property "Value" "AUDIO_LDO_IN"
+			(at 41.656 151.892 0)
 			(show_name no)
 			(do_not_autoplace no)
@@
 		)
 		(property "Footprint" "TestPoint:TestPoint_Pad_D2.0mm"
-			(at 55.88 158.75 0)
+			(at 35.56 158.75 0)
 			(hide yes)
 			(show_name no)
@@
 		)
 		(property "Datasheet" ""
-			(at 55.88 158.75 0)
+			(at 35.56 158.75 0)
 			(hide yes)
 			(show_name no)
@@
 		)
 		(property "Description" "test point"
-			(at 50.8 158.75 0)
+			(at 40.64 158.75 0)
 			(hide yes)
 			(show_name no)
@@
 		)
 		(property "LCSC" ""
-			(at 50.8 158.75 0)
+			(at 40.64 158.75 0)
 			(hide yes)
 			(show_name no)
@@
 		(on_board yes)
 		(in_pos_files yes)
-		(dnp yes)
+		(dnp no)
 		(property "Reference" "TP218"
-			(at 67.564 160.02 0)
+			(at 69.088 161.036 0)
 			(show_name no)
 			(do_not_autoplace no)
@@
 			)
 		)
-		(property "Value" "LDO_OUT"
-			(at 67.564 162.56 0)
+		(property "Value" "AUDIO_LDO_OUT"
+			(at 68.834 163.068 0)
 			(show_name no)
 			(do_not_autoplace no)
@@
 	(symbol
 		(lib_id "Device:C_Small")
-		(at 73.66 165.1 0)
+		(at 90.17 165.1 0)
 		(unit 1)
 		(body_style 1)
@@
 		(fields_autoplaced yes)
 		(property "Reference" "C229"
-			(at 76.2 163.8362 0)
+			(at 92.71 163.8362 0)
 			(show_name no)
 			(do_not_autoplace no)
@@
 		)
 		(property "Value" "1uF"
-			(at 76.2 166.3762 0)
+			(at 92.71 166.3762 0)
 			(show_name no)
 			(do_not_autoplace no)
@@
 		)
 		(property "Footprint" "Capacitor_SMD:C_0805_2012Metric"
-			(at 73.66 165.1 0)
+			(at 90.17 165.1 0)
 			(hide yes)
 			(show_name no)
@@
 		)
 		(property "Datasheet" ""
-			(at 73.66 165.1 0)
+			(at 90.17 165.1 0)
 			(hide yes)
 			(show_name no)
@@
 		)
 		(property "Description" "Unpolarized capacitor, small symbol"
-			(at 73.66 165.1 0)
+			(at 90.17 165.1 0)
 			(hide yes)
 			(show_name no)
@@
 		)
 		(property "LCSC" "C28323"
-			(at 73.66 165.1 0)
+			(at 90.17 165.1 0)
 			(hide yes)
 			(show_name no)

Commit message: footprints
Parts:
- TP201, TP202, TP203, TP204, TP205, TP206, TP207, TP208, TP209, TP210, TP211, TP212, TP213, TP214, TP215, TP216, TP217, TP218: footprint TestPoint:TestPoint_Pad_D2.0mm -> TestPoint:TestPoint_Keystone_5015_Micro_Mini
Changed lines of the file:
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@@
 			)
 		)
-		(property "Footprint" "TestPoint:TestPoint_Pad_D2.0mm"
+		(property "Footprint" "TestPoint:TestPoint_Keystone_5015_Micro_Mini"
 			(at 196.85 86.36 0)
 			(hide yes)
@@
 			)
 		)
-		(property "Footprint" "TestPoint:TestPoint_Pad_D2.0mm"
+		(property "Footprint" "TestPoint:TestPoint_Keystone_5015_Micro_Mini"
 			(at 196.85 83.82 0)
 			(hide yes)
@@
 			)
 		)
-		(property "Footprint" "TestPoint:TestPoint_Pad_D2.0mm"
+		(property "Footprint" "TestPoint:TestPoint_Keystone_5015_Micro_Mini"
 			(at 182.88 116.84 0)
 			(hide yes)
@@
 			)
 		)
-		(property "Footprint" "TestPoint:TestPoint_Pad_D2.0mm"
+		(property "Footprint" "TestPoint:TestPoint_Keystone_5015_Micro_Mini"
 			(at 101.6 64.77 0)
 			(hide yes)
@@
 			)
 		)
-		(property "Footprint" "TestPoint:TestPoint_Pad_D2.0mm"
+		(property "Footprint" "TestPoint:TestPoint_Keystone_5015_Micro_Mini"
 			(at 35.56 158.75 0)
 			(hide yes)
@@
 			)
 		)
-		(property "Footprint" "TestPoint:TestPoint_Pad_D2.0mm"
+		(property "Footprint" "TestPoint:TestPoint_Keystone_5015_Micro_Mini"
 			(at 251.46 83.82 0)
 			(hide yes)
@@
 			)
 		)
-		(property "Footprint" "TestPoint:TestPoint_Pad_D2.0mm"
+		(property "Footprint" "TestPoint:TestPoint_Keystone_5015_Micro_Mini"
 			(at 87.63 105.41 0)
 			(hide yes)
@@
 			)
 		)
-		(property "Footprint" "TestPoint:TestPoint_Pad_D2.0mm"
+		(property "Footprint" "TestPoint:TestPoint_Keystone_5015_Micro_Mini"
 			(at 74.93 158.75 0)
 			(hide yes)
@@
 			)
 		)
-		(property "Footprint" "TestPoint:TestPoint_Pad_D2.0mm"
+		(property "Footprint" "TestPoint:TestPoint_Keystone_5015_Micro_Mini"
 			(at 251.46 121.92 0)
 			(hide yes)
@@
 			)
 		)
-		(property "Footprint" "TestPoint:TestPoint_Pad_D2.0mm"
+		(property "Footprint" "TestPoint:TestPoint_Keystone_5015_Micro_Mini"
 			(at 91.44 116.84 0)
 			(hide yes)
@@
 			)
 		)
-		(property "Footprint" "TestPoint:TestPoint_Pad_D2.0mm"
+		(property "Footprint" "TestPoint:TestPoint_Keystone_5015_Micro_Mini"
 			(at 251.46 107.95 0)
 			(hide yes)
@@
 			)
 		)
-		(property "Footprint" "TestPoint:TestPoint_Pad_D2.0mm"
+		(property "Footprint" "TestPoint:TestPoint_Keystone_5015_Micro_Mini"
 			(at 187.96 113.03 0)
 			(hide yes)
@@
 			)
 		)
-		(property "Footprint" "TestPoint:TestPoint_Pad_D2.0mm"
+		(property "Footprint" "TestPoint:TestPoint_Keystone_5015_Micro_Mini"
 			(at 194.31 76.2 0)
 			(hide yes)
@@
 			)
 		)
-		(property "Footprint" "TestPoint:TestPoint_Pad_D2.0mm"
+		(property "Footprint" "TestPoint:TestPoint_Keystone_5015_Micro_Mini"
 			(at 81.28 87.63 0)
 			(hide yes)
@@
 			)
 		)
-		(property "Footprint" "TestPoint:TestPoint_Pad_D2.0mm"
+		(property "Footprint" "TestPoint:TestPoint_Keystone_5015_Micro_Mini"
 			(at 187.96 107.95 0)
 			(hide yes)
@@
 			)
 		)
-		(property "Footprint" "TestPoint:TestPoint_Pad_D2.0mm"
+		(property "Footprint" "TestPoint:TestPoint_Keystone_5015_Micro_Mini"
 			(at 251.46 69.85 0)
 			(hide yes)
@@
 			)
 		)
-		(property "Footprint" "TestPoint:TestPoint_Pad_D2.0mm"
+		(property "Footprint" "TestPoint:TestPoint_Keystone_5015_Micro_Mini"
 			(at 91.44 121.92 0)
 			(hide yes)
@@
 			)
 		)
-		(property "Footprint" "TestPoint:TestPoint_Pad_D2.0mm"
+		(property "Footprint" "TestPoint:TestPoint_Keystone_5015_Micro_Mini"
 			(at 87.63 110.49 0)
 			(hide yes)

Commit message: lot of testpoints
Parts:
- TP201, TP202, TP203, TP204, TP205, TP206, TP207, TP208, TP209, TP210, TP211, TP212, TP213, TP214, TP215, TP216, TP217, TP218: footprint TestPoint:TestPoint_Keystone_5015_Micro_Mini -> ledaw:named_TestPoint
Changed lines of the file:
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@@
 			)
 		)
-		(property "Footprint" "TestPoint:TestPoint_Keystone_5015_Micro_Mini"
+		(property "Footprint" "ledaw:named_TestPoint"
 			(at 196.85 86.36 0)
 			(hide yes)
@@
 			)
 		)
-		(property "Footprint" "TestPoint:TestPoint_Keystone_5015_Micro_Mini"
+		(property "Footprint" "ledaw:named_TestPoint"
 			(at 196.85 83.82 0)
 			(hide yes)
@@
 			)
 		)
-		(property "Footprint" "TestPoint:TestPoint_Keystone_5015_Micro_Mini"
+		(property "Footprint" "ledaw:named_TestPoint"
 			(at 182.88 116.84 0)
 			(hide yes)
@@
 			)
 		)
-		(property "Footprint" "TestPoint:TestPoint_Keystone_5015_Micro_Mini"
+		(property "Footprint" "ledaw:named_TestPoint"
 			(at 101.6 64.77 0)
 			(hide yes)
@@
 			)
 		)
-		(property "Footprint" "TestPoint:TestPoint_Keystone_5015_Micro_Mini"
+		(property "Footprint" "ledaw:named_TestPoint"
 			(at 35.56 158.75 0)
 			(hide yes)
@@
 			)
 		)
-		(property "Footprint" "TestPoint:TestPoint_Keystone_5015_Micro_Mini"
+		(property "Footprint" "ledaw:named_TestPoint"
 			(at 251.46 83.82 0)
 			(hide yes)
@@
 			)
 		)
-		(property "Footprint" "TestPoint:TestPoint_Keystone_5015_Micro_Mini"
+		(property "Footprint" "ledaw:named_TestPoint"
 			(at 87.63 105.41 0)
 			(hide yes)
@@
 			)
 		)
-		(property "Footprint" "TestPoint:TestPoint_Keystone_5015_Micro_Mini"
+		(property "Footprint" "ledaw:named_TestPoint"
 			(at 74.93 158.75 0)
 			(hide yes)
@@
 			)
 		)
-		(property "Footprint" "TestPoint:TestPoint_Keystone_5015_Micro_Mini"
+		(property "Footprint" "ledaw:named_TestPoint"
 			(at 251.46 121.92 0)
 			(hide yes)
@@
 			)
 		)
-		(property "Footprint" "TestPoint:TestPoint_Keystone_5015_Micro_Mini"
+		(property "Footprint" "ledaw:named_TestPoint"
 			(at 91.44 116.84 0)
 			(hide yes)
@@
 			)
 		)
-		(property "Footprint" "TestPoint:TestPoint_Keystone_5015_Micro_Mini"
+		(property "Footprint" "ledaw:named_TestPoint"
 			(at 251.46 107.95 0)
 			(hide yes)
@@
 			)
 		)
-		(property "Footprint" "TestPoint:TestPoint_Keystone_5015_Micro_Mini"
+		(property "Footprint" "ledaw:named_TestPoint"
 			(at 187.96 113.03 0)
 			(hide yes)
@@
 			)
 		)
-		(property "Footprint" "TestPoint:TestPoint_Keystone_5015_Micro_Mini"
+		(property "Footprint" "ledaw:named_TestPoint"
 			(at 194.31 76.2 0)
 			(hide yes)
@@
 			)
 		)
-		(property "Footprint" "TestPoint:TestPoint_Keystone_5015_Micro_Mini"
+		(property "Footprint" "ledaw:named_TestPoint"
 			(at 81.28 87.63 0)
 			(hide yes)
@@
 			)
 		)
-		(property "Footprint" "TestPoint:TestPoint_Keystone_5015_Micro_Mini"
+		(property "Footprint" "ledaw:named_TestPoint"
 			(at 187.96 107.95 0)
 			(hide yes)
@@
 			)
 		)
-		(property "Footprint" "TestPoint:TestPoint_Keystone_5015_Micro_Mini"
+		(property "Footprint" "ledaw:named_TestPoint"
 			(at 251.46 69.85 0)
 			(hide yes)
@@
 			)
 		)
-		(property "Footprint" "TestPoint:TestPoint_Keystone_5015_Micro_Mini"
+		(property "Footprint" "ledaw:named_TestPoint"
 			(at 91.44 121.92 0)
 			(hide yes)
@@
 			)
 		)
-		(property "Footprint" "TestPoint:TestPoint_Keystone_5015_Micro_Mini"
+		(property "Footprint" "ledaw:named_TestPoint"
 			(at 87.63 110.49 0)
 			(hide yes)

Commit message: delete hella TPs
Parts:
- removed TP202: SPKLP, ledaw:named_TestPoint, symbol Connector:TestPoint
- removed TP204: RECP, ledaw:named_TestPoint, symbol Connector:TestPoint
- removed TP205: SPKLN, ledaw:named_TestPoint, symbol Connector:TestPoint
- removed TP206: RECN, ledaw:named_TestPoint, symbol Connector:TestPoint
- removed TP208, TP213: INA1, ledaw:named_TestPoint, symbol Connector:TestPoint
- removed TP209: HPR, ledaw:named_TestPoint, symbol Connector:TestPoint
- removed TP210: SPKRP, ledaw:named_TestPoint, symbol Connector:TestPoint
- removed TP211, TP215: INA2, ledaw:named_TestPoint, symbol Connector:TestPoint
- removed TP212: HPL, ledaw:named_TestPoint, symbol Connector:TestPoint
- removed TP216: SPKRN, ledaw:named_TestPoint, symbol Connector:TestPoint
