File: hardware/board/usb.kicad_sch (KiCad schematic)
At the start: 10 parts, among them J501 USB_B_Micro, J502 USB_C_Receptacle_PowerOnly_24P, U501 TPD2EUSB30

Commit message: lot of testpoints
Parts:
- removed TP501: VBUS, TestPoint:TestPoint_Keystone_5015_Micro_Mini, symbol Connector:TestPoint
- TP502: footprint TestPoint:TestPoint_Keystone_5015_Micro_Mini -> ledaw:named_TestPoint
Changed lines of the file:
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@@
-	)
-	(junction
-		(at 57.15 152.4)
-		(diameter 0)
-		(color 0 0 0 0)
 	)
 	(junction
@@
 	(wire
 		(pts
-			(xy 57.15 152.4) (xy 81.28 152.4)
+			(xy 62.23 176.53) (xy 63.5 176.53)
 		)
 		(stroke
@@
 	(wire
 		(pts
-			(xy 62.23 176.53) (xy 63.5 176.53)
+			(xy 63.5 165.1) (xy 52.07 165.1)
 		)
 		(stroke
@@
 	(wire
 		(pts
-			(xy 63.5 165.1) (xy 52.07 165.1)
+			(xy 140.97 116.84) (xy 140.97 119.38)
+		)
+		(stroke
+			(width 0)
+			(type solid)
+		)
+	)
+	(wire
+		(pts
+			(xy 113.03 111.76) (xy 88.9 111.76)
+		)
+		(stroke
+			(width 0)
+			(type solid)
+		)
+	)
+	(wire
+		(pts
+			(xy 92.71 109.22) (xy 88.9 109.22)
+		)
+		(stroke
+			(width 0)
+			(type solid)
+		)
+	)
+	(wire
+		(pts
+			(xy 29.21 177.8) (xy 36.83 177.8)
 		)
 		(stroke
@@
 	(wire
 		(pts
-			(xy 140.97 116.84) (xy 140.97 119.38)
-		)
-		(stroke
-			(width 0)
-			(type solid)
-		)
-	)
-	(wire
-		(pts
-			(xy 113.03 111.76) (xy 88.9 111.76)
-		)
-		(stroke
-			(width 0)
-			(type solid)
-		)
-	)
-	(wire
-		(pts
-			(xy 92.71 109.22) (xy 88.9 109.22)
-		)
-		(stroke
-			(width 0)
-			(type solid)
-		)
-	)
-	(wire
-		(pts
-			(xy 29.21 177.8) (xy 36.83 177.8)
+			(xy 113.03 111.76) (xy 113.03 125.73)
+		)
+		(stroke
+			(width 0)
+			(type solid)
+		)
+	)
+	(wire
+		(pts
+			(xy 140.97 104.14) (xy 140.97 106.68)
+		)
+		(stroke
+			(width 0)
+			(type solid)
+		)
+	)
+	(wire
+		(pts
+			(xy 156.21 116.84) (xy 149.86 116.84)
+		)
+		(stroke
+			(width 0)
+			(type solid)
+		)
+	)
+	(wire
+		(pts
+			(xy 114.3 111.76) (xy 113.03 111.76)
+		)
+		(stroke
+			(width 0)
+			(type solid)
+		)
+	)
+	(wire
+		(pts
+			(xy 149.86 116.84) (xy 140.97 116.84)
+		)
+		(stroke
+			(width 0)
+			(type solid)
+		)
+	)
+	(wire
+		(pts
+			(xy 88.9 104.14) (xy 140.97 104.14)
+		)
+		(stroke
+			(width 0)
+			(type solid)
+		)
+	)
+	(wire
+		(pts
+			(xy 102.87 135.89) (xy 102.87 134.62)
+		)
+		(stroke
+			(width 0)
+			(type solid)
+		)
+	)
+	(wire
+		(pts
+			(xy 81.28 163.83) (xy 81.28 166.37)
+		)
+		(stroke
+			(width 0)
+			(type solid)
+		)
+	)
+	(wire
+		(pts
+			(xy 63.5 171.45) (xy 63.5 165.1)
 		)
 		(stroke
@@
 	(wire
 		(pts
-			(xy 113.03 111.76) (xy 113.03 125.73)
-		)
-		(stroke
-			(width 0)
-			(type solid)
-		)
-	)
-	(wire
-		(pts
-			(xy 140.97 104.14) (xy 140.97 106.68)
-		)
-		(stroke
-			(width 0)
-			(type solid)
-		)
-	)
-	(wire
-		(pts
-			(xy 156.21 116.84) (xy 149.86 116.84)
-		)
-		(stroke
-			(width 0)
-			(type solid)
-		)
-	)
-	(wire
-		(pts
-			(xy 114.3 111.76) (xy 113.03 111.76)
-		)
-		(stroke
-			(width 0)
-			(type solid)
-		)
-	)
-	(wire
-		(pts
-			(xy 149.86 116.84) (xy 140.97 116.84)
-		)
-		(stroke
-			(width 0)
-			(type solid)
-		)
-	)
-	(wire
-		(pts
-			(xy 88.9 104.14) (xy 140.97 104.14)
-		)
-		(stroke
-			(width 0)
-			(type solid)
-		)
-	)
-	(wire
-		(pts
-			(xy 102.87 135.89) (xy 102.87 134.62)
-		)
-		(stroke
-			(width 0)
-			(type solid)
-		)
-	)
-	(wire
-		(pts
-			(xy 81.28 163.83) (xy 81.28 166.37)
-		)
-		(stroke
-			(width 0)
-			(type solid)
-		)
-	)
-	(wire
-		(pts
-			(xy 63.5 171.45) (xy 63.5 165.1)
+			(xy 78.74 119.38) (xy 81.28 119.38)
 		)
 		(stroke
@@
 	(wire
 		(pts
-			(xy 78.74 119.38) (xy 81.28 119.38)
-		)
-		(stroke
-			(width 0)
-			(type default)
-		)
-	)
-	(wire
-		(pts
-			(xy 52.07 152.4) (xy 57.15 152.4)
+			(xy 52.07 152.4) (xy 81.28 152.4)
 		)
 		(stroke
@@
 			)
 		)
-		(property "Footprint" "TestPoint:TestPoint_Keystone_5015_Micro_Mini"
+		(property "Footprint" "ledaw:named_TestPoint"
 			(at 154.94 116.84 0)
 			(hide yes)
@@
 					(unit 1)
 				)
-			)
-		)
-	)
-	(symbol
-		(lib_id "Connector:TestPoint")
-		(at 57.15 152.4 0)
-		(unit 1)
-		(body_style 1)
-		(exclude_from_sim no)
-		(in_bom yes)
-		(on_board yes)
-		(in_pos_files yes)
-		(dnp no)
-		(fields_autoplaced yes)
-		(property "Reference" "TP501"
-			(at 59.69 147.8279 0)
-			(show_name no)
-			(do_not_autoplace no)
-			(effects
-				(font
-					(size 1.27 1.27)
-				)
-				(justify left)
-			)
-		)
-		(property "Value" "VBUS"
-			(at 59.69 150.3679 0)
-			(show_name no)
-			(do_not_autoplace no)
-			(effects
-				(font
-					(size 1.27 1.27)
-				)
-				(justify left)
-			)
-		)
-		(property "Footprint" "TestPoint:TestPoint_Keystone_5015_Micro_Mini"
-			(at 62.23 152.4 0)
-			(hide yes)
-			(show_name no)
-			(do_not_autoplace no)
-			(effects
-				(font
-					(size 1.27 1.27)
-				)
-			)
-		)
-		(property "Datasheet" ""
-			(at 62.23 152.4 0)
-			(hide yes)
-			(show_name no)
-			(do_not_autoplace no)
-			(effects
-				(font
-					(size 1.27 1.27)
-				)
-			)
-		)
-		(property "Description" "test point"
-			(at 57.15 152.4 0)
-			(hide yes)
-			(show_name no)
-			(do_not_autoplace no)
-			(effects
-				(font
-					(size 1.27 1.27)
-				)
-			)
-		)
-		(pin "1"
-		)
-		(instances
-			(project "board"
-				(path "/dd13fd41-39ab-4435-9074-5024f1786746/e77fa723-60b4-4aaf-b8c0-33f73a50a054"
-					(reference "TP501")
-					(unit 1)
-				)

Commit message: add back efuse
Parts:
- removed CR501: SMBJ5.0A-TR, Diode_SMD:D_SMB, symbol 2020-11-06_22-01-36:SMBJ5.0A-TR
- added C501: 100nF, Capacitor_SMD:C_0805_2012Metric, symbol Device:C_Small
- added C502: 3.3nF, Capacitor_SMD:C_0805_2012Metric, symbol Device:C_Small
- added C503: 1uF, Capacitor_SMD:C_0805_2012Metric, symbol Device:C_Small
- added R503: 1M, Resistor_SMD:R_0805_2012Metric, symbol Device:R_Small
- added R504: 390k, Resistor_SMD:R_0805_2012Metric, symbol Device:R_Small
- added R505: 10k, Resistor_SMD:R_0805_2012Metric, symbol Device:R_Small
- added R506: 681 @ 1%, Resistor_SMD:R_0805_2012Metric, symbol Device:R_Small
- added U502: TPS259531DSGR, ledaw:SON50P200X200X80-9N, symbol TPS259531DSGR:TPS259531DSGR
Connections:
- net +5V: now also C503.1, U502.5 (OUT); no longer J502.A4 (VBUS), J502.A9 (VBUS), J502.B4 (VBUS), J502.B9 (VBUS)
- net GND: now also C501.2, C502.2, C503.2, R504.2, R506.2, U502.8 (GND), U502.9 (GND)
- new net: C501.1, J502.A4 (VBUS), J502.A9 (VBUS), J502.B4 (VBUS), J502.B9 (VBUS), R503.1, U502.3 (IN), U502.4 (IN)
- new net: C502.1, U502.1 (DVDT)
- new net: R503.2, R504.1, U502.2 (EN/UVLO)
- new net +3V3: R505.1
- new net FUSE_ILM: R506.1, U502.7 (ILM)
- new net FUSE_~{FLT}: R505.2, U502.6 (~{FLT})
Other:
- note added: "fault not that useful cuz we can't do anything when there's no power"
- moved on the sheet: J502, R510, R511
