File: hardware/board/usb.kicad_sch (KiCad schematic)
At the start: 16 parts, among them J501 USB_B_Micro, J502 USB_C_Receptacle_PowerOnly_24P, U501 TPD2EUSB30, U502 TPS259531DSGR

Commit message: holes and shieeeeet
Parts:
- TP502: value USB_OTG_ID -> USB_OTGID
Changed lines of the file:
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@@
 			)
 		)
-		(property "Value" "USB_OTG_ID"
+		(property "Value" "USB_OTGID"
 			(at 152.4 114.8079 0)
 			(show_name no)

Commit message: rewrite LCSC
Parts:
- C503: LCSC C28323 -> C376926; MPN (none) -> TCC0805X7R105K500DT; Manufacturer (none) -> CCTC
- R501, R502: Digi-Key_PN 311-2.20KHRCT-ND -> (none); LCSC (none) -> C17520; MPN RC0603FR-072K2L -> 0805W8F2201T5E; Manufacturer Yageo -> UNI-ROYAL
- R503: LCSC C6351850 -> C17514; MPN (none) -> 0805W8F1004T5E; Manufacturer (none) -> UNI-ROYAL
- U501: LCSC (none) -> C97502
Changed lines of the file:
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@@
 		(in_pos_files yes)
 		(dnp no)
+		(property "LCSC" "C17520"
+			(at 140.97 123.19 0)
+			(hide yes)
+			(effects (font (size 1.27 1.27)))
+		)
 		(property "Reference" "R502"
 			(at 138.43 121.92 0)
@@
 			)
 		)
-		(property "Manufacturer" "Yageo"
+		(property "Manufacturer" "UNI-ROYAL"
 			(at 140.97 123.19 0)
 			(hide yes)
@@
 			)
 		)
-		(property "MPN" "RC0603FR-072K2L"
+		(property "MPN" "0805W8F2201T5E"
 			(at 140.97 123.19 0)
 			(hide yes)
@@
 			)
 		)
-		(property "Digi-Key_PN" "311-2.20KHRCT-ND"
+		(property "Digi-Key_PN" ""
 			(at 140.97 123.19 0)
 			(hide yes)
@@
 		(dnp no)
 		(fields_autoplaced yes)
+		(property "MPN" "TCC0805X7R105K500DT"
+			(at 156.21 45.72 0)
+			(hide yes)
+			(effects (font (size 1.27 1.27)))
+		)
+		(property "Manufacturer" "CCTC"
+			(at 156.21 45.72 0)
+			(hide yes)
+			(effects (font (size 1.27 1.27)))
+		)
 		(property "Reference" "C503"
 			(at 158.75 44.4562 0)
@@
 			)
 		)
-		(property "LCSC" "C28323"
+		(property "LCSC" "C376926"
 			(at 156.21 45.72 0)
 			(hide yes)
@@
 		(in_pos_files yes)
 		(dnp no)
+		(property "LCSC" "C17520"
+			(at 140.97 110.49 0)
+			(hide yes)
+			(effects (font (size 1.27 1.27)))
+		)
 		(property "Reference" "R501"
 			(at 138.43 109.22 0)
@@
 			)
 		)
-		(property "Manufacturer" "Yageo"
+		(property "Manufacturer" "UNI-ROYAL"
 			(at 140.97 110.49 0)
 			(hide yes)
@@
 			)
 		)
-		(property "MPN" "RC0603FR-072K2L"
+		(property "MPN" "0805W8F2201T5E"
 			(at 140.97 110.49 0)
 			(hide yes)
@@
 			)
 		)
-		(property "Digi-Key_PN" "311-2.20KHRCT-ND"
+		(property "Digi-Key_PN" ""
 			(at 140.97 110.49 0)
 			(hide yes)
@@
 		(in_pos_files yes)
 		(dnp no)
+		(property "MPN" "0805W8F1004T5E"
+			(at 85.09 46.99 0)
+			(hide yes)
+			(effects (font (size 1.27 1.27)))
+		)
+		(property "Manufacturer" "UNI-ROYAL"
+			(at 85.09 46.99 0)
+			(hide yes)
+			(effects (font (size 1.27 1.27)))
+		)
 		(property "Reference" "R503"
 			(at 82.55 45.7199 0)
@@
 			)
 		)
-		(property "LCSC" "C6351850"
+		(property "LCSC" "C17514"
 			(at 85.09 46.99 0)
 			(hide yes)
@@
 		(in_pos_files yes)
 		(dnp no)
+		(property "LCSC" "C97502"
+			(at 102.87 125.73 0)
+			(hide yes)
+			(effects (font (size 1.27 1.27)))
+		)
 		(property "Reference" "U501"
 			(at 102.87 115.57 0)
@@
 			)
 		)
-		(property "Datasheet" "http://www.ti.com/lit/ds/symlink/tpd2eusb30a.pdf"
+		(property "Datasheet" "https://www.ti.com/lit/ds/symlink/tpd2eusb30.pdf"
 			(at 102.87 125.73 0)
 			(hide yes)
