File: hardware/RP2350_80QFN_minimal/RP2350_80QFN_minimal.kicad_pcb (KiCad board)
At the start: 2 copper layers, 52 x 71.5 mm, 49 parts, among them J1 USB_B_Micro, J2 Conn_02x26_Odd_Even, J3 Conn_02x26_Odd_Even, J4 SM03B-SRSS-TB, SW1 SW_Push, SW2 SW_Push, U1 RP2350_80QFN, U2 NCP1117-3.3_SOT223, U3 W25Q128JVS, U4 DNF, Y1 ABM8-272-T3

Commit message: annotate 2350 example
Parts:
- renumbered C1 to C301, C5 to C302, C8 to C303, C10 to C304, C11 to C305, C12 to C306, C13 to C307, C14 to C308, C15 to C309, C16 to C310, C17 to C311, C18 to C312, C20 to C313, C21 to C314, C9 to C315, C6 to C316, C7 to C317, C2 to C318, C19 to C319, C22 to C320, C3 to C321, C4 to C322, H1 to H301, H2 to H302, H3 to H303, H4 to H304, J1 to J301, J2 to J302, J3 to J303, J4 to J304, L1 to L301, R3 to R301, R7 to R302, R8 to R303, R1 to R304, R9 to R305, R6 to R306, R10 to R307, R4 to R308, R13 to R309, R11 to R310, R2 to R311, SW1 to SW301, SW2 to SW302, U2 to U301, U3 to U302, U1 to U303, U4 to U304, Y1 to Y301
